File: inputs.kicad_sch (KiCad schematic)
At the start: 6 parts, among them SW1 SW_Omron_B3FS, SW2 SW_Omron_B3FS, SW3 SW_Omron_B3FS, SW4 SW_Omron_B3FS, SW5 SW_Omron_B3FS, SW6 SW_Omron_B3FS

Commit message: Add Midi & Rotary buttons
Parts:
- renumbered SW4 to SW_A, SW5 to SW_B, SW6 to SW_C, SW1 to SW_D, SW2 to SW_E, SW3 to SW_F
Connections:
- net SW_A: now reaches SW_A.1
- net SW_E: now reaches SW_E.1
- net SW_C: now reaches SW_C.1
- net SW_B: now reaches SW_B.1
- net SW_D: now reaches SW_D.1
- net SW_F: now reaches SW_F.1
Changed lines of the file:
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@@
     (stroke (width 0) (type default))
+  )
+  (label "SW_D" (at 34.29 41.91 180) (fields_autoplaced)
+    (effects (font (size 1.27 1.27)) (justify right bottom))
+  )
+  (label "SW_E" (at 77.47 41.91 180) (fields_autoplaced)
+    (effects (font (size 1.27 1.27)) (justify right bottom))
+  )
+  (label "SW_B" (at 77.47 73.66 180) (fields_autoplaced)
+    (effects (font (size 1.27 1.27)) (justify right bottom))
+  )
+  (label "SW_F" (at 118.11 41.91 180) (fields_autoplaced)
+    (effects (font (size 1.27 1.27)) (justify right bottom))
+  )
+  (label "SW_A" (at 34.29 73.66 180) (fields_autoplaced)
+    (effects (font (size 1.27 1.27)) (justify right bottom))
+  )
+  (label "SW_C" (at 118.11 72.39 180) (fields_autoplaced)
+    (effects (font (size 1.27 1.27)) (justify right bottom))
   )
   (symbol (lib_id "Switch:SW_Omron_B3FS") (at 39.37 73.66 0) (unit 1)
     (in_bom yes) (on_board yes) (dnp no) (fields_autoplaced)
-    (property "Reference" "SW4" (at 39.37 67.31 0)
+    (property "Reference" "SW_A" (at 39.37 67.31 0)
       (effects (font (size 1.27 1.27)))
     )
@@
       (project "pedalboard-hw"
         (path "/df521c2a-9827-4355-b809-366f4b88d5d7/e0e8fe71-102f-4387-ab09-5b5a9ebe3509"
-          (reference "SW4") (unit 1)
+          (reference "SW_A") (unit 1)
         )
       )
@@
   (symbol (lib_id "Switch:SW_Omron_B3FS") (at 82.55 41.91 0) (unit 1)
     (in_bom yes) (on_board yes) (dnp no) (fields_autoplaced)
-    (property "Reference" "SW2" (at 82.55 35.56 0)
+    (property "Reference" "SW_E" (at 82.55 35.56 0)
       (effects (font (size 1.27 1.27)))
     )
@@
       (project "pedalboard-hw"
         (path "/df521c2a-9827-4355-b809-366f4b88d5d7/e0e8fe71-102f-4387-ab09-5b5a9ebe3509"
-          (reference "SW2") (unit 1)
+          (reference "SW_E") (unit 1)
         )
       )
@@
   (symbol (lib_id "Switch:SW_Omron_B3FS") (at 123.19 72.39 0) (unit 1)
     (in_bom yes) (on_board yes) (dnp no) (fields_autoplaced)
-    (property "Reference" "SW6" (at 123.19 66.04 0)
+    (property "Reference" "SW_C" (at 123.19 66.04 0)
       (effects (font (size 1.27 1.27)))
     )
@@
       (project "pedalboard-hw"
         (path "/df521c2a-9827-4355-b809-366f4b88d5d7/e0e8fe71-102f-4387-ab09-5b5a9ebe3509"
-          (reference "SW6") (unit 1)
+          (reference "SW_C") (unit 1)
         )
       )
@@
   (symbol (lib_id "Switch:SW_Omron_B3FS") (at 82.55 73.66 0) (unit 1)
     (in_bom yes) (on_board yes) (dnp no) (fields_autoplaced)
-    (property "Reference" "SW5" (at 82.55 67.31 0)
+    (property "Reference" "SW_B" (at 82.55 67.31 0)
       (effects (font (size 1.27 1.27)))
     )
@@
       (project "pedalboard-hw"
         (path "/df521c2a-9827-4355-b809-366f4b88d5d7/e0e8fe71-102f-4387-ab09-5b5a9ebe3509"
-          (reference "SW5") (unit 1)
+          (reference "SW_B") (unit 1)
         )
       )
@@
   (symbol (lib_id "Switch:SW_Omron_B3FS") (at 39.37 41.91 0) (unit 1)
     (in_bom yes) (on_board yes) (dnp no) (fields_autoplaced)
-    (property "Reference" "SW1" (at 39.37 35.56 0)
+    (property "Reference" "SW_D" (at 39.37 35.56 0)
       (effects (font (size 1.27 1.27)))
     )
@@
       (project "pedalboard-hw"
         (path "/df521c2a-9827-4355-b809-366f4b88d5d7/e0e8fe71-102f-4387-ab09-5b5a9ebe3509"
-          (reference "SW1") (unit 1)
+          (reference "SW_D") (unit 1)
         )
       )
@@
   (symbol (lib_id "Switch:SW_Omron_B3FS") (at 123.19 41.91 0) (unit 1)
     (in_bom yes) (on_board yes) (dnp no) (fields_autoplaced)
-    (property "Reference" "SW3" (at 123.19 35.56 0)
+    (property "Reference" "SW_F" (at 123.19 35.56 0)
       (effects (font (size 1.27 1.27)))
     )
@@
       (project "pedalboard-hw"
         (path "/df521c2a-9827-4355-b809-366f4b88d5d7/e0e8fe71-102f-4387-ab09-5b5a9ebe3509"
-          (reference "SW3") (unit 1)
+          (reference "SW_F") (unit 1)
         )
       )
