File: pedalboard-hw.kicad_pcb (KiCad board)
At the start: 2 copper layers, 170 x 105 mm, 58 parts, among them J1 MIDI_OUT, J10 Audio IN Left, J11 Audio OUT Right, J12 Audio OUT Left, J13 Audio OUT, J14 Audio IN, J15 MIDI IN/OUT, J16 MIDI OUT J, J17 MIDI IN J, J2 MIDI_IN, J3 EXP, J4 RGB_LED_EXT, J5 Pico USB TP, J6 USB_A, J7 Raspberry_pi, J8 HiFi Berry, J9 Audio IN Right, SW1 D, SW2 E, SW3 F, SW4 A, SW5 B, SW6 C, SW7 VOL Rotary, SW8 GAIN Rotary, U1 Pico, U2 H11L1

Commit message: Auto place midi circuit
Parts:
- moved L3 99.3 mm to (136.0, 22.0)
- moved C1 41.1 mm to (79.0, 31.0)
- moved U2 27.4 mm to (59.2, 103.4)
- moved R2 22.4 mm to (68.2, 76.4)
- moved R4 18.6 mm to (78.2, 110.4)
- moved R1 18.4 mm to (67.2, 91.4)
- moved R3 17.1 mm to (62.2, 104.4)
- moved L4 13.1 mm to (71.2, 115.4)
- moved D11 11.3 mm to (75.2, 104.4)
- moved L2 10.3 mm to (62.2, 97.4)
- moved R5 10.2 mm to (72.5, 56.7)
- moved L1 3.20 mm to (68.2, 85.4)
Changed lines of the file:
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@@
     )
   )
-  (footprint "Resistor_THT:R_Axial_DIN0207_L6.3mm_D2.5mm_P10.16mm_Horizontal" (layer "F.Cu")
-    (at 79.95 63.7 180)
+  (footprint "Resistor_THT:R_Axial_DIN0207_L6.3mm_D2.5mm_P10.16mm_Horizontal" placed (layer "F.Cu")
+    (at 72.47 56.72 180)
     (descr "Resistor, Axial_DIN0207 series, Axial, Horizontal, pin pitch=10.16mm, 0.25W = 1/4W, length*diameter=6.3*2.5mm^2, http://cdn-reichelt.de/documents/datenblatt/B400/1_4W%23YAG.pdf")
     (tags "Resistor Axial_DIN0207 series Axial Horizontal pin pitch 10.16mm 0.25W = 1/4W length 6.3mm diameter 2.5mm")
@@
     )
   )
-  (footprint "Package_DIP:DIP-6_W7.62mm_LongPads" (layer "F.Cu")
-    (at 72.825 79.525 180)
+  (footprint "Package_DIP:DIP-6_W7.62mm_LongPads" placed (layer "F.Cu")
+    (at 59.25 103.36 180)
     (descr "6-lead though-hole mounted DIP package, row spacing 7.62 mm (300 mils), LongPads")
     (tags "THT DIP DIL PDIP 2.54mm 7.62mm 300mil LongPads")
@@
     )
   )
-  (footprint "Capacitor_THT:C_Disc_D3.0mm_W1.6mm_P2.50mm" (layer "F.Cu")
-    (at 65.35 69.8)
+  (footprint "Capacitor_THT:C_Disc_D3.0mm_W1.6mm_P2.50mm" placed (layer "F.Cu")
+    (at 79 31)
     (descr "C, Disc series, Radial, pin pitch=2.50mm, , diameter*width=3.0*1.6mm^2, Capacitor, http://www.vishay.com/docs/45233/krseries.pdf")
     (tags "C Disc series Radial pin pitch 2.50mm  diameter 3.0mm width 1.6mm Capacitor")
@@
     )
   )
-  (footprint "Resistor_THT:R_Axial_DIN0207_L6.3mm_D2.5mm_P10.16mm_Horizontal" (layer "F.Cu")
-    (at 49.65 96.8)
+  (footprint "Resistor_THT:R_Axial_DIN0207_L6.3mm_D2.5mm_P10.16mm_Horizontal" placed (layer "F.Cu")
+    (at 67.25 91.36)
     (descr "Resistor, Axial_DIN0207 series, Axial, Horizontal, pin pitch=10.16mm, 0.25W = 1/4W, length*diameter=6.3*2.5mm^2, http://cdn-reichelt.de/documents/datenblatt/B400/1_4W%23YAG.pdf")
     (tags "Resistor Axial_DIN0207 series Axial Horizontal pin pitch 10.16mm 0.25W = 1/4W length 6.3mm diameter 2.5mm")
@@
     )
   )
-  (footprint "Resistor_THT:R_Axial_DIN0207_L6.3mm_D2.5mm_P10.16mm_Horizontal" (layer "F.Cu")
-    (at 49.65 92.8)
+  (footprint "Resistor_THT:R_Axial_DIN0207_L6.3mm_D2.5mm_P10.16mm_Horizontal" placed (layer "F.Cu")
+    (at 62.25 104.36)
     (descr "Resistor, Axial_DIN0207 series, Axial, Horizontal, pin pitch=10.16mm, 0.25W = 1/4W, length*diameter=6.3*2.5mm^2, http://cdn-reichelt.de/documents/datenblatt/B400/1_4W%23YAG.pdf")
     (tags "Resistor Axial_DIN0207 series Axial Horizontal pin pitch 10.16mm 0.25W = 1/4W length 6.3mm diameter 2.5mm")
@@
     )
   )
-  (footprint "Resistor_THT:R_Axial_DIN0207_L6.3mm_D2.5mm_P10.16mm_Horizontal" (layer "F.Cu")
-    (at 62.35 100.8 180)
+  (footprint "Resistor_THT:R_Axial_DIN0207_L6.3mm_D2.5mm_P10.16mm_Horizontal" placed (layer "F.Cu")
+    (at 78.25 110.36 180)
     (descr "Resistor, Axial_DIN0207 series, Axial, Horizontal, pin pitch=10.16mm, 0.25W = 1/4W, length*diameter=6.3*2.5mm^2, http://cdn-reichelt.de/documents/datenblatt/B400/1_4W%23YAG.pdf")
     (tags "Resistor Axial_DIN0207 series Axial Horizontal pin pitch 10.16mm 0.25W = 1/4W length 6.3mm diameter 2.5mm")
@@
     )
   )
-  (footprint "Inductor_THT:L_Axial_L5.3mm_D2.2mm_P10.16mm_Horizontal_Vishay_IM-1" (layer "F.Cu")
-    (at 71 87)
+  (footprint "Inductor_THT:L_Axial_L5.3mm_D2.2mm_P10.16mm_Horizontal_Vishay_IM-1" placed (layer "F.Cu")
+    (at 68.25 85.36)
     (descr "Inductor, Axial series, Axial, Horizontal, pin pitch=10.16mm, , length*diameter=5.3*2.2mm^2, Vishay, IM-1, http://www.vishay.com/docs/34030/im.pdf")
     (tags "Inductor Axial series Axial Horizontal pin pitch 10.16mm  length 5.3mm diameter 2.2mm Vishay IM-1")
@@
     )
   )
-  (footprint "Diode_THT:D_DO-35_SOD27_P7.62mm_Horizontal" (layer "F.Cu")
-    (at 67 96.61 90)
+  (footprint "Diode_THT:D_DO-35_SOD27_P7.62mm_Horizontal" placed (layer "F.Cu")
+    (at 75.25 104.36 90)
     (descr "Diode, DO-35_SOD27 series, Axial, Horizontal, pin pitch=7.62mm, , length*diameter=4*2mm^2, , http://www.diodes.com/_files/packages/DO-35.pdf")
     (tags "Diode DO-35_SOD27 series Axial Horizontal pin pitch 7.62mm  length 4mm diameter 2mm")
@@
     )
   )
-  (footprint "Inductor_THT:L_Axial_L5.3mm_D2.2mm_P10.16mm_Horizontal_Vishay_IM-1" (layer "F.Cu")
-    (at 71 91.95)
+  (footprint "Inductor_THT:L_Axial_L5.3mm_D2.2mm_P10.16mm_Horizontal_Vishay_IM-1" placed (layer "F.Cu")
+    (at 62.25 97.36)
     (descr "Inductor, Axial series, Axial, Horizontal, pin pitch=10.16mm, , length*diameter=5.3*2.2mm^2, Vishay, IM-1, http://www.vishay.com/docs/34030/im.pdf")
     (tags "Inductor Axial series Axial Horizontal pin pitch 10.16mm  length 5.3mm diameter 2.2mm Vishay IM-1")
@@
     )
   )
-  (footprint "Inductor_THT:L_Axial_L5.3mm_D2.2mm_P10.16mm_Horizontal_Vishay_IM-1" (layer "F.Cu")
-    (at 71 102.25)
+  (footprint "Inductor_THT:L_Axial_L5.3mm_D2.2mm_P10.16mm_Horizontal_Vishay_IM-1" placed (layer "F.Cu")
+    (at 71.25 115.36)
     (descr "Inductor, Axial series, Axial, Horizontal, pin pitch=10.16mm, , length*diameter=5.3*2.2mm^2, Vishay, IM-1, http://www.vishay.com/docs/34030/im.pdf")
     (tags "Inductor Axial series Axial Horizontal pin pitch 10.16mm  length 5.3mm diameter 2.2mm Vishay IM-1")
@@
     )
   )
-  (footprint "Resistor_THT:R_Axial_DIN0207_L6.3mm_D2.5mm_P10.16mm_Horizontal" (layer "F.Cu")
-    (at 49.65 88.8)
+  (footprint "Resistor_THT:R_Axial_DIN0207_L6.3mm_D2.5mm_P10.16mm_Horizontal" placed (layer "F.Cu")
+    (at 68.25 76.36)
     (descr "Resistor, Axial_DIN0207 series, Axial, Horizontal, pin pitch=10.16mm, 0.25W = 1/4W, length*diameter=6.3*2.5mm^2, http://cdn-reichelt.de/documents/datenblatt/B400/1_4W%23YAG.pdf")
     (tags "Resistor Axial_DIN0207 series Axial Horizontal pin pitch 10.16mm 0.25W = 1/4W length 6.3mm diameter 2.5mm")
@@
     )
   )
-  (footprint "Inductor_THT:L_Axial_L5.3mm_D2.2mm_P10.16mm_Horizontal_Vishay_IM-1" (layer "F.Cu")
-    (at 71 97.1)
+  (footprint "Inductor_THT:L_Axial_L5.3mm_D2.2mm_P10.16mm_Horizontal_Vishay_IM-1" placed (layer "F.Cu")
+    (at 136 22)
     (descr "Inductor, Axial series, Axial, Horizontal, pin pitch=10.16mm, , length*diameter=5.3*2.2mm^2, Vishay, IM-1, http://www.vishay.com/docs/34030/im.pdf")
     (tags "Inductor Axial series Axial Horizontal pin pitch 10.16mm  length 5.3mm diameter 2.2mm Vishay IM-1")
@@
     )
   )
-  (footprint "Connector_PinHeader_2.00mm:PinHeader_1x02_P2.00mm_Vertical" (layer "B.Cu")
+  (footprint "Connector_PinHeader_2.00mm:PinHeader_1x02_P2.00mm_Vertical" locked (layer "B.Cu")
     (at 127 48 180)
     (descr "Through hole straight pin header, 1x02, 2.00mm pitch, single row")
@@
     (fp_line (start 1 1) (end 1 -3)
       (stroke (width 0.1) (type solid)) (layer "B.Fab"))
-    (pad "1" thru_hole rect (at 0 0 180) (size 1.35 1.35) (drill 0.8) (layers "*.Cu" "*.Mask")
+    (pad "1" thru_hole rect locked (at 0 0 180) (size 1.35 1.35) (drill 0.8) (layers "*.Cu" "*.Mask")
       (net 48 "/Audio/USB_DM") (pinfunction "Pin_1") (pintype "passive"))
-    (pad "2" thru_hole oval (at 0 -2 180) (size 1.35 1.35) (drill 0.8) (layers "*.Cu" "*.Mask")
+    (pad "2" thru_hole oval locked (at 0 -2 180) (size 1.35 1.35) (drill 0.8) (layers "*.Cu" "*.Mask")
       (net 123 "/Audio/USB_DP") (pinfunction "Pin_2") (pintype "passive"))
     (model "${KICAD6_3DMODEL_DIR}/Connector_PinHeader_2.00mm.3dshapes/PinHeader_1x02_P2.00mm_Vertical.wrl"

Commit message: Name the input networks for better routing
Parts:
- moved L3 92.6 mm to (81.0, 96.5), turned to -90 degrees
Routing:
- net Net-(J13-Pin_2): track 0.00 -> 55.8 mm
- net Net-(J13-Pin_6): track 0.00 -> 23.6 mm
Changed lines of the file:
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@@
   )
   (footprint "Inductor_THT:L_Axial_L5.3mm_D2.2mm_P10.16mm_Horizontal_Vishay_IM-1" placed (layer "F.Cu")
-    (at 136 22)
+    (at 80.96 96.52 -90)
     (descr "Inductor, Axial series, Axial, Horizontal, pin pitch=10.16mm, , length*diameter=5.3*2.2mm^2, Vishay, IM-1, http://www.vishay.com/docs/34030/im.pdf")
     (tags "Inductor Axial series Axial Horizontal pin pitch 10.16mm  length 5.3mm diameter 2.2mm Vishay IM-1")
@@
     (property "ki_keywords" "inductor choke coil reactor magnetic")
     (attr through_hole)
-    (fp_text reference "L3" (at 5.08 -2.22) (layer "F.SilkS")
+    (fp_text reference "L3" (at 5.08 -2.22 90) (layer "F.SilkS")
         (effects (font (size 1 1) (thickness 0.15)))
     )
-    (fp_text value "1K@100MHz" (at 5.08 2.22) (layer "F.Fab")
+    (fp_text value "1K@100MHz" (at 5.08 2.22 90) (layer "F.Fab")
         (effects (font (size 1 1) (thickness 0.15)))
     )
-    (fp_text user "${REFERENCE}" (at 5.08 0) (layer "F.Fab")
+    (fp_text user "${REFERENCE}" (at 5.08 0 90) (layer "F.Fab")
         (effects (font (size 1 1) (thickness 0.15)))
     )
@@
     (fp_line (start 10.16 0) (end 7.73 0)
       (stroke (width 0.1) (type solid)) (layer "F.Fab"))
-    (pad "1" thru_hole circle (at 0 0) (size 1.6 1.6) (drill 0.8) (layers "*.Cu" "*.Mask")
+    (pad "1" thru_hole circle (at 0 0 270) (size 1.6 1.6) (drill 0.8) (layers "*.Cu" "*.Mask")
       (net 119 "Net-(J15-Pin_6)") (pinfunction "1") (pintype "passive"))
-    (pad "2" thru_hole oval (at 10.16 0) (size 1.6 1.6) (drill 0.8) (layers "*.Cu" "*.Mask")
+    (pad "2" thru_hole oval (at 10.16 0 270) (size 1.6 1.6) (drill 0.8) (layers "*.Cu" "*.Mask")
       (net 116 "Net-(L3-Pad2)") (pinfunction "2") (pintype "passive"))
     (model "${KICAD6_3DMODEL_DIR}/Inductor_THT.3dshapes/L_Axial_L5.3mm_D2.2mm_P10.16mm_Horizontal_Vishay_IM-1.wrl"
@@
   (gr_arc (start 190 124) (mid 189.707107 124.707107) (end 189 125)
     (stroke (width 0.1) (type default)) (layer "Edge.Cuts"))
+  (segment (start 39.812 108.077) (end 39.939 108.204) (width 0.25) (layer "F.Cu") (net 89))
+  (segment (start 45.273 116.078) (end 60.64 116.078) (width 0.25) (layer "F.Cu") (net 89))
+  (segment (start 36.225 92.79) (end 36.225 107.792) (width 0.25) (layer "F.Cu") (net 89))
+  (segment (start 61.7732 121.5292) (end 58.7962 121.5292) (width 0.25) (layer "F.Cu") (net 89))
+  (segment (start 36.51 108.077) (end 39.812 108.077) (width 0.25) (layer "F.Cu") (net 89))
+  (segment (start 60.64 116.078) (end 61.783 117.221) (width 0.25) (layer "F.Cu") (net 89))
+  (segment (start 36.225 107.792) (end 36.51 108.077) (width 0.25) (layer "F.Cu") (net 89))
+  (segment (start 39.939 110.744) (end 45.273 116.078) (width 0.25) (layer "F.Cu") (net 89))
+  (segment (start 61.783 121.539) (end 61.7732 121.5292) (width 0.25) (layer "F.Cu") (net 89))
+  (segment (start 34.435 91) (end 36.225 92.79) (width 0.25) (layer "F.Cu") (net 89))
+  (segment (start 39.939 108.204) (end 39.939 110.744) (width 0.25) (layer "F.Cu") (net 89))
+  (segment (start 61.783 117.221) (end 61.783 121.539) (width 0.25) (layer "F.Cu") (net 89))
+  (segment (start 49.591 121.539) (end 49.6008 121.5292) (width 0.25) (layer "F.Cu") (net 94))
+  (segment (start 34.4 111.2) (end 39.252 111.2) (width 0.25) (layer "F.Cu") (net 94))
+  (segment (start 39.252 111.2) (end 49.591 121.539) (width 0.25) (layer "F.Cu") (net 94))
+  (segment (start 49.6008 121.5292) (end 53.7162 121.5292) (width 0.25) (layer "F.Cu") (net 94))
 )

Commit message: Routing of the audio output
Connections:
- net Net-(J14-Pin_1) renamed /Audio/audio out R-
- net Net-(J14-Pin_5) renamed /Audio/audio out L+
- J10 pad S: Net-(J14-Pin_4) -> GNDA
- J14 pad 3: Net-(J14-Pin_3) -> GNDA
- J14 pad 4: Net-(J14-Pin_4) -> GNDA
- J9 pad S: Net-(J14-Pin_3) -> GNDA
Routing:
- net Net-(J13-Pin_4): track 0.00 -> 63.8 mm
- net Net-(J13-Pin_2): track 55.8 -> 53.3 mm

Commit message: Re-place midi circuit
Parts:
- moved U2 15.6 mm to (66.5, 89.5)
- moved R1 13.2 mm to (80.3, 89.9), turned to 180 degrees
- moved L1 1.41 mm to (69.7, 85.5)
Changed lines of the file:
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@@
   )
   (footprint "Package_DIP:DIP-6_W7.62mm_LongPads" placed (layer "F.Cu")
-    (at 59.25 103.36 180)
+    (at 66.497 89.52 180)
     (descr "6-lead though-hole mounted DIP package, row spacing 7.62 mm (300 mils), LongPads")
     (tags "THT DIP DIL PDIP 2.54mm 7.62mm 300mil LongPads")
@@
   )
   (footprint "Resistor_THT:R_Axial_DIN0207_L6.3mm_D2.5mm_P10.16mm_Horizontal" placed (layer "F.Cu")
-    (at 67.25 91.36)
+    (at 80.325 89.916 180)
     (descr "Resistor, Axial_DIN0207 series, Axial, Horizontal, pin pitch=10.16mm, 0.25W = 1/4W, length*diameter=6.3*2.5mm^2, http://cdn-reichelt.de/documents/datenblatt/B400/1_4W%23YAG.pdf")
     (tags "Resistor Axial_DIN0207 series Axial Horizontal pin pitch 10.16mm 0.25W = 1/4W length 6.3mm diameter 2.5mm")
@@
     (fp_line (start 10.16 0) (end 8.23 0)
       (stroke (width 0.1) (type solid)) (layer "F.Fab"))
-    (pad "1" thru_hole circle (at 0 0) (size 1.6 1.6) (drill 0.8) (layers "*.Cu" "*.Mask")
+    (pad "1" thru_hole circle (at 0 0 180) (size 1.6 1.6) (drill 0.8) (layers "*.Cu" "*.Mask")
       (net 114 "Net-(L1-Pad2)") (pintype "passive"))
-    (pad "2" thru_hole oval (at 10.16 0) (size 1.6 1.6) (drill 0.8) (layers "*.Cu" "*.Mask")
+    (pad "2" thru_hole oval (at 10.16 0 180) (size 1.6 1.6) (drill 0.8) (layers "*.Cu" "*.Mask")
       (net 14 "Net-(D11-K)") (pintype "passive"))
     (model "${KICAD6_3DMODEL_DIR}/Resistor_THT.3dshapes/R_Axial_DIN0207_L6.3mm_D2.5mm_P10.16mm_Horizontal.wrl"
@@
   )
   (footprint "Inductor_THT:L_Axial_L5.3mm_D2.2mm_P10.16mm_Horizontal_Vishay_IM-1" placed (layer "F.Cu")
-    (at 68.25 85.36)
+    (at 69.657 85.471)
     (descr "Inductor, Axial series, Axial, Horizontal, pin pitch=10.16mm, , length*diameter=5.3*2.2mm^2, Vishay, IM-1, http://www.vishay.com/docs/34030/im.pdf")
     (tags "Inductor Axial series Axial Horizontal pin pitch 10.16mm  length 5.3mm diameter 2.2mm Vishay IM-1")

Commit message: Route the differential analog input channels
Connections:
- net /Audio/audio out L+ renamed /Audio/audio_out_L+
- net /Audio/audio out R- renamed /Audio/audio_out_R-
- net Net-(J14-Pin_2) renamed /Audio/audio_out_R+
- net Net-(J14-Pin_6) renamed /Audio/audio_out_L-
Routing:
- net /Audio/audio_out_R+: track 0.00 -> 238.2 mm
- net /Audio/audio_out_R-: track 0.00 -> 233.8 mm
- net /Audio/audio_out_L-: track 0.00 -> 191.8 mm
- net /Audio/audio_out_L+: track 0.00 -> 191.7 mm

Commit message: Improve Routing of stereo output
Routing:
- net Net-(J13-Pin_2): track 53.3 -> 49.2 mm
Changed lines of the file:
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@@
   (segment (start 36.383 107.569) (end 21.778 107.569) (width 0.25) (layer "F.Cu") (net 86))
   (segment (start 23.116 91) (end 21.735 91) (width 0.25) (layer "F.Cu") (net 86))
-  (segment (start 34.435 91) (end 36.225 92.79) (width 0.25) (layer "F.Cu") (net 88))
-  (segment (start 59.878 115.316) (end 61.783 117.221) (width 0.25) (layer "F.Cu") (net 88))
-  (segment (start 36.225 92.806) (end 38.288 94.869) (width 0.25) (layer "F.Cu") (net 88))
-  (segment (start 61.7732 121.5292) (end 58.7962 121.5292) (width 0.25) (layer "F.Cu") (net 88))
-  (segment (start 38.288 94.869) (end 38.288 107.95) (width 0.25) (layer "F.Cu") (net 88))
-  (segment (start 38.288 107.95) (end 45.781 115.443) (width 0.25) (layer "F.Cu") (net 88))
-  (segment (start 61.783 117.221) (end 61.783 121.539) (width 0.25) (layer "F.Cu") (net 88))
-  (segment (start 45.781 115.443) (end 59.751 115.443) (width 0.25) (layer "F.Cu") (net 88))
-  (segment (start 36.225 92.79) (end 36.225 92.806) (width 0.25) (layer "F.Cu") (net 88))
-  (segment (start 61.783 121.539) (end 61.7732 121.5292) (width 0.25) (layer "F.Cu") (net 88))
-  (segment (start 59.751 115.443) (end 59.878 115.316) (width 0.25) (layer "F.Cu") (net 88))
+  (segment (start 43.876 112.649) (end 42.987 112.649) (width 0.25) (layer "F.Cu") (net 88))
+  (segment (start 60.386 119.9394) (end 60.386 117.602) (width 0.25) (layer "F.Cu") (net 88))
+  (segment (start 60.132 117.348) (end 48.575 117.348) (width 0.25) (layer "F.Cu") (net 88))
+  (segment (start 38.288 106.299) (end 38.288 94.869) (width 0.25) (layer "F.Cu") (net 88))
+  (segment (start 48.575 117.348) (end 43.876 112.649) (width 0.25) (layer "F.Cu") (net 88))
+  (segment (start 42.987 112.649) (end 40.447 110.109) (width 0.25) (layer "F.Cu") (net 88))
+  (segment (start 40.447 108.458) (end 38.288 106.299) (width 0.25) (layer "F.Cu") (net 88))
+  (segment (start 36.225 92.806) (end 36.225 92.79) (width 0.25) (layer "F.Cu") (net 88))
+  (segment (start 58.7962 121.5292) (end 60.386 119.9394) (width 0.25) (layer "F.Cu") (net 88))
+  (segment (start 38.288 94.869) (end 36.225 92.806) (width 0.25) (layer "F.Cu") (net 88))
+  (segment (start 40.447 110.109) (end 40.447 108.458) (width 0.25) (layer "F.Cu") (net 88))
+  (segment (start 36.225 92.79) (end 34.435 91) (width 0.25) (layer "F.Cu") (net 88))
+  (segment (start 60.386 117.602) (end 60.132 117.348) (width 0.25) (layer "F.Cu") (net 88))
   (segment (start 47.686 121.539) (end 37.399 111.252) (width 0.25) (layer "F.Cu") (net 93))
   (segment (start 36.966 111.2) (end 34.4 111.2) (width 0.25) (layer "F.Cu") (net 93))
