File: pedalboard-hw.kicad_pcb (KiCad board)
At the start: 2 copper layers, 170 x 105 mm, 58 parts, among them J1 MIDI_OUT, J10 Audio IN Left, J11 Audio OUT Right, J12 Audio OUT Left, J13 Audio OUT, J14 Audio IN, J15 MIDI IN/OUT, J16 MIDI OUT J, J17 MIDI IN J, J2 MIDI_IN, J3 EXP, J4 RGB_LED_EXT, J5 Pico USB TP, J6 USB_A, J7 Raspberry_pi, J8 HiFi Berry, J9 Audio IN Right, SW1 D, SW2 E, SW3 F, SW4 A, SW5 B, SW6 C, SW7 VOL Rotary, SW8 GAIN Rotary, U1 Pico, U2 H11L1

Commit message: Analog Out GND Panes
Parts:
- moved U2 4.58 mm to (69.0, 85.7)
- moved R4 3.55 mm to (81.7, 109.6)
- moved L1 2.45 mm to (71.9, 84.6)
- moved R3 2.25 mm to (62.2, 102.1)
- moved L4 1.96 mm to (73.1, 114.7)
Connections:
- J10 pad S: GNDA -> /Audio/GND_analog_out_L
- J14 pad 3: GNDA -> /Audio/GND_analog_out_R
- J14 pad 4: GNDA -> /Audio/GND_analog_out_L
- J9 pad S: GNDA -> /Audio/GND_analog_out_R
Routing:
- net /Audio/GND_analog_out_L: track 0.00 -> 16.5 mm, vias 0 -> 2
- added copper zone on B.Cu, net /Audio/GND_analog_out_L
- added copper zone on F.Cu, net /Audio/GND_analog_out_L
- added copper zone on B.Cu, net /Audio/GND_analog_out_R
- added copper zone on F.Cu, net /Audio/GND_analog_out_R
Changed lines of the file:
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@@
   (net 73 "/Audio/audio_out_R-")
   (net 74 "unconnected-(J9-PadRN)")
-  (net 75 "GNDA")
+  (net 75 "/Audio/GND_analog_out_R")
   (net 76 "unconnected-(J9-PadSN)")
   (net 77 "/Audio/audio_out_R+")
@@
   (net 123 "/Audio/V_BUS")
   (net 124 "Net-(D1-DIN)")
+  (net 125 "/Audio/GND_analog_out_L")
   (footprint "Capacitor_THT:C_Disc_D3.0mm_W1.6mm_P2.50mm" locked (layer "F.Cu")
     (at 141.15 52.4)
@@
       (net 80 "unconnected-(J10-PadRN)") (pintype "passive"))
     (pad "S" thru_hole circle locked (at 12.7 0) (size 3 3) (drill 1.4) (layers "*.Cu" "*.Mask")
-      (net 75 "GNDA") (pintype "passive"))
+      (net 125 "/Audio/GND_analog_out_L") (pintype "passive"))
     (pad "SN" thru_hole circle locked (at 12.7 16.23) (size 3 3) (drill 1.4) (layers "*.Cu" "*.Mask")
       (net 82 "unconnected-(J10-PadSN)") (pintype "passive"))
@@
   )
   (footprint "Package_DIP:DIP-6_W7.62mm_LongPads" placed (layer "F.Cu")
-    (at 66.497 89.52 180)
+    (at 69.037 85.71 180)
     (descr "6-lead though-hole mounted DIP package, row spacing 7.62 mm (300 mils), LongPads")
     (tags "THT DIP DIL PDIP 2.54mm 7.62mm 300mil LongPads")
@@
       (net 74 "unconnected-(J9-PadRN)") (pintype "passive"))
     (pad "S" thru_hole circle locked (at 12.7 0) (size 3 3) (drill 1.4) (layers "*.Cu" "*.Mask")
-      (net 75 "GNDA") (pintype "passive"))
+      (net 75 "/Audio/GND_analog_out_R") (pintype "passive"))
     (pad "SN" thru_hole circle locked (at 12.7 16.23) (size 3 3) (drill 1.4) (layers "*.Cu" "*.Mask")
       (net 76 "unconnected-(J9-PadSN)") (pintype "passive"))
@@
   )
   (footprint "Resistor_THT:R_Axial_DIN0207_L6.3mm_D2.5mm_P10.16mm_Horizontal" placed (layer "F.Cu")
-    (at 62.25 104.36)
+    (at 62.25 102.108)
     (descr "Resistor, Axial_DIN0207 series, Axial, Horizontal, pin pitch=10.16mm, 0.25W = 1/4W, length*diameter=6.3*2.5mm^2, http://cdn-reichelt.de/documents/datenblatt/B400/1_4W%23YAG.pdf")
     (tags "Resistor Axial_DIN0207 series Axial Horizontal pin pitch 10.16mm 0.25W = 1/4W length 6.3mm diameter 2.5mm")
@@
   )
   (footprint "Resistor_THT:R_Axial_DIN0207_L6.3mm_D2.5mm_P10.16mm_Horizontal" placed (layer "F.Cu")
-    (at 78.25 110.36 180)
+    (at 81.722 109.601 180)
     (descr "Resistor, Axial_DIN0207 series, Axial, Horizontal, pin pitch=10.16mm, 0.25W = 1/4W, length*diameter=6.3*2.5mm^2, http://cdn-reichelt.de/documents/datenblatt/B400/1_4W%23YAG.pdf")
     (tags "Resistor Axial_DIN0207 series Axial Horizontal pin pitch 10.16mm 0.25W = 1/4W length 6.3mm diameter 2.5mm")
@@
   )
   (footprint "Inductor_THT:L_Axial_L5.3mm_D2.2mm_P10.16mm_Horizontal_Vishay_IM-1" placed (layer "F.Cu")
-    (at 69.657 85.471)
+    (at 71.943 84.582)
     (descr "Inductor, Axial series, Axial, Horizontal, pin pitch=10.16mm, , length*diameter=5.3*2.2mm^2, Vishay, IM-1, http://www.vishay.com/docs/34030/im.pdf")
     (tags "Inductor Axial series Axial Horizontal pin pitch 10.16mm  length 5.3mm diameter 2.2mm Vishay IM-1")
@@
   )
   (footprint "Inductor_THT:L_Axial_L5.3mm_D2.2mm_P10.16mm_Horizontal_Vishay_IM-1" placed (layer "F.Cu")
-    (at 71.25 115.36)
+    (at 73.086 114.681)
     (descr "Inductor, Axial series, Axial, Horizontal, pin pitch=10.16mm, , length*diameter=5.3*2.2mm^2, Vishay, IM-1, http://www.vishay.com/docs/34030/im.pdf")
     (tags "Inductor Axial series Axial Horizontal pin pitch 10.16mm  length 5.3mm diameter 2.2mm Vishay IM-1")
@@
       (net 77 "/Audio/audio_out_R+") (pinfunction "Pin_2") (pintype "passive"))
     (pad "3" thru_hole oval locked (at 0 -2.54 180) (size 1.7 1.7) (drill 1) (layers "*.Cu" "*.Mask")
-      (net 75 "GNDA") (pinfunction "Pin_3") (pintype "passive"))
+      (net 75 "/Audio/GND_analog_out_R") (pinfunction "Pin_3") (pintype "passive"))
     (pad "4" thru_hole oval locked (at -2.54 -2.54 180) (size 1.7 1.7) (drill 1) (layers "*.Cu" "*.Mask")
-      (net 75 "GNDA") (pinfunction "Pin_4") (pintype "passive"))
+      (net 125 "/Audio/GND_analog_out_L") (pinfunction "Pin_4") (pintype "passive"))
     (pad "5" thru_hole oval locked (at 0 -5.08 180) (size 1.7 1.7) (drill 1) (layers "*.Cu" "*.Mask")
       (net 81 "/Audio/audio_out_L+") (pinfunction "Pin_5") (pintype "passive"))
@@
   (segment (start 49.591 121.539) (end 47.686 121.539) (width 0.25) (layer "F.Cu") (net 93))
   (segment (start 49.6008 121.5292) (end 53.7162 121.5292) (width 0.25) (layer "F.Cu") (net 93))
+  (segment (start 56.175 77.1904) (end 54.8794 78.486) (width 0.25) (layer "F.Cu") (net 125))
+  (segment (start 54.8794 78.486) (end 53.02 78.486) (width 0.25) (layer "F.Cu") (net 125))
+  (via (at 105.344 120.523) (size 0.8) (drill 0.4) (layers "F.Cu" "B.Cu") (free) (net 125))
+  (via (at 175.956 102.108) (size 0.8) (drill 0.4) (layers "F.Cu" "B.Cu") (free) (net 125))
+  (segment (start 188.3 94.995) (end 188.3 100.178) (width 0.25) (layer "B.Cu") (net 125))
+  (segment (start 188.3 100.178) (end 188.275 100.203) (width 0.25) (layer "B.Cu") (net 125))
+  (segment (start 188.275 100.203) (end 180.655 100.203) (width 0.25) (layer "B.Cu") (net 125))
+  (zone (net 75) (net_name "/Audio/GND_analog_out_R") (layers "F&B.Cu") (name "GND_analog_out_R") (hatch edge 0.5)
+    (connect_pads (clearance 0.4))
+    (min_thickness 0.25) (filled_areas_thickness no)
+    (fill yes (thermal_gap 0.5) (thermal_bridge_width 0.5))
+    (polygon
+      (pts
+        (xy 54.415994 77.47)
+        (xy 52.131 77.343)
+        (xy 52.131 101.219)
+        (xy 72.324 121.412)
+        (xy 145.984 121.412)
+        (xy 150.81 116.586)
+        (xy 177.734 116.586)
+        (xy 179.131 115.189)
+        (xy 179.131 108.712)
+        (xy 181.925 105.918)
+        (xy 181.925 85.471)
+        (xy 177.861 81.407)
+        (xy 171.511 81.407)
+        (xy 171.511 71.882)
+        (xy 171.638 71.755)
+        (xy 177.353 71.755)
+        (xy 180.02 69.088)
+        (xy 182.433 69.088)
+        (xy 185.1 71.755)
+        (xy 190.053 71.755)
+        (xy 190.053 123.952)
+        (xy 189.164 124.841)
+        (xy 189.164 124.968)
+        (xy 69.784 124.968)
+        (xy 46.67 101.854)
+        (xy 46.67 73.533)
+        (xy 50.226 69.977)
+        (xy 56.195 69.977)
+        (xy 57.592 71.374)
+        (xy 57.592 74.93)
+      )
+    )
+  )
+  (zone (net 125) (net_name "/Audio/GND_analog_out_L") (layers "F&B.Cu") (hatch edge 0.5)
+    (priority 1)
+    (connect_pads (clearance 0.4))
+    (min_thickness 0.25) (filled_areas_thickness no)
+    (fill yes (thermal_gap 0.5) (thermal_bridge_width 0.5))
+    (polygon
+      (pts
+        (xy 58.473411 81.534)
+        (xy 58.44613 76.835)
+        (xy 56.654223 76.835)
+        (xy 55.288565 78.232)
+        (xy 52.131 78.232)
+        (xy 52.131 101.219)
+        (xy 72.324 121.412)
+        (xy 145.984 121.412)
+        (xy 150.81 116.586)
+        (xy 177.734 116.586)
+        (xy 179.131 115.189)
+        (xy 179.131 108.712)
+        (xy 181.925 105.918)
+        (xy 181.925 100.3935)
+        (xy 181.925 94.869)
+        (xy 181.925 85.471)
+        (xy 180.147 83.693)
+        (xy 168.717 83.693)
+        (xy 168.717 110.998)
+        (xy 167.701 112.014)
+        (xy 146.619 112.014)
+        (xy 142.047 116.586)
+        (xy 115.123 116.586)
+        (xy 111.313 112.776)
+        (xy 98.737816 112.905184)
+        (xy 98.74 112.903)
+        (xy 95.438 112.903)
+        (xy 90.485 117.856)
+        (xy 74.61 117.856)
+        (xy 57.592 100.838)
+        (xy 57.522908 82.69176)
+      )
+    )
+  )
 )

Commit message: Analog Out GND Panes
Parts:
- moved C9 4.49 mm to (47.4, 110.4)
Connections:
- net /Audio/GND_analog_out_L renamed /Audio/GND_in_L
- net /Audio/GND_analog_out_R renamed /Audio/GND_in_R
- net /Audio/audio_out_L+ renamed /Audio/audio_in_L+
- net /Audio/audio_out_L- renamed /Audio/in_L-
- net /Audio/audio_out_R+ renamed /Audio/in_R+
- net /Audio/audio_out_R- renamed /Audio/in_R-
- net Net-(J13-Pin_4) renamed /Audio/GND_out
Routing:
- added copper zone on B.Cu, net /Audio/GND_out
- added copper zone on F.Cu, net /Audio/GND_out
