File: pedalboard-hw.kicad_pcb (KiCad board)
At the start: 2 copper layers, 170 x 105 mm, 58 parts, among them J1 MIDI_OUT, J10 Audio IN Left, J11 Audio OUT Right, J12 Audio OUT Left, J13 Audio OUT, J14 Audio IN, J15 MIDI IN/OUT, J16 MIDI OUT J, J17 MIDI IN J, J2 MIDI_IN, J3 EXP, J4 RGB_LED_EXT, J5 Pico USB TP, J6 USB_A, J7 Raspberry_pi, J8 HiFi Berry, J9 Audio IN Right, SW1 D, SW2 E, SW3 F, SW4 A, SW5 B, SW6 C, SW7 VOL Rotary, SW8 GAIN Rotary, U1 Pico, U2 H11L1

Commit message: Fixing connection issues
Routing:
- net GND: track 36.7 -> 103.7 mm
- net /MIDI/SW_B: track 81.4 -> 76.2 mm
- net Net-(J15-Pin_3): track 97.9 -> 101.1 mm
- net /Audio/GND_in_L: vias 2 -> 3
Changed lines of the file:
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@@
-      )
-      (stroke (width 0.1) (type solid)) (fill solid) (layer "Dwgs.User"))
-    (fp_poly
-      (pts
-        (xy 3.7 20.2)
-        (xy -3.7 20.2)
-        (xy -3.7 24.9)
-        (xy 3.7 24.9)
       )
       (stroke (width 0.1) (type solid)) (fill solid) (layer "Dwgs.User"))
@@
     (stroke (width 0.1) (type default)) (layer "Edge.Cuts"))
   (segment (start 157.455 101.54) (end 156.555 100.64) (width 0.25) (layer "B.Cu") (net 1))
+  (segment (start 117.595 121.5) (end 117.655 121.44) (width 0.25) (layer "B.Cu") (net 1))
+  (segment (start 117.655 115.34) (end 117.755 115.24) (width 0.25) (layer "B.Cu") (net 1))
+  (segment (start 117.655 121.44) (end 117.655 115.34) (width 0.25) (layer "B.Cu") (net 1))
   (segment (start 157.555 122.905) (end 157.555 110.14) (width 0.25) (layer "B.Cu") (net 1))
   (segment (start 116.975 31.025) (end 116 32) (width 0.25) (layer "B.Cu") (net 1))
+  (segment (start 77.4322 26.54) (end 75.855 26.54) (width 0.25) (layer "B.Cu") (net 1))
   (segment (start 157.46 123) (end 157.555 122.905) (width 0.25) (layer "B.Cu") (net 1))
   (segment (start 156.555 100.64) (end 151 100.64) (width 0.25) (layer "B.Cu") (net 1))
   (segment (start 157.555 110.14) (end 157.455 110.04) (width 0.25) (layer "B.Cu") (net 1))
+  (segment (start 114.9172 23.4172) (end 80.555 23.4172) (width 0.25) (layer "B.Cu") (net 1))
+  (segment (start 116 24.5) (end 114.9172 23.4172) (width 0.25) (layer "B.Cu") (net 1))
   (segment (start 157.455 110.04) (end 157.455 101.54) (width 0.25) (layer "B.Cu") (net 1))
+  (segment (start 111.25 121.5) (end 98.75 121.5) (width 0.25) (layer "B.Cu") (net 1))
+  (segment (start 111.25 121.5) (end 117.595 121.5) (width 0.25) (layer "B.Cu") (net 1))
+  (segment (start 80.555 23.4172) (end 77.4322 26.54) (width 0.25) (layer "B.Cu") (net 1))
   (segment (start 116 24.5) (end 116.975 25.475) (width 0.25) (layer "B.Cu") (net 1))
   (segment (start 116.975 25.475) (end 116.975 31.025) (width 0.25) (layer "B.Cu") (net 1))
@@
   (segment (start 175.615 33.8) (end 143 33.8) (width 0.25) (layer "B.Cu") (net 19))
   (segment (start 132.82 38.59) (end 131.365 37.135) (width 0.25) (layer "B.Cu") (net 19))
+  (segment (start 124.59 62.005) (end 124.59 57.89) (width 0.25) (layer "F.Cu") (net 21))
+  (segment (start 119.555 67.04) (end 124.59 62.005) (width 0.25) (layer "F.Cu") (net 21))
   (segment (start 66.335 77.46) (end 69.06 80.185) (width 0.25) (layer "F.Cu") (net 21))
   (segment (start 95.432614 65.34) (end 97.132614 67.04) (width 0.25) (layer "F.Cu") (net 21))
   (segment (start 64.655 77.46) (end 66.335 77.46) (width 0.25) (layer "F.Cu") (net 21))
-  (segment (start 119.555 67.04) (end 124.955 61.64) (width 0.25) (layer "F.Cu") (net 21))
-  (segment (start 124.59 61.275) (end 124.59 57.89) (width 0.25) (layer "F.Cu") (net 21))
-  (segment (start 124.955 61.64) (end 124.59 61.275) (width 0.25) (layer "F.Cu") (net 21))
   (segment (start 97.132614 67.04) (end 119.555 67.04) (width 0.25) (layer "F.Cu") (net 21))
   (segment (start 69.06 80.185) (end 83.905 65.34) (width 0.25) (layer "F.Cu") (net 21))
@@
   (segment (start 24.7 74.1) (end 21 70.4) (width 0.25) (layer "B.Cu") (net 95))
   (segment (start 21 61.24) (end 102.53 61.24) (width 0.25) (layer "B.Cu") (net 95))
-  (segment (start 119.06 115.74) (end 119.06 67.06) (width 0.25) (layer "B.Cu") (net 96))
   (segment (start 98.75 116.5) (end 111.25 116.5) (width 0.25) (layer "B.Cu") (net 96))
-  (segment (start 111.25 116.5) (end 118.3 116.5) (width 0.25) (layer "B.Cu") (net 96))
-  (segment (start 118.3 116.5) (end 119.06 115.74) (width 0.25) (layer "B.Cu") (net 96))
-  (segment (start 119.06 67.06) (end 111.89 59.89) (width 0.25) (layer "B.Cu") (net 96))
   (segment (start 111.89 59.89) (end 111.89 57.89) (width 0.25) (layer "B.Cu") (net 96))
+  (segment (start 115.055 116.5) (end 115.055 63.055) (width 0.25) (layer "B.Cu") (net 96))
+  (segment (start 115.055 63.055) (end 111.89 59.89) (width 0.25) (layer "B.Cu") (net 96))
+  (segment (start 111.25 116.5) (end 115.055 116.5) (width 0.25) (layer "B.Cu") (net 96))
   (segment (start 134.655 39.94) (end 133.427792 39.94) (width 0.25) (layer "B.Cu") (net 97))
   (segment (start 173.75 116.5) (end 173.51 116.74) (width 0.25) (layer "B.Cu") (net 97))
@@
   (segment (start 113.5 29.5) (end 113.5 33.585) (width 0.25) (layer "B.Cu") (net 113))
   (segment (start 62.855 82.64) (end 58.955 86.54) (width 0.25) (layer "B.Cu") (net 113))
-  (segment (start 87.665 35.8405) (end 87.665 35.386886) (width 0.25) (layer "F.Cu") (net 114))
-  (segment (start 89.0055 34.5) (end 87.665 35.8405) (width 0.25) (layer "F.Cu") (net 114))
+  (segment (start 89.0055 34.5) (end 86.778114 34.5) (width 0.25) (layer "F.Cu") (net 114))
   (segment (start 66.605 72.19) (end 70.655 76.24) (width 0.25) (layer "F.Cu") (net 114))
-  (segment (start 72.355 76.24) (end 70.775 76.24) (width 0.25) (layer "F.Cu") (net 114))
+  (segment (start 63.955 38.985584) (end 63.955 63.34) (width 0.25) (layer "F.Cu") (net 114))
   (segment (start 96.5 32.285) (end 96.5 29.5) (width 0.25) (layer "F.Cu") (net 114))
   (segment (start 96.555 32.34) (end 96.5 32.285) (width 0.25) (layer "F.Cu") (net 114))
-  (segment (start 63.955 38.985584) (end 63.955 63.34) (width 0.25) (layer "F.Cu") (net 114))
-  (segment (start 68.600584 34.34) (end 63.955 38.985584) (width 0.25) (layer "F.Cu") (net 114))
+  (segment (start 74.150584 28.79) (end 63.955 38.985584) (width 0.25) (layer "F.Cu") (net 114))
+  (segment (start 81.068114 28.79) (end 74.150584 28.79) (width 0.25) (layer "F.Cu") (net 114))
+  (segment (start 96.5 29.5) (end 99 29.5) (width 0.25) (layer "F.Cu") (net 114))
+  (segment (start 72.355 76.24) (end 70.775 76.24) (width 0.25) (layer "F.Cu") (net 114))
+  (segment (start 89.0055 34.5) (end 94.395 34.5) (width 0.25) (layer "F.Cu") (net 114))
+  (segment (start 71.755 63.34) (end 75.355 66.94) (width 0.25) (layer "F.Cu") (net 114))
+  (segment (start 75.355 73.24) (end 72.355 76.24) (width 0.25) (layer "F.Cu") (net 114))
+  (segment (start 70.655 76.24) (end 70.775 76.24) (width 0.25) (layer "F.Cu") (net 114))
+  (segment (start 86.778114 34.5) (end 81.068114 28.79) (width 0.25) (layer "F.Cu") (net 114))
+  (segment (start 63.955 63.34) (end 71.755 63.34) (width 0.25) (layer "F.Cu") (net 114))
   (segment (start 75.355 66.94) (end 75.355 73.24) (width 0.25) (layer "F.Cu") (net 114))
-  (segment (start 96.5 29.5) (end 99 29.5) (width 0.25) (layer "F.Cu") (net 114))
-  (segment (start 89.0055 34.5) (end 94.395 34.5) (width 0.25) (layer "F.Cu") (net 114))
-  (segment (start 87.665 35.386886) (end 86.618114 34.34) (width 0.25) (layer "F.Cu") (net 114))
-  (segment (start 86.618114 34.34) (end 68.600584 34.34) (width 0.25) (layer "F.Cu") (net 114))
-  (segment (start 63.955 63.34) (end 71.755 63.34) (width 0.25) (layer "F.Cu") (net 114))
-  (segment (start 70.655 76.24) (end 70.775 76.24) (width 0.25) (layer "F.Cu") (net 114))
-  (segment (start 75.355 73.24) (end 72.355 76.24) (width 0.25) (layer "F.Cu") (net 114))
-  (segment (start 71.755 63.34) (end 75.355 66.94) (width 0.25) (layer "F.Cu") (net 114))
   (segment (start 67.04 72.19) (end 66.605 72.19) (width 0.25) (layer "F.Cu") (net 114))
   (segment (start 94.395 34.5) (end 96.555 32.34) (width 0.25) (layer "F.Cu") (net 114))
@@
   (segment (start 54.8794 78.486) (end 53.02 78.486) (width 0.25) (layer "F.Cu") (net 123))
   (via (at 105.344 120.523) (size 0.8) (drill 0.4) (layers "F.Cu" "B.Cu") (free) (net 123))
+  (via (at 129.155 120.74) (size 0.8) (drill 0.4) (layers "F.Cu" "B.Cu") (free) (net 123))
   (via (at 175.956 102.108) (size 0.8) (drill 0.4) (layers "F.Cu" "B.Cu") (free) (net 123))
   (segment (start 188.3 94.995) (end 188.3 100.178) (width 0.25) (layer "B.Cu") (net 123))
