File: pedalboard-hw.kicad_pcb (KiCad board)
At the start: 2 copper layers, 170 x 105 mm, 58 parts, among them J1 MIDI_OUT, J10 Audio IN Left, J11 Audio OUT Right, J12 Audio OUT Left, J13 Audio OUT, J14 Audio IN, J15 MIDI IN/OUT, J16 MIDI OUT J, J17 MIDI IN J, J2 MIDI_IN, J3 EXP, J4 RGB_LED_EXT, J5 Pico USB TP, J6 USB_A, J7 Raspberry_pi, J8 HiFi Berry, J9 Audio IN Right, SW1 D, SW2 E, SW3 F, SW4 A, SW5 B, SW6 C, SW7 VOL Rotary, SW8 GAIN Rotary, U1 Pico, U2 H11L1

Commit message: Fixing connection issues
Connections:
- U1 pad 38: GND -> unconnected-(U1-GND-Pad38)
Routing:
- net GND: track 103.7 -> 134.1 mm
- net /MIDI/SW_D: track 74.2 -> 86.7 mm
- net /MIDI/SW_C: track 138.5 -> 151.0 mm
Changed lines of the file:
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@@
   (net 124 "/Audio/audio_in_L+")
   (net 125 "/Audio/GND_out")
+  (net 126 "unconnected-(U1-GND-Pad38)")
   (footprint "Capacitor_THT:C_Disc_D3.0mm_W1.6mm_P2.50mm" locked (layer "F.Cu")
     (at 147.055 48.04 90)
@@
       (net 46 "unconnected-(U1-3V3_EN-Pad37)") (pinfunction "3V3_EN") (pintype "input"))
     (pad "38" thru_hole rect locked (at 8.89 19.05 90) (size 1.7 1.7) (drill 1.02) (layers "*.Cu" "*.Mask")
-      (net 1 "GND") (pinfunction "GND") (pintype "bidirectional"))
+      (net 126 "unconnected-(U1-GND-Pad38)") (pinfunction "GND") (pintype "bidirectional"))
     (pad "38" smd rect locked (at 8.89 19.05 90) (size 3.5 1.7) (drill (offset 0.9 0)) (layers "B.Cu" "B.Mask")
-      (net 1 "GND") (pinfunction "GND") (pintype "bidirectional"))
+      (net 126 "unconnected-(U1-GND-Pad38)") (pinfunction "GND") (pintype "bidirectional"))
     (pad "39" thru_hole oval locked (at 8.89 21.59 90) (size 1.7 1.7) (drill 1.02) (layers "*.Cu" "*.Mask")
       (net 47 "unconnected-(U1-VSYS-Pad39)") (pinfunction "VSYS") (pintype "power_in"))
@@
   (segment (start 117.595 121.5) (end 117.655 121.44) (width 0.25) (layer "B.Cu") (net 1))
   (segment (start 117.655 115.34) (end 117.755 115.24) (width 0.25) (layer "B.Cu") (net 1))
+  (segment (start 171.075 124.175) (end 173.75 121.5) (width 0.25) (layer "B.Cu") (net 1))
   (segment (start 117.655 121.44) (end 117.655 115.34) (width 0.25) (layer "B.Cu") (net 1))
   (segment (start 157.555 122.905) (end 157.555 110.14) (width 0.25) (layer "B.Cu") (net 1))
   (segment (start 116.975 31.025) (end 116 32) (width 0.25) (layer "B.Cu") (net 1))
   (segment (start 77.4322 26.54) (end 75.855 26.54) (width 0.25) (layer "B.Cu") (net 1))
+  (segment (start 157.46 123) (end 158.635 124.175) (width 0.25) (layer "B.Cu") (net 1))
   (segment (start 157.46 123) (end 157.555 122.905) (width 0.25) (layer "B.Cu") (net 1))
   (segment (start 156.555 100.64) (end 151 100.64) (width 0.25) (layer "B.Cu") (net 1))
+  (segment (start 158.635 124.175) (end 171.075 124.175) (width 0.25) (layer "B.Cu") (net 1))
   (segment (start 157.555 110.14) (end 157.455 110.04) (width 0.25) (layer "B.Cu") (net 1))
   (segment (start 114.9172 23.4172) (end 80.555 23.4172) (width 0.25) (layer "B.Cu") (net 1))
@@
   (segment (start 111.25 121.5) (end 117.595 121.5) (width 0.25) (layer "B.Cu") (net 1))
   (segment (start 80.555 23.4172) (end 77.4322 26.54) (width 0.25) (layer "B.Cu") (net 1))
+  (segment (start 173.75 121.5) (end 186.25 121.5) (width 0.25) (layer "B.Cu") (net 1))
   (segment (start 116 24.5) (end 116.975 25.475) (width 0.25) (layer "B.Cu") (net 1))
   (segment (start 116.975 25.475) (end 116.975 31.025) (width 0.25) (layer "B.Cu") (net 1))
@@
   (segment (start 36.25 64.5) (end 39.06 61.69) (width 0.25) (layer "B.Cu") (net 92))
   (segment (start 104.62 61.69) (end 106.81 59.5) (width 0.25) (layer "B.Cu") (net 92))
+  (segment (start 36.25 64.5) (end 23.75 64.5) (width 0.25) (layer "B.Cu") (net 92))
   (segment (start 98.75 64.5) (end 111.25 64.5) (width 0.25) (layer "F.Cu") (net 93))
   (segment (start 111.25 64.5) (end 111.25 61.07) (width 0.25) (layer "F.Cu") (net 93))
@@
   (segment (start 115.055 63.055) (end 111.89 59.89) (width 0.25) (layer "B.Cu") (net 96))
   (segment (start 111.25 116.5) (end 115.055 116.5) (width 0.25) (layer "B.Cu") (net 96))
+  (segment (start 173.75 116.5) (end 186.25 116.5) (width 0.25) (layer "B.Cu") (net 97))
   (segment (start 134.655 39.94) (end 133.427792 39.94) (width 0.25) (layer "B.Cu") (net 97))
   (segment (start 173.75 116.5) (end 173.51 116.74) (width 0.25) (layer "B.Cu") (net 97))

Commit message: Refactor connection between pi an hifberry
Parts:
- moved C7 6.97 mm to (110.1, 80.4), turned to 90 degrees
Routing:
- net Net-(J7-5V-Pad2): track 72.0 -> 99.2 mm
- net Net-(J7-3V3-Pad1): track 70.4 -> 97.3 mm
- net Net-(J7-5V-Pad4): track 70.0 -> 96.3 mm
- net Net-(J7-SDA/GPIO2): track 68.9 -> 94.8 mm
- net Net-(J7-SCL/GPIO3): track 67.8 -> 91.3 mm
- net Net-(J7-GPIO14/TXD): track 67.5 -> 89.4 mm
- net Net-(J7-GCLK0/GPIO4): track 67.3 -> 87.9 mm
- net Net-(J7-GPIO15/RXD): track 67.3 -> 84.0 mm
- net Net-(J7-GPIO17): track 73.4 -> 82.6 mm
- net Net-(J7-GPIO18/PWM0): track 73.5 -> 81.1 mm
- net Net-(J7-GPIO27): track 72.4 -> 79.9 mm
- net Net-(J7-GPIO23): track 68.7 -> 75.3 mm
- net Net-(J7-GPIO22): track 69.9 -> 76.5 mm
- net Net-(J7-GPIO19/MISO1): track 80.6 -> 74.3 mm
- net Net-(J7-GPIO20/MOSI1): track 84.6 -> 78.4 mm
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
Commit message: Fixing connection issues
Routing:
- net GND: track 134.1 -> 147.2 mm, vias 0 -> 2
- net /Audio/GND_in_R: track 0.00 -> 4.54 mm, vias 0 -> 1
Changed lines of the file:
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@@
   (gr_arc (start 190 124) (mid 189.707107 124.707107) (end 189 125)
     (stroke (width 0.1) (type default)) (layer "Edge.Cuts"))
+  (segment (start 151.615 31.5) (end 149.75 31.5) (width 0.25) (layer "F.Cu") (net 1))
+  (segment (start 143.14 54.825) (end 143.155 54.84) (width 0.25) (layer "F.Cu") (net 1))
+  (segment (start 143.14 48) (end 143.14 54.825) (width 0.25) (layer "F.Cu") (net 1))
+  (segment (start 152.655 32.54) (end 151.615 31.5) (width 0.25) (layer "F.Cu") (net 1))
+  (segment (start 152.655 35.44) (end 152.655 32.54) (width 0.25) (layer "F.Cu") (net 1))
+  (via (at 152.655 35.74) (size 0.8) (drill 0.4) (layers "F.Cu" "B.Cu") (free) (net 1))
+  (via (at 143.155 54.84) (size 0.8) (drill 0.4) (layers "F.Cu" "B.Cu") (free) (net 1))
   (segment (start 157.455 101.54) (end 156.555 100.64) (width 0.25) (layer "B.Cu") (net 1))
   (segment (start 117.595 121.5) (end 117.655 121.44) (width 0.25) (layer "B.Cu") (net 1))
@@
   (segment (start 146.7798 123.473) (end 151.2248 119.028) (width 0.2) (layer "F.Cu") (net 119))
   (segment (start 181.6372 71.726) (end 178.5832 74.78) (width 0.2) (layer "F.Cu") (net 119))
+  (segment (start 54.8854 75.94) (end 57.655 75.94) (width 0.25) (layer "F.Cu") (net 120))
+  (segment (start 53.635 77.1904) (end 54.8854 75.94) (width 0.25) (layer "F.Cu") (net 120))
+  (via (at 105.055 122.54) (size 0.8) (drill 0.4) (layers "F.Cu" "B.Cu") (free) (net 120))
   (segment (start 48.858 74.2018) (end 48.858 101.1852) (width 0.2) (layer "F.Cu") (net 121))
   (segment (start 177.9468 74.78) (end 175.6 74.78) (width 0.2) (layer "F.Cu") (net 121))
@@
   (segment (start 56.175 77.1904) (end 54.8794 78.486) (width 0.25) (layer "F.Cu") (net 123))
   (segment (start 54.8794 78.486) (end 53.02 78.486) (width 0.25) (layer "F.Cu") (net 123))
-  (via (at 105.344 120.523) (size 0.8) (drill 0.4) (layers "F.Cu" "B.Cu") (free) (net 123))
-  (via (at 129.155 120.74) (size 0.8) (drill 0.4) (layers "F.Cu" "B.Cu") (free) (net 123))
+  (via (at 162.055 113.04) (size 0.8) (drill 0.4) (layers "F.Cu" "B.Cu") (free) (net 123))
+  (via (at 105.055 120.523) (size 0.8) (drill 0.4) (layers "F.Cu" "B.Cu") (free) (net 123))
   (via (at 175.956 102.108) (size 0.8) (drill 0.4) (layers "F.Cu" "B.Cu") (free) (net 123))
   (segment (start 188.3 94.995) (end 188.3 100.178) (width 0.25) (layer "B.Cu") (net 123))
@@
     (polygon
       (pts
-        (xy 54.415994 77.47)
-        (xy 52.131 77.343)
+        (xy 54.955 76.34)
+        (xy 54.955 77.94)
+        (xy 52.131 77.94)
         (xy 52.131 101.219)
         (xy 72.324 121.412)
@@
         (xy 50.226 69.977)
         (xy 56.195 69.977)
-        (xy 57.592 71.374)
-        (xy 57.592 74.93)
+        (xy 58.555 71.374)
+        (xy 58.65904 76.34)
       )
     )

Commit message: Fixing connection issues
Parts:
- moved C6 11.9 mm to (44.4, 71.5), turned to -90 degrees
- moved C9 1.16 mm to (44.2, 101.7), turned to 90 degrees
Routing:
- net +3.3V: track 0.00 -> 3.85 mm, vias 0 -> 1
- net Net-(D8-DOUT): track 80.2 -> 83.8 mm
- net Net-(D10-DIN): track 30.2 -> 29.6 mm
Changed lines of the file:
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@@
   )
   (footprint "Capacitor_THT:C_Disc_D3.0mm_W1.6mm_P2.50mm" (layer "F.Cu")
-    (at 43 101.7)
+    (at 44.155 101.7 90)
     (descr "C, Disc series, Radial, pin pitch=2.50mm, , diameter*width=3.0*1.6mm^2, Capacitor, http://www.vishay.com/docs/45233/krseries.pdf")
     (tags "C Disc series Radial pin pitch 2.50mm  diameter 3.0mm width 1.6mm Capacitor")
@@
     (property "ki_keywords" "cap capacitor")
     (attr through_hole)
-    (fp_text reference "C9" (at 4.6 0.15) (layer "F.SilkS")
+    (fp_text reference "C9" (at 4.6 0.15 90) (layer "F.SilkS")
         (effects (font (size 1 1) (thickness 0.15)))
     )
-    (fp_text value "100nF" (at 1.25 2.05) (layer "F.Fab")
+    (fp_text value "100nF" (at 1.25 2.05 90) (layer "F.Fab")
         (effects (font (size 1 1) (thickness 0.15)))
     )
-    (fp_text user "${REFERENCE}" (at 1.25 0) (layer "F.Fab")
+    (fp_text user "${REFERENCE}" (at 1.25 0 90) (layer "F.Fab")
         (effects (font (size 0.6 0.6) (thickness 0.09)))
     )
@@
     (fp_line (start 2.75 0.8) (end 2.75 -0.8)
       (stroke (width 0.1) (type solid)) (layer "F.Fab"))
-    (pad "1" thru_hole circle (at 0 0) (size 1.6 1.6) (drill 0.8) (layers "*.Cu" "*.Mask")
+    (pad "1" thru_hole circle (at 0 0 90) (size 1.6 1.6) (drill 0.8) (layers "*.Cu" "*.Mask")
       (net 2 "+3.3V") (pintype "passive"))
-    (pad "2" thru_hole circle (at 2.5 0) (size 1.6 1.6) (drill 0.8) (layers "*.Cu" "*.Mask")
+    (pad "2" thru_hole circle (at 2.5 0 90) (size 1.6 1.6) (drill 0.8) (layers "*.Cu" "*.Mask")
       (net 1 "GND") (pintype "passive"))
     (model "${KICAD6_3DMODEL_DIR}/Capacitor_THT.3dshapes/C_Disc_D3.0mm_W1.6mm_P2.50mm.wrl"
@@
       (solder_mask_margin 0.0508) (thermal_bridge_angle 45))
   )
-  (footprint "Capacitor_THT:C_Disc_D3.0mm_W1.6mm_P2.50mm" locked (layer "F.Cu")
-    (at 42.9 83.4)
+  (footprint "Capacitor_THT:C_Disc_D3.0mm_W1.6mm_P2.50mm" (layer "F.Cu")
+    (at 44.355 71.54 -90)
     (descr "C, Disc series, Radial, pin pitch=2.50mm, , diameter*width=3.0*1.6mm^2, Capacitor, http://www.vishay.com/docs/45233/krseries.pdf")
     (tags "C Disc series Radial pin pitch 2.50mm  diameter 3.0mm width 1.6mm Capacitor")
@@
     (property "ki_keywords" "cap capacitor")
     (attr through_hole)
-    (fp_text reference "C6" (at 4.6 0) (layer "F.SilkS")
+    (fp_text reference "C6" (at -2.6 0 90) (layer "F.SilkS")
         (effects (font (size 1 1) (thickness 0.15)))
     )
-    (fp_text value "100nF" (at 1.25 2.05) (layer "F.Fab")
+    (fp_text value "100nF" (at 1.25 2.05 90) (layer "F.Fab")
         (effects (font (size 1 1) (thickness 0.15)))
     )
-    (fp_text user "${REFERENCE}" (at 1.25 0) (layer "F.Fab")
+    (fp_text user "${REFERENCE}" (at 1.25 0 90) (layer "F.Fab")
         (effects (font (size 0.6 0.6) (thickness 0.09)))
     )
@@
     (fp_line (start 2.75 0.8) (end 2.75 -0.8)
       (stroke (width 0.1) (type solid)) (layer "F.Fab"))
-    (pad "1" thru_hole circle locked (at 0 0) (size 1.6 1.6) (drill 0.8) (layers "*.Cu" "*.Mask")
+    (pad "1" thru_hole circle (at 0 0 270) (size 1.6 1.6) (drill 0.8) (layers "*.Cu" "*.Mask")
       (net 2 "+3.3V") (pintype "passive"))
-    (pad "2" thru_hole circle locked (at 2.5 0) (size 1.6 1.6) (drill 0.8) (layers "*.Cu" "*.Mask")
+    (pad "2" thru_hole circle (at 2.5 0 270) (size 1.6 1.6) (drill 0.8) (layers "*.Cu" "*.Mask")
       (net 1 "GND") (pintype "passive"))
     (model "${KICAD6_3DMODEL_DIR}/Capacitor_THT.3dshapes/C_Disc_D3.0mm_W1.6mm_P2.50mm.wrl"
@@
   (segment (start 116 24.5) (end 116.975 25.475) (width 0.25) (layer "B.Cu") (net 1))
   (segment (start 116.975 25.475) (end 116.975 31.025) (width 0.25) (layer "B.Cu") (net 1))
+  (via (at 43.355 82.84) (size 0.8) (drill 0.4) (layers "F.Cu" "B.Cu") (free) (net 2))
+  (segment (start 43.37 79) (end 43.37 82.825) (width 0.25) (layer "B.Cu") (net 2))
+  (segment (start 43.37 82.825) (end 43.355 82.84) (width 0.25) (layer "B.Cu") (net 2))
   (segment (start 69.41 48) (end 69.585 47.825) (width 0.25) (layer "F.Cu") (net 3))
   (segment (start 90.425 47.825) (end 90.6 48) (width 0.25) (layer "F.Cu") (net 3))
@@
   (segment (start 103.1 79) (end 103.1 101.44) (width 0.25) (layer "B.Cu") (net 10))
   (segment (start 106.91 105.25) (end 106.91 106) (width 0.25) (layer "B.Cu") (net 10))
-  (segment (start 48.6 65.6) (end 42.1 72.1) (width 0.25) (layer "B.Cu") (net 11))
-  (segment (start 102.007139 73.732139) (end 97.432139 73.732139) (width 0.25) (layer "B.Cu") (net 11))
-  (segment (start 106.91 79) (end 106.91 78.635) (width 0.25) (layer "B.Cu") (net 11))
-  (segment (start 42.1 72.1) (end 42.1 79) (width 0.25) (layer "B.Cu") (net 11))
   (segment (start 97.432139 73.732139) (end 89.3 65.6) (width 0.25) (layer "B.Cu") (net 11))
-  (segment (start 89.3 65.6) (end 48.6 65.6) (width 0.25) (layer "B.Cu") (net 11))
+  (segment (start 42.395 65.6) (end 42.1 65.895) (width 0.25) (layer "B.Cu") (net 11))
+  (segment (start 42.1 65.895) (end 42.1 79) (width 0.25) (layer "B.Cu") (net 11))
+  (segment (start 89.3 65.6) (end 42.395 65.6) (width 0.25) (layer "B.Cu") (net 11))
   (segment (start 106.91 78.635) (end 102.007139 73.732139) (width 0.25) (layer "B.Cu") (net 11))
+  (segment (start 102.007139 73.732139) (end 97.432139 73.732139) (width 0.25) (layer "B.Cu") (net 11))
+  (segment (start 106.91 79) (end 106.91 78.635) (width 0.25) (layer "B.Cu") (net 11))
+  (segment (start 42.375 81.64) (end 41.775 82.24) (width 0.25) (layer "F.Cu") (net 12))
   (segment (start 41.775 105.675) (end 42.1 106) (width 0.25) (layer "F.Cu") (net 12))
-  (segment (start 45.91 79.365) (end 44.075 81.2) (width 0.25) (layer "F.Cu") (net 12))
-  (segment (start 44.075 81.2) (end 41.8 81.2) (width 0.25) (layer "F.Cu") (net 12))
-  (segment (start 41.8 81.2) (end 41.775 81.225) (width 0.25) (layer "F.Cu") (net 12))
+  (segment (start 45.91 79.365) (end 43.635 81.64) (width 0.25) (layer "F.Cu") (net 12))
+  (segment (start 41.775 82.24) (end 41.775 105.675) (width 0.25) (layer "F.Cu") (net 12))
   (segment (start 45.91 79) (end 45.91 79.365) (width 0.25) (layer "F.Cu") (net 12))
-  (segment (start 41.775 81.225) (end 41.775 105.675) (width 0.25) (layer "F.Cu") (net 12))
+  (segment (start 43.635 81.64) (end 42.375 81.64) (width 0.25) (layer "F.Cu") (net 12))
   (segment (start 45.91 106) (end 45.91 107.9) (width 0.25) (layer "B.Cu") (net 13))
   (segment (start 45.91 107.9) (end 51.285 113.275) (width 0.25) (layer "B.Cu") (net 13))

Commit message: Remove holes in pico footprint
Parts:
- moved C2 8.96 mm to (66.3, 43.4)
Changed lines of the file:
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@@
   )
   (footprint "Capacitor_THT:C_Disc_D3.0mm_W1.6mm_P2.50mm" locked (layer "F.Cu")
-    (at 66.25 52.4)
+    (at 66.305 43.44)
     (descr "C, Disc series, Radial, pin pitch=2.50mm, , diameter*width=3.0*1.6mm^2, Capacitor, http://www.vishay.com/docs/45233/krseries.pdf")
     (tags "C Disc series Radial pin pitch 2.50mm  diameter 3.0mm width 1.6mm Capacitor")
@@
     (fp_line (start -10.5 25.5) (end -10.5 25.2)
       (stroke (width 0.12) (type solid)) (layer "B.SilkS"))
-    (fp_line (start -10.5 25.5) (end 10.5 25.5)
-      (stroke (width 0.12) (type solid)) (layer "B.SilkS"))
     (fp_line (start -7.493 22.833) (end -7.493 25.5)
       (stroke (width 0.12) (type solid)) (layer "B.SilkS"))
@@
     (fp_line (start 10.5 25.5) (end 10.5 -25.5)
       (stroke (width 0.12) (type solid)) (layer "B.Fab"))
-    (pad "" np_thru_hole oval locked (at -2.725 24 90) (size 1.8 1.8) (drill 1.8) (layers "*.Cu" "*.Mask"))
-    (pad "" np_thru_hole oval locked (at -2.425 20.97 90) (size 1.5 1.5) (drill 1.5) (layers "*.Cu" "*.Mask"))
-    (pad "" np_thru_hole oval locked (at 2.425 20.97 90) (size 1.5 1.5) (drill 1.5) (layers "*.Cu" "*.Mask"))
-    (pad "" np_thru_hole oval locked (at 2.725 24 90) (size 1.8 1.8) (drill 1.8) (layers "*.Cu" "*.Mask"))
     (pad "1" thru_hole oval locked (at -8.89 24.13 90) (size 1.7 1.7) (drill 1.02) (layers "*.Cu" "*.Mask")
       (net 22 "Net-(U1-GPIO0)") (pinfunction "GPIO0") (pintype "bidirectional"))

Commit message: Improve GND layer
Routing:
- net Net-(U1-AGND): track 99.9 -> 101.5 mm
- net Net-(J15-Pin_1): track 107.9 -> 109.1 mm
- net Net-(J15-Pin_4): track 145.5 -> 146.3 mm
- net /Audio/GND_in_L: vias 3 -> 4

Commit message: Improve 3v3 layer
Parts:
- moved C1 1.40 mm to (72.0, 69.7)
Routing:
- net Net-(J15-Pin_3): track 101.1 -> 96.4 mm
- net Net-(U1-GPIO1): track 74.1 -> 75.8 mm
- net /MIDI/ROT_GAIN_A: track 63.4 -> 61.9 mm
- net Net-(U1-GPIO0): track 88.4 -> 87.0 mm
- net Net-(J15-Pin_2): track 82.1 -> 81.3 mm
- net /MIDI/SW_GAIN: track 76.8 -> 76.1 mm
- net Net-(J15-Pin_1): track 109.1 -> 109.7 mm
