File: audio.kicad_sch (KiCad schematic)
At the start: 8 parts, among them J10 NMJ6HCD2, J11 Audio OUT Right, J12 Audio OUT Left, J13 Audio IN, J14 Audio IN, J7 Raspberry_pi, J8 HiFi Berry, J9 Audio IN Right

Commit message: use sockets for HiFiBerry
Parts:
- J13, J14: footprint Connector_PinHeader_2.54mm:PinHeader_2x03_P2.54mm_Vertical -> Connector_PinSocket_2.54mm:PinSocket_2x03_P2.54mm_Vertical
- J8: footprint Connector_PinHeader_2.54mm:PinHeader_2x20_P2.54mm_Vertical -> Connector_PinSocket_2.54mm:PinSocket_2x20_P2.54mm_Vertical
Changed lines of the file:
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@@
       (effects (font (size 1.27 1.27)))
     )
-    (property "Footprint" "Connector_PinHeader_2.54mm:PinHeader_2x03_P2.54mm_Vertical" (at 92.71 154.94 0)
+    (property "Footprint" "Connector_PinSocket_2.54mm:PinSocket_2x03_P2.54mm_Vertical" (at 92.71 154.94 0)
       (effects (font (size 1.27 1.27)) hide)
     )
@@
       (effects (font (size 1.27 1.27)) (justify left))
     )
-    (property "Footprint" "Connector_PinHeader_2.54mm:PinHeader_2x20_P2.54mm_Vertical" (at 184.15 80.01 0)
+    (property "Footprint" "Connector_PinSocket_2.54mm:PinSocket_2x20_P2.54mm_Vertical" (at 184.15 80.01 0)
       (effects (font (size 1.27 1.27)) hide)
     )
@@
       (effects (font (size 1.27 1.27)))
     )
-    (property "Footprint" "Connector_PinHeader_2.54mm:PinHeader_2x03_P2.54mm_Vertical" (at 67.31 154.94 0)
-      (effects (font (size 1.27 1.27)) hide)
-    )
+    (property "Footprint" "Connector_PinSocket_2.54mm:PinSocket_2x03_P2.54mm_Vertical" (at 67.31 154.94 0)
+      (effects (font (size 1.27 1.27)) hide)
+    )

Commit message: Fix Audio Connectors
Parts:
- J10: value NMJ6HCD2 -> Audio IN Left
- J13: value Audio IN -> Audio OUT
Changed lines of the file:
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@@
       (effects (font (size 1.27 1.27)) (justify left))
     )
-    (property "Value" "NMJ6HCD2" (at 44.45 166.37 90)
+    (property "Value" "Audio IN Left" (at 44.45 166.37 90)
       (effects (font (size 1.27 1.27)) (justify left))
     )
@@
       (effects (font (size 1.27 1.27)))
     )
-    (property "Value" "Audio IN" (at 93.98 149.86 0)
+    (property "Value" "Audio OUT" (at 93.98 149.86 0)
       (effects (font (size 1.27 1.27)))
     )

Commit message: Connect the USB between the processors
Parts:
- added J6: USB_A, Connector_PinHeader_2.54mm:PinHeader_1x04_P2.54mm_Vertical, symbol Connector:USB_A
Connections:
- new net USB_DM: J6.2 (D-)
- new net USB_DP: J6.3 (D+)
- new net USB_GND: J6.4 (GND), J6.5 (Shield)
- new net V_BUS: J6.1 (VBUS)
Changed lines of the file:
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@@
   (junction (at 186.69 118.11) (diameter 0) (color 0 0 0 0)
   )
+  (junction (at 259.08 93.98) (diameter 0) (color 0 0 0 0)
+  )
   (junction (at 184.15 118.11) (diameter 0) (color 0 0 0 0)
   )
@@
     (stroke (width 0) (type default))
   )
+  (wire (pts (xy 259.08 101.6) (xy 262.89 101.6))
+    (stroke (width 0) (type default))
+  )
   (wire (pts (xy 120.65 113.03) (xy 120.65 120.65))
     (stroke (width 0) (type default))
@@
     (stroke (width 0) (type default))
   )
+  (wire (pts (xy 267.97 80.01) (xy 273.05 80.01))
+    (stroke (width 0) (type default))
+  )
   (wire (pts (xy 87.63 17.78) (xy 223.52 17.78))
     (stroke (width 0) (type default))
@@
     (stroke (width 0) (type default))
   )
+  (wire (pts (xy 259.08 93.98) (xy 259.08 101.6))
+    (stroke (width 0) (type default))
+  )
   (wire (pts (xy 219.71 21.59) (xy 219.71 87.63))
     (stroke (width 0) (type default))
@@
     (stroke (width 0) (type default))
   )
+  (wire (pts (xy 267.97 74.93) (xy 274.32 74.93))
+    (stroke (width 0) (type default))
+  )
+  (wire (pts (xy 259.08 93.98) (xy 257.81 93.98))
+    (stroke (width 0) (type default))
+  )
   (wire (pts (xy 92.71 22.86) (xy 218.44 22.86))
     (stroke (width 0) (type default))
@@
     (stroke (width 0) (type default))
   )
+  (wire (pts (xy 257.81 90.17) (xy 257.81 93.98))
+    (stroke (width 0) (type default))
+  )
   (wire (pts (xy 100.33 157.48) (xy 105.41 157.48))
     (stroke (width 0) (type default))
@@
     (stroke (width 0) (type default))
   )
+  (wire (pts (xy 260.35 90.17) (xy 260.35 93.98))
+    (stroke (width 0) (type default))
+  )
   (wire (pts (xy 105.41 97.79) (xy 86.36 97.79))
     (stroke (width 0) (type default))
@@
     (stroke (width 0) (type default))
   )
+  (wire (pts (xy 260.35 93.98) (xy 259.08 93.98))
+    (stroke (width 0) (type default))
+  )
   (wire (pts (xy 31.75 176.53) (xy 31.75 171.45))
     (stroke (width 0) (type default))
@@
     (stroke (width 0) (type default))
   )
+  (wire (pts (xy 267.97 82.55) (xy 273.05 82.55))
+    (stroke (width 0) (type default))
+  )
   (wire (pts (xy 146.05 92.71) (xy 163.83 92.71))
     (stroke (width 0) (type default))
@@
   (wire (pts (xy 217.17 80.01) (xy 204.47 80.01))
     (stroke (width 0) (type default))
+  )
+  (hierarchical_label "USB_DP" (shape input) (at 273.05 80.01 0) (fields_autoplaced)
+    (effects (font (size 1.27 1.27)) (justify left))
+  )
+  (hierarchical_label "V_BUS" (shape input) (at 274.32 74.93 0) (fields_autoplaced)
+    (effects (font (size 1.27 1.27)) (justify left))
+  )
+  (hierarchical_label "USB_DM" (shape input) (at 273.05 82.55 0) (fields_autoplaced)
+    (effects (font (size 1.27 1.27)) (justify left))
+  )
+  (hierarchical_label "USB_GND" (shape input) (at 262.89 101.6 0) (fields_autoplaced)
+    (effects (font (size 1.27 1.27)) (justify left))
   )
   (symbol (lib_id "Connector_Audio:NMJ6HCD2") (at 36.83 166.37 270) (unit 1)
@@
         )
       )
+    )
+  )
+  (symbol (lib_id "Connector:USB_A") (at 260.35 80.01 0) (unit 1)
+    (in_bom yes) (on_board yes) (dnp no) (fields_autoplaced)
+    (property "Reference" "J6" (at 260.35 68.58 0)
+      (effects (font (size 1.27 1.27)))
+    )
+    (property "Value" "USB_A" (at 260.35 71.12 0)
+      (effects (font (size 1.27 1.27)))
+    )
+    (property "Footprint" "Connector_PinHeader_2.54mm:PinHeader_1x04_P2.54mm_Vertical" (at 264.16 81.28 0)
+      (effects (font (size 1.27 1.27)) hide)
+    )
+    (property "Datasheet" " ~" (at 264.16 81.28 0)
+      (effects (font (size 1.27 1.27)) hide)
+    )
+    (pin "1")
+    (pin "2")
+    (pin "3")
+    (pin "4")
+    (pin "5")
+    (instances
+      (project "pedalboard-hw"
+        (path "/df521c2a-9827-4355-b809-366f4b88d5d7/6bd0afd4-cd8b-4c1d-a236-891eed0b2d91"
+          (reference "J6") (unit 1)
+        )
+      )

Commit message: Name the input networks for better routing
Connections:
- net GNDA: now reaches J10.S, J14.4 (Pin_4)
- net GNDA: now also J14.3 (Pin_3), J9.S
- net audio out L+: now reaches J10.T, J14.5 (Pin_5)
- net audio out R-: now reaches J14.1 (Pin_1), J9.R
Changed lines of the file:
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@@
-    (stroke (width 0) (type default))
-  )
-  (wire (pts (xy 62.23 154.94) (xy 41.91 154.94))
     (stroke (width 0) (type default))
   )
@@
     (stroke (width 0) (type default))
   )
-  (wire (pts (xy 62.23 157.48) (xy 22.86 157.48))
-    (stroke (width 0) (type default))
-  )
   (wire (pts (xy 22.86 176.53) (xy 31.75 176.53))
     (stroke (width 0) (type default))
@@
     (stroke (width 0) (type default))
   )
-  (wire (pts (xy 62.23 152.4) (xy 36.83 152.4))
-    (stroke (width 0) (type default))
-  )
   (wire (pts (xy 93.98 80.01) (xy 93.98 24.13))
     (stroke (width 0) (type default))
@@
     (stroke (width 0) (type default))
   )
-  (wire (pts (xy 81.28 184.15) (xy 41.91 184.15))
-    (stroke (width 0) (type default))
-  )
   (wire (pts (xy 176.53 118.11) (xy 176.53 127))
     (stroke (width 0) (type default))
@@
     (stroke (width 0) (type default))
   )
-  (wire (pts (xy 81.28 154.94) (xy 81.28 184.15))
-    (stroke (width 0) (type default))
-  )
   (wire (pts (xy 120.65 120.65) (xy 118.11 120.65))
     (stroke (width 0) (type default))
@@
     (stroke (width 0) (type default))
   )
+  (wire (pts (xy 41.91 144.78) (xy 41.91 147.32))
+    (stroke (width 0) (type default))
+  )
   (wire (pts (xy 36.83 179.07) (xy 36.83 171.45))
     (stroke (width 0) (type default))
@@
     (stroke (width 0) (type default))
   )
-  (wire (pts (xy 41.91 184.15) (xy 41.91 171.45))
-    (stroke (width 0) (type default))
-  )
   (wire (pts (xy 189.23 118.11) (xy 186.69 118.11))
     (stroke (width 0) (type default))
@@
     (stroke (width 0) (type default))
   )
+  (wire (pts (xy 57.15 154.94) (xy 62.23 154.94))
+    (stroke (width 0) (type default))
+  )
   (wire (pts (xy 115.57 113.03) (xy 115.57 120.65))
     (stroke (width 0) (type default))
@@
     (stroke (width 0) (type default))
   )
-  (wire (pts (xy 41.91 154.94) (xy 41.91 144.78))
+  (wire (pts (xy 74.93 154.94) (xy 81.28 154.94))
     (stroke (width 0) (type default))
   )
@@
     (stroke (width 0) (type default))
   )
+  (wire (pts (xy 22.86 157.48) (xy 62.23 157.48))
+    (stroke (width 0) (type default))
+  )
   (wire (pts (xy 208.28 57.15) (xy 204.47 57.15))
     (stroke (width 0) (type default))
@@
     (stroke (width 0) (type default))
   )
+  (wire (pts (xy 41.91 171.45) (xy 41.91 172.72))
+    (stroke (width 0) (type default))
+  )
   (wire (pts (xy 99.06 29.21) (xy 212.09 29.21))
     (stroke (width 0) (type default))
@@
     (stroke (width 0) (type default))
   )
+  (wire (pts (xy 36.83 152.4) (xy 62.23 152.4))
+    (stroke (width 0) (type default))
+  )
   (wire (pts (xy 105.41 77.47) (xy 95.25 77.47))
     (stroke (width 0) (type default))
@@
     (stroke (width 0) (type default))
   )
-  (wire (pts (xy 74.93 154.94) (xy 81.28 154.94))
-    (stroke (width 0) (type default))
-  )
   (wire (pts (xy 118.11 113.03) (xy 118.11 120.65))
     (stroke (width 0) (type default))
@@
   (wire (pts (xy 217.17 80.01) (xy 204.47 80.01))
     (stroke (width 0) (type default))
+  )
+  (label "audio out L+" (at 39.37 157.48 0) (fields_autoplaced)
+    (effects (font (size 1.27 1.27)) (justify left bottom))
+  )
+  (label "audio out R-" (at 39.37 152.4 0) (fields_autoplaced)
+    (effects (font (size 1.27 1.27)) (justify left bottom))
+  )
+  (label "audio out L-" (at 77.47 171.45 90) (fields_autoplaced)
+    (effects (font (size 1.27 1.27)) (justify left bottom))
+  )
+  (label "audio out R+" (at 77.47 147.32 90) (fields_autoplaced)
+    (effects (font (size 1.27 1.27)) (justify left bottom))
   )
   (hierarchical_label "USB_DP" (shape input) (at 273.05 80.01 0) (fields_autoplaced)
@@
     )
   )
+  (symbol (lib_id "power:GNDA") (at 41.91 147.32 0) (unit 1)
+    (in_bom yes) (on_board yes) (dnp no)
+    (property "Reference" "#PWR031" (at 41.91 153.67 0)
+      (effects (font (size 1.27 1.27)) hide)
+    )
+    (property "Value" "GNDA" (at 44.45 147.32 0)
+      (effects (font (size 1.27 1.27)))
+    )
+    (property "Footprint" "" (at 41.91 147.32 0)
+      (effects (font (size 1.27 1.27)) hide)
+    )
+    (property "Datasheet" "" (at 41.91 147.32 0)
+      (effects (font (size 1.27 1.27)) hide)
+    )
+    (pin "1")
+    (instances
+      (project "pedalboard-hw"
+        (path "/df521c2a-9827-4355-b809-366f4b88d5d7/6bd0afd4-cd8b-4c1d-a236-891eed0b2d91"
+          (reference "#PWR031") (unit 1)
+        )
+      )
+    )
+  )
   (symbol (lib_id "Connector_Audio:NMJ6HCD2") (at 36.83 139.7 270) (unit 1)
     (in_bom yes) (on_board yes) (dnp no) (fields_autoplaced)
@@
         (path "/df521c2a-9827-4355-b809-366f4b88d5d7/6bd0afd4-cd8b-4c1d-a236-891eed0b2d91"
           (reference "J9") (unit 1)
+        )
+      )
+    )
+  )
+  (symbol (lib_id "power:GNDA") (at 57.15 154.94 0) (unit 1)
+    (in_bom yes) (on_board yes) (dnp no)
+    (property "Reference" "#PWR030" (at 57.15 161.29 0)
+      (effects (font (size 1.27 1.27)) hide)
+    )
+    (property "Value" "GNDA" (at 54.61 154.94 0)
+      (effects (font (size 1.27 1.27)))
+    )
+    (property "Footprint" "" (at 57.15 154.94 0)
+      (effects (font (size 1.27 1.27)) hide)
+    )
+    (property "Datasheet" "" (at 57.15 154.94 0)
+      (effects (font (size 1.27 1.27)) hide)
+    )
+    (pin "1")
+    (instances
+      (project "pedalboard-hw"
+        (path "/df521c2a-9827-4355-b809-366f4b88d5d7/6bd0afd4-cd8b-4c1d-a236-891eed0b2d91"
+          (reference "#PWR030") (unit 1)
         )
       )
@@
         )
       )
+    )
+  )
+  (symbol (lib_id "power:GNDA") (at 41.91 172.72 0) (unit 1)
+    (in_bom yes) (on_board yes) (dnp no)
+    (property "Reference" "#PWR032" (at 41.91 179.07 0)
+      (effects (font (size 1.27 1.27)) hide)
+    )
+    (property "Value" "GNDA" (at 44.45 172.72 0)
+      (effects (font (size 1.27 1.27)))
+    )
+    (property "Footprint" "" (at 41.91 172.72 0)
+      (effects (font (size 1.27 1.27)) hide)
+    )
+    (property "Datasheet" "" (at 41.91 172.72 0)
+      (effects (font (size 1.27 1.27)) hide)
+    )
+    (pin "1")
+    (instances
+      (project "pedalboard-hw"
+        (path "/df521c2a-9827-4355-b809-366f4b88d5d7/6bd0afd4-cd8b-4c1d-a236-891eed0b2d91"
+          (reference "#PWR032") (unit 1)
+        )
+      )
+    )
+  )
+  (symbol (lib_id "power:GNDA") (at 81.28 154.94 0) (unit 1)
+    (in_bom yes) (on_board yes) (dnp no)
+    (property "Reference" "#PWR029" (at 81.28 161.29 0)
+      (effects (font (size 1.27 1.27)) hide)
+    )
+    (property "Value" "GNDA" (at 82.55 153.67 0)
+      (effects (font (size 1.27 1.27)))
+    )
+    (property "Footprint" "" (at 81.28 154.94 0)
+      (effects (font (size 1.27 1.27)) hide)
+    )
+    (property "Datasheet" "" (at 81.28 154.94 0)
+      (effects (font (size 1.27 1.27)) hide)
+    )
+    (pin "1")
+    (instances
+      (project "pedalboard-hw"
+        (path "/df521c2a-9827-4355-b809-366f4b88d5d7/6bd0afd4-cd8b-4c1d-a236-891eed0b2d91"
+          (reference "#PWR029") (unit 1)
+        )
+      )

Commit message: try to label again audio in
Connections:
- net audio_out_L-: now reaches J10.R, J14.6 (Pin_6)
- net audio_out_R+: now reaches J14.2 (Pin_2), J9.T
- net audio out L+ renamed audio_out_L+
- net audio out R- renamed audio_out_R-
Changed lines of the file:
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@@
     (stroke (width 0) (type default))
   )
-  (label "audio out L+" (at 39.37 157.48 0) (fields_autoplaced)
+  (label "audio_out_L+" (at 39.37 157.48 0) (fields_autoplaced)
     (effects (font (size 1.27 1.27)) (justify left bottom))
   )
-  (label "audio out R-" (at 39.37 152.4 0) (fields_autoplaced)
+  (label "audio_out_R-" (at 39.37 152.4 0) (fields_autoplaced)
     (effects (font (size 1.27 1.27)) (justify left bottom))
   )
-  (label "audio out L-" (at 77.47 171.45 90) (fields_autoplaced)
+  (label "audio_out_L-" (at 52.07 179.07 0) (fields_autoplaced)
     (effects (font (size 1.27 1.27)) (justify left bottom))
   )
-  (label "audio out R+" (at 77.47 147.32 90) (fields_autoplaced)
+  (label "audio_out_R+" (at 58.42 125.73 0) (fields_autoplaced)
     (effects (font (size 1.27 1.27)) (justify left bottom))
   )

Commit message: Analog Out GND Panes
Connections:
- net GNDA renamed GND_analog_out_L
- net GND_analog_out_L: no longer J14.3 (Pin_3), J9.S
- new net GND_analog_out_R: J14.3 (Pin_3), J9.S
Changed lines of the file:
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@@
+    (stroke (width 0) (type default))
+  )
+  (wire (pts (xy 41.91 172.72) (xy 77.47 172.72))
     (stroke (width 0) (type default))
   )
@@
     (stroke (width 0) (type default))
   )
-  (wire (pts (xy 41.91 144.78) (xy 41.91 147.32))
+  (wire (pts (xy 41.91 144.78) (xy 41.91 154.94))
     (stroke (width 0) (type default))
   )
@@
     (stroke (width 0) (type default))
   )
+  (wire (pts (xy 77.47 154.94) (xy 74.93 154.94))
+    (stroke (width 0) (type default))
+  )
+  (wire (pts (xy 77.47 172.72) (xy 77.47 154.94))
+    (stroke (width 0) (type default))
+  )
   (wire (pts (xy 109.22 154.94) (xy 127 154.94))
     (stroke (width 0) (type default))
@@
     (stroke (width 0) (type default))
   )
+  (wire (pts (xy 41.91 154.94) (xy 62.23 154.94))
+    (stroke (width 0) (type default))
+  )
   (wire (pts (xy 90.17 20.32) (xy 90.17 90.17))
     (stroke (width 0) (type default))
@@
     (stroke (width 0) (type default))
   )
-  (wire (pts (xy 57.15 154.94) (xy 62.23 154.94))
-    (stroke (width 0) (type default))
-  )
   (wire (pts (xy 115.57 113.03) (xy 115.57 120.65))
     (stroke (width 0) (type default))
   )
   (wire (pts (xy 210.82 30.48) (xy 210.82 64.77))
-    (stroke (width 0) (type default))
-  )
-  (wire (pts (xy 74.93 154.94) (xy 81.28 154.94))
     (stroke (width 0) (type default))
   )
@@
   )
   (label "audio_out_R+" (at 58.42 125.73 0) (fields_autoplaced)
+    (effects (font (size 1.27 1.27)) (justify left bottom))
+  )
+  (label "GND_analog_out_L" (at 54.61 172.72 0) (fields_autoplaced)
+    (effects (font (size 1.27 1.27)) (justify left bottom))
+  )
+  (label "GND_analog_out_R" (at 45.72 154.94 0) (fields_autoplaced)
     (effects (font (size 1.27 1.27)) (justify left bottom))
   )
@@
     )
   )
-  (symbol (lib_id "power:GNDA") (at 41.91 147.32 0) (unit 1)
-    (in_bom yes) (on_board yes) (dnp no)
-    (property "Reference" "#PWR031" (at 41.91 153.67 0)
-      (effects (font (size 1.27 1.27)) hide)
-    )
-    (property "Value" "GNDA" (at 44.45 147.32 0)
-      (effects (font (size 1.27 1.27)))
-    )
-    (property "Footprint" "" (at 41.91 147.32 0)
-      (effects (font (size 1.27 1.27)) hide)
-    )
-    (property "Datasheet" "" (at 41.91 147.32 0)
-      (effects (font (size 1.27 1.27)) hide)
-    )
-    (pin "1")
-    (instances
-      (project "pedalboard-hw"
-        (path "/df521c2a-9827-4355-b809-366f4b88d5d7/6bd0afd4-cd8b-4c1d-a236-891eed0b2d91"
-          (reference "#PWR031") (unit 1)
-        )
-      )
-    )
-  )
   (symbol (lib_id "Connector_Audio:NMJ6HCD2") (at 36.83 139.7 270) (unit 1)
     (in_bom yes) (on_board yes) (dnp no) (fields_autoplaced)
@@
         (path "/df521c2a-9827-4355-b809-366f4b88d5d7/6bd0afd4-cd8b-4c1d-a236-891eed0b2d91"
           (reference "J9") (unit 1)
-        )
-      )
-    )
-  )
-  (symbol (lib_id "power:GNDA") (at 57.15 154.94 0) (unit 1)
-    (in_bom yes) (on_board yes) (dnp no)
-    (property "Reference" "#PWR030" (at 57.15 161.29 0)
-      (effects (font (size 1.27 1.27)) hide)
-    )
-    (property "Value" "GNDA" (at 54.61 154.94 0)
-      (effects (font (size 1.27 1.27)))
-    )
-    (property "Footprint" "" (at 57.15 154.94 0)
-      (effects (font (size 1.27 1.27)) hide)
-    )
-    (property "Datasheet" "" (at 57.15 154.94 0)
-      (effects (font (size 1.27 1.27)) hide)
-    )
-    (pin "1")
-    (instances
-      (project "pedalboard-hw"
-        (path "/df521c2a-9827-4355-b809-366f4b88d5d7/6bd0afd4-cd8b-4c1d-a236-891eed0b2d91"
-          (reference "#PWR030") (unit 1)
         )
       )
@@
         )
       )
-    )
-  )
-  (symbol (lib_id "power:GNDA") (at 41.91 172.72 0) (unit 1)
-    (in_bom yes) (on_board yes) (dnp no)
-    (property "Reference" "#PWR032" (at 41.91 179.07 0)
-      (effects (font (size 1.27 1.27)) hide)
-    )
-    (property "Value" "GNDA" (at 44.45 172.72 0)
-      (effects (font (size 1.27 1.27)))
-    )
-    (property "Footprint" "" (at 41.91 172.72 0)
-      (effects (font (size 1.27 1.27)) hide)
-    )
-    (property "Datasheet" "" (at 41.91 172.72 0)
-      (effects (font (size 1.27 1.27)) hide)
-    )
-    (pin "1")
-    (instances
-      (project "pedalboard-hw"
-        (path "/df521c2a-9827-4355-b809-366f4b88d5d7/6bd0afd4-cd8b-4c1d-a236-891eed0b2d91"
-          (reference "#PWR032") (unit 1)
-        )
-      )
-    )
-  )
-  (symbol (lib_id "power:GNDA") (at 81.28 154.94 0) (unit 1)
-    (in_bom yes) (on_board yes) (dnp no)
-    (property "Reference" "#PWR029" (at 81.28 161.29 0)
-      (effects (font (size 1.27 1.27)) hide)
-    )
-    (property "Value" "GNDA" (at 82.55 153.67 0)
-      (effects (font (size 1.27 1.27)))
-    )
-    (property "Footprint" "" (at 81.28 154.94 0)
-      (effects (font (size 1.27 1.27)) hide)
-    )
-    (property "Datasheet" "" (at 81.28 154.94 0)
-      (effects (font (size 1.27 1.27)) hide)
-    )
-    (pin "1")
-    (instances
-      (project "pedalboard-hw"
-        (path "/df521c2a-9827-4355-b809-366f4b88d5d7/6bd0afd4-cd8b-4c1d-a236-891eed0b2d91"
-          (reference "#PWR029") (unit 1)
-        )
-      )

Commit message: Analog Out GND Panes
Connections:
- net GND_out: now reaches J11.S, J12.S, J13.4 (Pin_4)
- net GND_analog_out_L renamed GND_in_L
- net GND_analog_out_R renamed GND_in_R
- net audio_out_L+ renamed audio_in_L+
- net audio_out_L- renamed in_L-
- net audio_out_R+ renamed in_R+
- net audio_out_R- renamed in_R-
Changed lines of the file:
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@@
     (stroke (width 0) (type default))
   )
-  (label "audio_out_L+" (at 39.37 157.48 0) (fields_autoplaced)
+  (label "audio_in_L+" (at 39.37 157.48 0) (fields_autoplaced)
     (effects (font (size 1.27 1.27)) (justify left bottom))
   )
-  (label "audio_out_R-" (at 39.37 152.4 0) (fields_autoplaced)
+  (label "in_R-" (at 39.37 152.4 0) (fields_autoplaced)
     (effects (font (size 1.27 1.27)) (justify left bottom))
   )
-  (label "audio_out_L-" (at 52.07 179.07 0) (fields_autoplaced)
+  (label "in_L-" (at 52.07 179.07 0) (fields_autoplaced)
     (effects (font (size 1.27 1.27)) (justify left bottom))
   )
-  (label "audio_out_R+" (at 58.42 125.73 0) (fields_autoplaced)
+  (label "in_R+" (at 58.42 125.73 0) (fields_autoplaced)
     (effects (font (size 1.27 1.27)) (justify left bottom))
   )
-  (label "GND_analog_out_L" (at 54.61 172.72 0) (fields_autoplaced)
+  (label "GND_out" (at 110.49 181.61 0) (fields_autoplaced)
     (effects (font (size 1.27 1.27)) (justify left bottom))
   )
-  (label "GND_analog_out_R" (at 45.72 154.94 0) (fields_autoplaced)
+  (label "GND_in_L" (at 54.61 172.72 0) (fields_autoplaced)
     (effects (font (size 1.27 1.27)) (justify left bottom))
   )
+  (label "GND_in_R" (at 45.72 154.94 0) (fields_autoplaced)
+    (effects (font (size 1.27 1.27)) (justify left bottom))
+  )

Commit message: Connect USB
Connections:
- net USB_DM renamed USB_DN
Changed lines of the file:
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@@
     (effects (font (size 1.27 1.27)) (justify left))
   )
-  (hierarchical_label "USB_DM" (shape input) (at 273.05 82.55 0) (fields_autoplaced)
+  (hierarchical_label "USB_DN" (shape input) (at 273.05 82.55 0) (fields_autoplaced)
     (effects (font (size 1.27 1.27)) (justify left))
   )
