File: audio.kicad_sch (KiCad schematic)
At the start: 9 parts, among them J10 Audio IN Left, J11 Audio OUT Right, J12 Audio OUT Left, J13 Audio OUT, J14 Audio IN, J6 USB_A, J7 Raspberry_pi, J8 HiFi Berry, J9 Audio IN Right

Commit message: Put HifiBerry into project library
Parts:
- J8: footprint Connector_PinSocket_2.54mm:PinSocket_2x20_P2.54mm_Vertical -> Pedalboard Library:HiFi Berry DAC ADC+
Changed lines of the file:
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@@
       (effects (font (size 1.27 1.27)) (justify left))
     )
-    (property "Footprint" "Connector_PinSocket_2.54mm:PinSocket_2x20_P2.54mm_Vertical" (at 184.15 80.01 0)
+    (property "Footprint" "Pedalboard Library:HiFi Berry DAC ADC+" (at 184.15 80.01 0)
       (effects (font (size 1.27 1.27)) hide)
     )

Commit message: Put RPI nano into project library
Parts:
- J7: footprint Connector_PinHeader_2.54mm:PinHeader_2x20_P2.54mm_Vertical -> Pedalboard Library:Raspberry PI Compute Module CM4 Nano A
Changed lines of the file:
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@@
       (effects (font (size 1.27 1.27)) (justify left))
     )
-    (property "Footprint" "Connector_PinHeader_2.54mm:PinHeader_2x20_P2.54mm_Vertical" (at 125.73 80.01 0)
+    (property "Footprint" "Pedalboard Library:Raspberry PI Compute Module CM4 Nano A" (at 125.73 80.01 0)
       (effects (font (size 1.27 1.27)) hide)
     )

Commit message: Put USB A Plut into project library
Parts:
- J6: footprint Connector_PinHeader_2.54mm:PinHeader_1x04_P2.54mm_Vertical -> Pedalboard Library:USB A BCB Male Plug
Changed lines of the file:
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@@
       (effects (font (size 1.27 1.27)))
     )
-    (property "Footprint" "Connector_PinHeader_2.54mm:PinHeader_1x04_P2.54mm_Vertical" (at 264.16 81.28 0)
+    (property "Footprint" "Pedalboard Library:USB A BCB Male Plug" (at 264.16 81.28 0)
       (effects (font (size 1.27 1.27)) hide)
     )

Commit message: Add links to digikey
Parts:
- J10, J11, J12, J9: Supplier (none) -> https://www.digikey.ch/de/products/detail/schurter-inc/4833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
- J13, J14, J7, J8: Supplier (none) -> https://www.digikey.ch/de/products/detail/w%C3%BCrth-elektr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
- J6: Supplier (none) -> https://www.digikey.ch/de/products/detail/gct/USB1061-GF-L-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
Changed lines of the file:
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@@
       (effects (font (size 1.27 1.27)) hide)
     )
-    (property "Datasheet" "https://www.neutrik.com/en/product/nmj6hcd2" (at 36.83 166.37 0)
+    (property "Datasheet" "https://us.schurter.com/bundles/snceschurter/epim/_ProdPool_/newDS/en/typ_4833.2330.pdf" (at 36.83 166.37 0)
+      (effects (font (size 1.27 1.27)) hide)
+    )
+    (property "Supplier" "https://www.digikey.ch/de/products/detail/schurter-inc/4833-2330/9451854" (at 36.83 166.37 0)
       (effects (font (size 1.27 1.27)) hide)
     )
@@
       (effects (font (size 1.27 1.27)) hide)
     )
-    (property "Datasheet" "~" (at 92.71 154.94 0)
+    (property "Datasheet" "https://www.we-online.com/components/products/datasheet/61300621821.pdf" (at 92.71 154.94 0)
+      (effects (font (size 1.27 1.27)) hide)
+    )
+    (property "Supplier" "https://www.digikey.ch/de/products/detail/w%C3%BCrth-elektronik/61300621821/16608633" (at 92.71 154.94 0)
       (effects (font (size 1.27 1.27)) hide)
     )
@@
       (effects (font (size 1.27 1.27)) hide)
     )
-    (property "Datasheet" "https://www.raspberrypi.org/documentation/hardware/raspberrypi/schematics/rpi_SCH_3bplus_1p0_reduced.pdf" (at 125.73 80.01 0)
+    (property "Datasheet" "https://www.waveshare.com/wiki/CM4-NANO-A" (at 125.73 80.01 0)
+      (effects (font (size 1.27 1.27)) hide)
+    )
+    (property "Supplier" "https://www.digikey.ch/de/products/detail/w%C3%BCrth-elektronik/61304021121/4846886" (at 125.73 80.01 0)
       (effects (font (size 1.27 1.27)) hide)
     )
@@
       (effects (font (size 1.27 1.27)) hide)
     )
-    (property "Datasheet" "https://www.neutrik.com/en/product/nmj6hcd2" (at 36.83 139.7 0)
+    (property "Datasheet" "https://us.schurter.com/bundles/snceschurter/epim/_ProdPool_/newDS/en/typ_4833.2330.pdf" (at 36.83 139.7 0)
+      (effects (font (size 1.27 1.27)) hide)
+    )
+    (property "Supplier" "https://www.digikey.ch/de/products/detail/schurter-inc/4833-2330/9451854" (at 36.83 139.7 0)
       (effects (font (size 1.27 1.27)) hide)
     )
@@
     )
     (property "Datasheet" "https://www.hifiberry.com/docs/data-sheets/datasheet-dac-adc-pro/" (at 184.15 80.01 0)
+      (effects (font (size 1.27 1.27)) hide)
+    )
+    (property "Supplier" "https://www.digikey.ch/de/products/detail/w%C3%BCrth-elektronik/61302021821/16608495" (at 184.15 80.01 0)
       (effects (font (size 1.27 1.27)) hide)
     )
@@
       (effects (font (size 1.27 1.27)) hide)
     )
-    (property "Datasheet" " ~" (at 264.16 81.28 0)
+    (property "Datasheet" "https://media.digikey.com/pdf/Data%20Sheets/GCT%20PDFs/USB1061_Spec.pdf" (at 264.16 81.28 0)
+      (effects (font (size 1.27 1.27)) hide)
+    )
+    (property "Supplier" "https://www.digikey.ch/de/products/detail/gct/USB1061-GF-L-A/10649776" (at 260.35 80.01 0)
       (effects (font (size 1.27 1.27)) hide)
     )
@@
       (effects (font (size 1.27 1.27)) hide)
     )
-    (property "Datasheet" "~" (at 67.31 154.94 0)
+    (property "Datasheet" "https://www.we-online.com/components/products/datasheet/61300621821.pdf" (at 67.31 154.94 0)
+      (effects (font (size 1.27 1.27)) hide)
+    )
+    (property "Supplier" "https://www.digikey.ch/de/products/detail/w%C3%BCrth-elektronik/61300621821/16608633" (at 67.31 154.94 0)
       (effects (font (size 1.27 1.27)) hide)
     )
@@
       (effects (font (size 1.27 1.27)) hide)
     )
-    (property "Datasheet" "https://www.neutrik.com/en/product/nmj6hcd2" (at 132.08 167.64 0)
+    (property "Datasheet" "https://us.schurter.com/bundles/snceschurter/epim/_ProdPool_/newDS/en/typ_4833.2330.pdf" (at 132.08 167.64 0)
+      (effects (font (size 1.27 1.27)) hide)
+    )
+    (property "Supplier" "https://www.digikey.ch/de/products/detail/schurter-inc/4833-2330/9451854" (at 132.08 167.64 0)
       (effects (font (size 1.27 1.27)) hide)
     )
@@
       (effects (font (size 1.27 1.27)) hide)
     )
-    (property "Datasheet" "https://www.neutrik.com/en/product/nmj6hcd2" (at 132.08 140.97 0)
-      (effects (font (size 1.27 1.27)) hide)
-    )
+    (property "Datasheet" "https://us.schurter.com/bundles/snceschurter/epim/_ProdPool_/newDS/en/typ_4833.2330.pdf" (at 132.08 140.97 0)
+      (effects (font (size 1.27 1.27)) hide)
+    )
+    (property "Supplier" "https://www.digikey.ch/de/products/detail/schurter-inc/4833-2330/9451854" (at 132.08 140.97 0)
+      (effects (font (size 1.27 1.27)) hide)
+    )

Commit message: Fix BOM
Parts:
- J8: Supplier https://www.digikey.ch/de/products/detail/w%C3%BCrth-elektronik/61302021821/16608495 -> https://www.digikey.ch/de/products/detail/w%C3%BCrth-elektronik/61304021821/16608657
Changed lines of the file:
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@@
       (effects (font (size 1.27 1.27)) hide)
     )
-    (property "Supplier" "https://www.digikey.ch/de/products/detail/w%C3%BCrth-elektronik/61302021821/16608495" (at 184.15 80.01 0)
+    (property "Supplier" "https://www.digikey.ch/de/products/detail/w%C3%BCrth-elektronik/61304021821/16608657" (at 184.15 80.01 0)
       (effects (font (size 1.27 1.27)) hide)
     )

Commit message: Add the audio mounting holes to the schema
Parts:
- added H1, H2, H3, H4, H5: MountingHole, MountingHole:MountingHole_2.7mm_M2.5_DIN965, symbol Mechanical:MountingHole
Changed lines of the file:
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@@
     (effects (font (size 1.27 1.27)) (justify left))
+  )
+  (symbol (lib_id "Mechanical:MountingHole") (at 53.34 54.61 0) (unit 1)
+    (in_bom yes) (on_board yes) (dnp no) (fields_autoplaced)
+    (property "Reference" "H5" (at 55.88 53.975 0)
+      (effects (font (size 1.27 1.27)) (justify left))
+    )
+    (property "Value" "MountingHole" (at 55.88 56.515 0)
+      (effects (font (size 1.27 1.27)) (justify left))
+    )
+    (property "Footprint" "MountingHole:MountingHole_2.7mm_M2.5_DIN965" (at 53.34 54.61 0)
+      (effects (font (size 1.27 1.27)) hide)
+    )
+    (property "Datasheet" "~" (at 53.34 54.61 0)
+      (effects (font (size 1.27 1.27)) hide)
+    )
+    (instances
+      (project "pedalboard-hw"
+        (path "/df521c2a-9827-4355-b809-366f4b88d5d7/6bd0afd4-cd8b-4c1d-a236-891eed0b2d91"
+          (reference "H5") (unit 1)
+        )
+      )
+    )
+  )
+  (symbol (lib_id "Mechanical:MountingHole") (at 67.31 36.83 0) (unit 1)
+    (in_bom yes) (on_board yes) (dnp no) (fields_autoplaced)
+    (property "Reference" "H4" (at 69.85 36.195 0)
+      (effects (font (size 1.27 1.27)) (justify left))
+    )
+    (property "Value" "MountingHole" (at 69.85 38.735 0)
+      (effects (font (size 1.27 1.27)) (justify left))
+    )
+    (property "Footprint" "MountingHole:MountingHole_2.7mm_M2.5_DIN965" (at 67.31 36.83 0)
+      (effects (font (size 1.27 1.27)) hide)
+    )
+    (property "Datasheet" "~" (at 67.31 36.83 0)
+      (effects (font (size 1.27 1.27)) hide)
+    )
+    (instances
+      (project "pedalboard-hw"
+        (path "/df521c2a-9827-4355-b809-366f4b88d5d7/6bd0afd4-cd8b-4c1d-a236-891eed0b2d91"
+          (reference "H4") (unit 1)
+        )
+      )
+    )
   )
   (symbol (lib_id "Connector_Audio:NMJ6HCD2") (at 36.83 166.37 270) (unit 1)
@@
         (path "/df521c2a-9827-4355-b809-366f4b88d5d7/6bd0afd4-cd8b-4c1d-a236-891eed0b2d91"
           (reference "J10") (unit 1)
+        )
+      )
+    )
+  )
+  (symbol (lib_id "Mechanical:MountingHole") (at 20.32 36.83 0) (unit 1)
+    (in_bom yes) (on_board yes) (dnp no) (fields_autoplaced)
+    (property "Reference" "H1" (at 22.86 36.195 0)
+      (effects (font (size 1.27 1.27)) (justify left))
+    )
+    (property "Value" "MountingHole" (at 22.86 38.735 0)
+      (effects (font (size 1.27 1.27)) (justify left))
+    )
+    (property "Footprint" "MountingHole:MountingHole_2.7mm_M2.5_DIN965" (at 20.32 36.83 0)
+      (effects (font (size 1.27 1.27)) hide)
+    )
+    (property "Datasheet" "~" (at 20.32 36.83 0)
+      (effects (font (size 1.27 1.27)) hide)
+    )
+    (instances
+      (project "pedalboard-hw"
+        (path "/df521c2a-9827-4355-b809-366f4b88d5d7/6bd0afd4-cd8b-4c1d-a236-891eed0b2d91"
+          (reference "H1") (unit 1)
         )
       )
@@
     )
   )
+  (symbol (lib_id "Mechanical:MountingHole") (at 20.32 54.61 0) (unit 1)
+    (in_bom yes) (on_board yes) (dnp no) (fields_autoplaced)
+    (property "Reference" "H2" (at 22.86 53.975 0)
+      (effects (font (size 1.27 1.27)) (justify left))
+    )
+    (property "Value" "MountingHole" (at 22.86 56.515 0)
+      (effects (font (size 1.27 1.27)) (justify left))
+    )
+    (property "Footprint" "MountingHole:MountingHole_2.7mm_M2.5_DIN965" (at 20.32 54.61 0)
+      (effects (font (size 1.27 1.27)) hide)
+    )
+    (property "Datasheet" "~" (at 20.32 54.61 0)
+      (effects (font (size 1.27 1.27)) hide)
+    )
+    (instances
+      (project "pedalboard-hw"
+        (path "/df521c2a-9827-4355-b809-366f4b88d5d7/6bd0afd4-cd8b-4c1d-a236-891eed0b2d91"
+          (reference "H2") (unit 1)
+        )
+      )
+    )
+  )
   (symbol (lib_id "Connector_Audio:NMJ6HCD2") (at 36.83 139.7 270) (unit 1)
     (in_bom yes) (on_board yes) (dnp no) (fields_autoplaced)
@@
         )
       )
+    )
+  )
+  (symbol (lib_id "Mechanical:MountingHole") (at 53.34 36.83 0) (unit 1)
+    (in_bom yes) (on_board yes) (dnp no) (fields_autoplaced)
+    (property "Reference" "H3" (at 55.88 36.195 0)
+      (effects (font (size 1.27 1.27)) (justify left))
+    )
+    (property "Value" "MountingHole" (at 55.88 38.735 0)
+      (effects (font (size 1.27 1.27)) (justify left))
+    )
+    (property "Footprint" "MountingHole:MountingHole_2.7mm_M2.5_DIN965" (at 53.34 36.83 0)
+      (effects (font (size 1.27 1.27)) hide)
+    )
+    (property "Datasheet" "~" (at 53.34 36.83 0)
+      (effects (font (size 1.27 1.27)) hide)
+    )
+    (instances
+      (project "pedalboard-hw"
+        (path "/df521c2a-9827-4355-b809-366f4b88d5d7/6bd0afd4-cd8b-4c1d-a236-891eed0b2d91"
+          (reference "H3") (unit 1)
+        )
+      )

Commit message: Fix Jack component
Parts:
- J10, J11, J12, J9: Supplier https://www.digikey.ch/de/products/detail/schurter-inc/4833-2330/9451854 -> https://www.digikey.ch/de/products/detail/schurter-inc/4833-2320/2644235
Changed lines of the file:
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@@
       (effects (font (size 1.27 1.27)) hide)
     )
-    (property "Datasheet" "https://us.schurter.com/bundles/snceschurter/epim/_ProdPool_/newDS/en/typ_4833.2330.pdf" (at 36.83 166.37 0)
-      (effects (font (size 1.27 1.27)) hide)
-    )
-    (property "Supplier" "https://www.digikey.ch/de/products/detail/schurter-inc/4833-2330/9451854" (at 36.83 166.37 0)
+    (property "Datasheet" "https://www.digikey.ch/de/products/detail/schurter-inc/4833-2320/2644235" (at 36.83 166.37 0)
+      (effects (font (size 1.27 1.27)) hide)
+    )
+    (property "Supplier" "https://www.digikey.ch/de/products/detail/schurter-inc/4833-2320/2644235" (at 36.83 166.37 0)
       (effects (font (size 1.27 1.27)) hide)
     )
@@
       (effects (font (size 1.27 1.27)) hide)
     )
-    (property "Datasheet" "https://us.schurter.com/bundles/snceschurter/epim/_ProdPool_/newDS/en/typ_4833.2330.pdf" (at 36.83 139.7 0)
-      (effects (font (size 1.27 1.27)) hide)
-    )
-    (property "Supplier" "https://www.digikey.ch/de/products/detail/schurter-inc/4833-2330/9451854" (at 36.83 139.7 0)
+    (property "Datasheet" "https://www.digikey.ch/de/products/detail/schurter-inc/4833-2320/2644235" (at 36.83 139.7 0)
+      (effects (font (size 1.27 1.27)) hide)
+    )
+    (property "Supplier" "https://www.digikey.ch/de/products/detail/schurter-inc/4833-2320/2644235" (at 36.83 139.7 0)
       (effects (font (size 1.27 1.27)) hide)
     )
@@
       (effects (font (size 1.27 1.27)) hide)
     )
-    (property "Datasheet" "https://us.schurter.com/bundles/snceschurter/epim/_ProdPool_/newDS/en/typ_4833.2330.pdf" (at 132.08 167.64 0)
-      (effects (font (size 1.27 1.27)) hide)
-    )
-    (property "Supplier" "https://www.digikey.ch/de/products/detail/schurter-inc/4833-2330/9451854" (at 132.08 167.64 0)
+    (property "Datasheet" "https://www.digikey.ch/de/products/detail/schurter-inc/4833-2320/2644235" (at 132.08 167.64 0)
+      (effects (font (size 1.27 1.27)) hide)
+    )
+    (property "Supplier" "https://www.digikey.ch/de/products/detail/schurter-inc/4833-2320/2644235" (at 132.08 167.64 0)
       (effects (font (size 1.27 1.27)) hide)
     )
@@
       (effects (font (size 1.27 1.27)) hide)
     )
-    (property "Datasheet" "https://us.schurter.com/bundles/snceschurter/epim/_ProdPool_/newDS/en/typ_4833.2330.pdf" (at 132.08 140.97 0)
-      (effects (font (size 1.27 1.27)) hide)
-    )
-    (property "Supplier" "https://www.digikey.ch/de/products/detail/schurter-inc/4833-2330/9451854" (at 132.08 140.97 0)
-      (effects (font (size 1.27 1.27)) hide)
-    )
+    (property "Datasheet" "https://www.digikey.ch/de/products/detail/schurter-inc/4833-2320/2644235" (at 132.08 140.97 0)
+      (effects (font (size 1.27 1.27)) hide)
+    )
+    (property "Supplier" "https://www.digikey.ch/de/products/detail/schurter-inc/4833-2320/2644235" (at 132.08 140.97 0)
+      (effects (font (size 1.27 1.27)) hide)
+    )

Commit message: Improve Audio in Routing (since now there is more space under the HIFI berry
Connections:
- net audio_in_L+ renamed in_L+
Changed lines of the file:
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@@
     (stroke (width 0) (type default))
   )
-  (label "audio_in_L+" (at 39.37 157.48 0) (fields_autoplaced)
+  (label "in_L+" (at 39.37 157.48 0) (fields_autoplaced)
     (effects (font (size 1.27 1.27)) (justify left bottom))
   )
