File: audio.kicad_sch (KiCad schematic)
At the start: 11 parts, among them J10 Audio IN Left, J11 Audio OUT Right, J12 Audio OUT Left, J6 USB_A, J7 Raspberry_pi, J8 HiFi Berry, J9 Audio IN Right

Commit message: use solder jumpers instead of own nasty fuses
Parts:
- removed F4, F5: ~, Pedalboard Library:Trace_Fuse, symbol Device:Fuse_Small
- added JP1, JP2: SJP, Jumper:SolderJumper-2_P1.3mm_Bridged_RoundedPad1.0x1.5mm, symbol Jumper:SolderJumper_2_Bridged
Connections:
- net audio_in_stereo: now also JP2.2 (B)
- net audio_out_stereo: now also JP1.2 (B)
- net at J10.SN: now also JP2.1 (A)
- net at J12.SN: now also JP1.1 (A)
Changed lines of the file:
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@@
-    (stroke (width 0) (type default))
-  )
-  (wire (pts (xy 68.58 124.46) (xy 68.58 195.58))
     (stroke (width 0) (type default))
   )
@@
     (stroke (width 0) (type default))
   )
+  (wire (pts (xy 78.74 127) (xy 78.74 185.42))
+    (stroke (width 0) (type default))
+  )
   (wire (pts (xy 182.88 148.59) (xy 182.88 153.67))
     (stroke (width 0) (type default))
@@
     (stroke (width 0) (type default))
   )
-  (wire (pts (xy 78.74 124.46) (xy 78.74 185.42))
-    (stroke (width 0) (type default))
-  )
   (wire (pts (xy 104.14 165.1) (xy 104.14 157.48))
     (stroke (width 0) (type default))
@@
   )
   (wire (pts (xy 224.79 97.79) (xy 204.47 97.79))
+    (stroke (width 0) (type default))
+  )
+  (wire (pts (xy 68.58 127) (xy 68.58 195.58))
     (stroke (width 0) (type default))
   )
@@
     )
   )
-  (symbol (lib_id "Device:Fuse_Small") (at 78.74 121.92 270) (mirror x) (unit 1)
+  (symbol (lib_id "Jumper:SolderJumper_2_Bridged") (at 78.74 123.19 90) (unit 1)
     (in_bom yes) (on_board yes) (dnp no)
-    (property "Reference" "F5" (at 77.47 122.555 90)
+    (property "Reference" "JP2" (at 81.28 125.73 90)
       (effects (font (size 1.27 1.27)) (justify right))
     )
-    (property "Value" "~" (at 77.47 123.825 90)
+    (property "Value" "SJP" (at 81.28 123.19 90)
       (effects (font (size 1.27 1.27)) (justify right))
     )
-    (property "Footprint" "Pedalboard Library:Trace_Fuse" (at 78.74 121.92 0)
-      (effects (font (size 1.27 1.27)) hide)
-    )
-    (property "Datasheet" "~" (at 78.74 121.92 0)
+    (property "Footprint" "Jumper:SolderJumper-2_P1.3mm_Bridged_RoundedPad1.0x1.5mm" (at 78.74 123.19 0)
+      (effects (font (size 1.27 1.27)) hide)
+    )
+    (property "Datasheet" "~" (at 78.74 123.19 0)
       (effects (font (size 1.27 1.27)) hide)
     )
@@
       (project "pedalboard-hw"
         (path "/df521c2a-9827-4355-b809-366f4b88d5d7/6bd0afd4-cd8b-4c1d-a236-891eed0b2d91"
-          (reference "F5") (unit 1)
+          (reference "JP2") (unit 1)
         )
       )
@@
         (path "/df521c2a-9827-4355-b809-366f4b88d5d7/6bd0afd4-cd8b-4c1d-a236-891eed0b2d91"
           (reference "J7") (unit 1)
+        )
+      )
+    )
+  )
+  (symbol (lib_id "Jumper:SolderJumper_2_Bridged") (at 68.58 123.19 90) (unit 1)
+    (in_bom yes) (on_board yes) (dnp no)
+    (property "Reference" "JP1" (at 63.5 125.73 90)
+      (effects (font (size 1.27 1.27)) (justify right))
+    )
+    (property "Value" "SJP" (at 63.5 123.19 90)
+      (effects (font (size 1.27 1.27)) (justify right))
+    )
+    (property "Footprint" "Jumper:SolderJumper-2_P1.3mm_Bridged_RoundedPad1.0x1.5mm" (at 68.58 123.19 0)
+      (effects (font (size 1.27 1.27)) hide)
+    )
+    (property "Datasheet" "~" (at 68.58 123.19 0)
+      (effects (font (size 1.27 1.27)) hide)
+    )
+    (pin "1")
+    (pin "2")
+    (instances
+      (project "pedalboard-hw"
+        (path "/df521c2a-9827-4355-b809-366f4b88d5d7/6bd0afd4-cd8b-4c1d-a236-891eed0b2d91"
+          (reference "JP1") (unit 1)
         )
       )
@@
         )
       )
-    )
-  )
-  (symbol (lib_id "Device:Fuse_Small") (at 68.58 121.92 270) (mirror x) (unit 1)
-    (in_bom yes) (on_board yes) (dnp no)
-    (property "Reference" "F4" (at 67.31 122.555 90)
-      (effects (font (size 1.27 1.27)) (justify right))
-    )
-    (property "Value" "~" (at 67.31 123.825 90)
-      (effects (font (size 1.27 1.27)) (justify right))
-    )
-    (property "Footprint" "Pedalboard Library:Trace_Fuse" (at 68.58 121.92 0)
-      (effects (font (size 1.27 1.27)) hide)
-    )
-    (property "Datasheet" "~" (at 68.58 121.92 0)
-      (effects (font (size 1.27 1.27)) hide)
-    )
-    (pin "1")
-    (pin "2")
-    (instances
-      (project "pedalboard-hw"
-        (path "/df521c2a-9827-4355-b809-366f4b88d5d7/6bd0afd4-cd8b-4c1d-a236-891eed0b2d91"
-          (reference "F4") (unit 1)
-        )
-      )

Commit message: Initial Revision of CM4
Parts:
- removed J6: USB_A, Pedalboard Library:USB A BCB Male Plug, symbol Connector:USB_A
- removed J7: Raspberry_pi, Pedalboard Library:Raspberry PI Compute Module CM4 Nano A, symbol Connector:Raspberry_Pi_2_3
- added CM4: ComputeModule4-CM4, Pedalboard Library:Raspberry-Pi-4-Compute-Module, symbol pedalboard:ComputeModule4-CM4
- added D5: LED Y, LED_SMD:LED_0805_2012Metric, symbol Device:LED
- added D6: LED G, LED_SMD:LED_0805_2012Metric, symbol Device:LED
- added R2, R6: 7.5K, Resistor_SMD:R_0805_2012Metric, symbol Device:R
Connections:
- net +5VP: now also J8.4 (5V), CM4.77 (+5v_(Input)), CM4.79 (+5v_(Input)), CM4.81 (+5v_(Input)), CM4.83 (+5v_(Input)), CM4.85 (+5v_(Input)), CM4.87 (+5v_(Input))
- net GND: now also CM4.1 (GND), CM4.13 (GND), CM4.14 (GND), CM4.2 (GND), CM4.22 (GND), CM4.23 (GND), CM4.32 (GND), CM4.33 (GND), CM4.42 (GND), CM4.43 (GND), CM4.52 (GND), CM4.53 (GND), CM4.59 (GND), CM4.60 (GND), CM4.65 (GND), CM4.66 (GND), CM4.7 (GND), CM4.71 (GND), CM4.74 (GND), CM4.8 (GND), CM4.98 (GND)
- net INT_MIDI_RX: now also CM4.51 (GPIO15); no longer J8.10 (GPIO15/RXD)
- net INT_MIDI_TX: now also CM4.55 (GPIO14); no longer J8.8 (GPIO14/TXD)
- net audio_in_stereo: now also CM4.48 (GPIO27); no longer J8.13 (GPIO27)
- net audio_out_stereo: now also CM4.24 (GPIO26); no longer J8.37 (GPIO26)
- net audio_pcm_clk: now also CM4.49 (GPIO18)
- net audio_pcm_din: now also CM4.27 (GPIO20)
- net audio_pcm_dout: now also CM4.25 (GPIO21)
- net audio_pcm_fs: now also CM4.26 (GPIO19)
- net conf_i2c_scl: now also CM4.56 (GPIO3)
- net conf_i2c_sda: now also CM4.58 (GPIO2)
- net CM4_3V3: now reaches J8.1 (3V3)
- net CM4_3V3: now also J8.17 (3V3), CM4.84 (+3.3v_(Output)), CM4.86 (+3.3v_(Output)), R2.2, R6.2
- new net: D5.2 (A), R2.1
- new net: D6.2 (A), R6.1
- new net CM4_LED_ACT: CM4.21 (PI_nLED_Activity), D5.1 (K)
- new net CM4_LED_PWR: CM4.95 (nPI_LED_PWR), D6.1 (K)
Other:
- moved on the sheet: H10, H11, J9, JP1, JP2

Commit message: Set the GPIO reference to 3.3V
Connections:
- net CM4_3V3: now also CM4.78 (GPIO_VREF(1.8v/3.3v_Input))
Changed lines of the file:
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@@
   (junction (at 109.22 171.45) (diameter 0) (color 0 0 0 0)
+  )
+  (junction (at 17.78 128.27) (diameter 0) (color 0 0 0 0)
   )
   (junction (at 105.41 52.07) (diameter 0) (color 0 0 0 0)
@@
     (stroke (width 0) (type default))
   )
+  (wire (pts (xy 17.78 120.65) (xy 17.78 128.27))
+    (stroke (width 0) (type default))
+  )
   (wire (pts (xy 189.23 39.37) (xy 186.69 39.37))
     (stroke (width 0) (type default))
@@
     (stroke (width 0) (type default))
   )
+  (wire (pts (xy 17.78 120.65) (xy 40.64 120.65))
+    (stroke (width 0) (type default))
+  )

Commit message: Driver for LED
Parts:
- added U3: 74AHCT1G32SE-7, SOT-353_SC-70-5, symbol 74AHCT1G32SE-7:74AHCT1G32SE-7
- R2: value 7.5K -> 1k
- R6: value 7.5K -> 1K
Connections:
- net CM4_3V3: now also U3.5 (VCC); no longer R6.2
- net CM4_LED_PWR: now also U3.1 (A); no longer D6.1 (K)
- net GND: now also D6.1 (K), U3.2 (B), U3.3 (GND)
- new net: R6.2, U3.4 (Y)
Other:
- moved on the sheet: D5, H10, H11, R2

Commit message: Connect complete GPIO header
Connections:
- net INT_MIDI_RX: now also J8.10 (GPIO15/RXD)
- net INT_MIDI_TX: now also J8.8 (GPIO14/TXD)
- net audio_in_stereo: now also J8.13 (GPIO27)
- net audio_out_stereo: now also J8.37 (GPIO26)
- net CM4_GPIO13: now reaches CM4.28 (GPIO13)
- net CM4_GPIO13: now also J8.33 (PWM1/GPIO13)
- net CM4_GPIO16: now reaches CM4.29 (GPIO16)
- net CM4_GPIO16: now also J8.36 (GPIO16)
- net CM4_GPIO6: now reaches CM4.30 (GPIO6)
- net CM4_GPIO6: now also J8.31 (GCLK2/GPIO6)
- net CM4_GPIO12: now reaches CM4.31 (GPIO12)
- net CM4_GPIO12: now also J8.32 (PWM0/GPIO12)
- net CM4_GPIO5: now reaches CM4.34 (GPIO5)
- net CM4_GPIO5: now also J8.29 (GCLK1/GPIO5)
- net CM4_ID_SC: now reaches CM4.35 (ID_SC)
- net CM4_ID_SC: now also J8.28 (ID_SC/GPIO1)
- net CM4_ID_SD: now reaches CM4.36 (ID_SD)
- net CM4_ID_SD: now also J8.27 (ID_SD/GPIO0)
- net CM4_GPIO7: now reaches CM4.37 (GPIO7)
- net CM4_GPIO7: now also J8.26 (~{CE1}/GPIO7)
- net CM4_GPIO11: now reaches CM4.38 (GPIO11)
- net CM4_GPIO11: now also J8.23 (SCLK0/GPIO11)
- net CM4_GPIO8: now reaches CM4.39 (GPIO8)
- net CM4_GPIO8: now also J8.24 (~{CE0}/GPIO8)
- net CM4_GPIO9: now reaches CM4.40 (GPIO9)
- net CM4_GPIO9: now also J8.21 (MISO0/GPIO9)
- net CM4_GPIO25: now reaches CM4.41 (GPIO25)
- net CM4_GPIO25: now also J8.22 (GPIO25)
- net CM4_GPIO10: now reaches CM4.44 (GPIO10)
- net CM4_GPIO10: now also J8.19 (MOSI0/GPIO10)
- net CM4_GPIO24: now reaches CM4.45 (GPIO24)
- net CM4_GPIO24: now also J8.18 (GPIO24)
- net CM4_GPIO22: now reaches CM4.46 (GPIO22)
- net CM4_GPIO22: now also J8.15 (GPIO22)
- net CM4_GPIO23: now reaches CM4.47 (GPIO23)
- net CM4_GPIO23: now also J8.16 (GPIO23)
- net CM4_GPIO17: now reaches CM4.50 (GPIO17)
- net CM4_GPIO17: now also J8.11 (GPIO17)
- net CM4_GPIO4: now reaches CM4.54 (GPIO4)
- net CM4_GPIO4: now also J8.7 (GCLK0/GPIO4)

Commit message: Add mounting hole for sound card
Parts:
- added H13, H8: MountingHole, MountingHole:MountingHole_2.7mm_M2.5_DIN965, symbol Mechanical:MountingHole
Other:
- moved on the sheet: H10, H11
Changed lines of the file:
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@@
     (effects (font (size 1.27 1.27)) (justify left))
   )
-  (symbol (lib_id "Mechanical:MountingHole") (at 20.32 177.8 0) (unit 1)
-    (in_bom yes) (on_board yes) (dnp no) (fields_autoplaced)
-    (property "Reference" "H10" (at 22.86 177.165 0)
-      (effects (font (size 1.27 1.27)) (justify left))
-    )
-    (property "Value" "MountingHole" (at 22.86 179.705 0)
-      (effects (font (size 1.27 1.27)) (justify left))
-    )
-    (property "Footprint" "MountingHole:MountingHole_2.7mm_M2.5_DIN965" (at 20.32 177.8 0)
-      (effects (font (size 1.27 1.27)) hide)
-    )
-    (property "Datasheet" "~" (at 20.32 177.8 0)
+  (symbol (lib_id "Mechanical:MountingHole") (at 15.24 181.61 0) (unit 1)
+    (in_bom yes) (on_board yes) (dnp no) (fields_autoplaced)
+    (property "Reference" "H10" (at 17.78 180.975 0)
+      (effects (font (size 1.27 1.27)) (justify left))
+    )
+    (property "Value" "MountingHole" (at 17.78 183.515 0)
+      (effects (font (size 1.27 1.27)) (justify left))
+    )
+    (property "Footprint" "MountingHole:MountingHole_2.7mm_M2.5_DIN965" (at 15.24 181.61 0)
+      (effects (font (size 1.27 1.27)) hide)
+    )
+    (property "Datasheet" "~" (at 15.24 181.61 0)
       (effects (font (size 1.27 1.27)) hide)
     )
@@
     )
   )
+  (symbol (lib_id "Mechanical:MountingHole") (at 33.02 181.61 0) (unit 1)
+    (in_bom yes) (on_board yes) (dnp no) (fields_autoplaced)
+    (property "Reference" "H8" (at 35.56 180.975 0)
+      (effects (font (size 1.27 1.27)) (justify left))
+    )
+    (property "Value" "MountingHole" (at 35.56 183.515 0)
+      (effects (font (size 1.27 1.27)) (justify left))
+    )
+    (property "Footprint" "MountingHole:MountingHole_2.7mm_M2.5_DIN965" (at 33.02 181.61 0)
+      (effects (font (size 1.27 1.27)) hide)
+    )
+    (property "Datasheet" "~" (at 33.02 181.61 0)
+      (effects (font (size 1.27 1.27)) hide)
+    )
+    (instances
+      (project "pedalboard-hw"
+        (path "/df521c2a-9827-4355-b809-366f4b88d5d7/6bd0afd4-cd8b-4c1d-a236-891eed0b2d91"
+          (reference "H8") (unit 1)
+        )
+      )
+    )
+  )
   (symbol (lib_id "74AHCT1G32SE-7:74AHCT1G32SE-7") (at 252.73 50.8 0) (unit 1)
     (in_bom yes) (on_board yes) (dnp no) (fields_autoplaced)
@@
     )
   )
-  (symbol (lib_id "Mechanical:MountingHole") (at 20.32 189.23 0) (unit 1)
-    (in_bom yes) (on_board yes) (dnp no) (fields_autoplaced)
-    (property "Reference" "H11" (at 22.86 188.595 0)
-      (effects (font (size 1.27 1.27)) (justify left))
-    )
-    (property "Value" "MountingHole" (at 22.86 191.135 0)
-      (effects (font (size 1.27 1.27)) (justify left))
-    )
-    (property "Footprint" "MountingHole:MountingHole_2.7mm_M2.5_DIN965" (at 20.32 189.23 0)
-      (effects (font (size 1.27 1.27)) hide)
-    )
-    (property "Datasheet" "~" (at 20.32 189.23 0)
+  (symbol (lib_id "Mechanical:MountingHole") (at 15.24 193.04 0) (unit 1)
+    (in_bom yes) (on_board yes) (dnp no) (fields_autoplaced)
+    (property "Reference" "H11" (at 17.78 192.405 0)
+      (effects (font (size 1.27 1.27)) (justify left))
+    )
+    (property "Value" "MountingHole" (at 17.78 194.945 0)
+      (effects (font (size 1.27 1.27)) (justify left))
+    )
+    (property "Footprint" "MountingHole:MountingHole_2.7mm_M2.5_DIN965" (at 15.24 193.04 0)
+      (effects (font (size 1.27 1.27)) hide)
+    )
+    (property "Datasheet" "~" (at 15.24 193.04 0)
       (effects (font (size 1.27 1.27)) hide)
     )
@@
         )
       )
+    )
+  )
+  (symbol (lib_id "Mechanical:MountingHole") (at 33.02 193.04 0) (unit 1)
+    (in_bom yes) (on_board yes) (dnp no) (fields_autoplaced)
+    (property "Reference" "H13" (at 35.56 192.405 0)
+      (effects (font (size 1.27 1.27)) (justify left))
+    )
+    (property "Value" "MountingHole" (at 35.56 194.945 0)
+      (effects (font (size 1.27 1.27)) (justify left))
+    )
+    (property "Footprint" "MountingHole:MountingHole_2.7mm_M2.5_DIN965" (at 33.02 193.04 0)
+      (effects (font (size 1.27 1.27)) hide)
+    )
+    (property "Datasheet" "~" (at 33.02 193.04 0)
+      (effects (font (size 1.27 1.27)) hide)
+    )
+    (instances
+      (project "pedalboard-hw"
+        (path "/df521c2a-9827-4355-b809-366f4b88d5d7/6bd0afd4-cd8b-4c1d-a236-891eed0b2d91"
+          (reference "H13") (unit 1)
+        )
+      )

Commit message: All pins unconnected
Connections:
- no-connect marks 10 -> 50
Changed lines of the file:
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@@
   (junction (at 187.96 153.67) (diameter 0) (color 0 0 0 0)
   )
+  (no_connect (at 101.6 110.49))
+  (no_connect (at 101.6 100.33))
   (no_connect (at 262.89 116.84))
+  (no_connect (at 40.64 123.19))
+  (no_connect (at 101.6 36.83))
+  (no_connect (at 101.6 34.29))
+  (no_connect (at 101.6 146.05))
+  (no_connect (at 40.64 143.51))
+  (no_connect (at 40.64 26.67))
   (no_connect (at 257.81 116.84))
+  (no_connect (at 40.64 148.59))
   (no_connect (at 262.89 147.32))
+  (no_connect (at 101.6 41.91))
+  (no_connect (at 101.6 95.25))
+  (no_connect (at 40.64 140.97))
   (no_connect (at 260.35 116.84))
+  (no_connect (at 40.64 138.43))
   (no_connect (at 267.97 147.32))
+  (no_connect (at 101.6 140.97))
+  (no_connect (at 101.6 44.45))
+  (no_connect (at 40.64 29.21))
+  (no_connect (at 101.6 138.43))
+  (no_connect (at 101.6 107.95))
   (no_connect (at 260.35 147.32))
+  (no_connect (at 40.64 133.35))
+  (no_connect (at 101.6 46.99))
+  (no_connect (at 40.64 34.29))
+  (no_connect (at 40.64 107.95))
+  (no_connect (at 40.64 135.89))
+  (no_connect (at 40.64 46.99))
+  (no_connect (at 40.64 44.45))
+  (no_connect (at 101.6 29.21))
+  (no_connect (at 40.64 41.91))
+  (no_connect (at 40.64 113.03))
+  (no_connect (at 40.64 36.83))
   (no_connect (at 106.68 166.37))
+  (no_connect (at 101.6 118.11))
+  (no_connect (at 40.64 102.87))
   (no_connect (at 204.47 114.3))
+  (no_connect (at 101.6 115.57))
+  (no_connect (at 40.64 118.11))
+  (no_connect (at 101.6 135.89))
+  (no_connect (at 40.64 100.33))
+  (no_connect (at 101.6 102.87))
+  (no_connect (at 101.6 148.59))
+  (no_connect (at 40.64 125.73))
+  (no_connect (at 101.6 26.67))
   (no_connect (at 204.47 124.46))
+  (no_connect (at 40.64 110.49))
   (no_connect (at 267.97 116.84))
   (wire (pts (xy 234.95 60.96) (xy 234.95 71.12))
@@
   )
   (symbol (lib_id "power:GND") (at 105.41 113.03 0) (unit 1)
-    (in_bom yes) (on_board yes) (dnp no) (fields_autoplaced)
+    (in_bom yes) (on_board yes) (dnp no)
     (property "Reference" "#PWR036" (at 105.41 119.38 0)
       (effects (font (size 1.27 1.27)) hide)
     )
-    (property "Value" "GND" (at 105.41 118.11 0)
+    (property "Value" "GND" (at 109.22 114.3 0)
       (effects (font (size 1.27 1.27)))
     )
@@
   )
   (symbol (lib_id "power:+5VP") (at 111.76 120.65 0) (unit 1)
-    (in_bom yes) (on_board yes) (dnp no) (fields_autoplaced)
+    (in_bom yes) (on_board yes) (dnp no)
     (property "Reference" "#PWR037" (at 111.76 124.46 0)
       (effects (font (size 1.27 1.27)) hide)
     )
-    (property "Value" "+5VP" (at 111.76 115.57 0)
+    (property "Value" "+5VP" (at 115.57 119.38 0)
       (effects (font (size 1.27 1.27)))
     )

Commit message: Start to clean up the BOM
Parts:
- CM4: Field4 Hirose -> (none); Field5 2x DF40C-100DS-0.4V -> (none)
- U3: DigiKey_Part_Number 74AHCT1G32SE-7DITR-ND -> (none); MF Diodes Inc. -> (none); MP 74AHCT1G32SE-7 -> (none); MPN 74AHCT1G32SE-7 -> (none); OC_FARNELL 2057398 -> (none); OC_NEWARK 64T4877 -> (none); PACKAGE SOT-353-5 -> (none)
Changed lines of the file:
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@@
       (effects (font (size 1.27 1.27)) hide)
     )
-    (property "Datasheet" "" (at 215.9 106.68 0)
-      (effects (font (size 1.27 1.27)) hide)
-    )
-    (property "Field4" "Hirose" (at 71.12 16.51 0)
-      (effects (font (size 1.27 1.27)))
-    )
-    (property "Field5" "2x DF40C-100DS-0.4V" (at 71.12 19.05 0)
-      (effects (font (size 1.27 1.27)))
+    (property "Datasheet" "DF40C-100DS-0.4V" (at 215.9 106.68 0)
+      (effects (font (size 1.27 1.27)) hide)
     )
     (pin "1")
@@
       (effects (font (size 1.27 1.27)) hide)
     )
-    (property "DigiKey_Part_Number" "74AHCT1G32SE-7DITR-ND" (at 252.73 50.8 0)
-      (effects (font (size 1.27 1.27)) (justify bottom) hide)
-    )
-    (property "MF" "Diodes Inc." (at 252.73 50.8 0)
-      (effects (font (size 1.27 1.27)) (justify bottom) hide)
-    )
-    (property "PACKAGE" "SOT-353-5" (at 252.73 50.8 0)
-      (effects (font (size 1.27 1.27)) (justify bottom) hide)
-    )
-    (property "MPN" "74AHCT1G32SE-7" (at 252.73 50.8 0)
-      (effects (font (size 1.27 1.27)) (justify bottom) hide)
-    )
-    (property "OC_FARNELL" "2057398" (at 252.73 50.8 0)
-      (effects (font (size 1.27 1.27)) (justify bottom) hide)
-    )
-    (property "MP" "74AHCT1G32SE-7" (at 252.73 50.8 0)
-      (effects (font (size 1.27 1.27)) (justify bottom) hide)
-    )
-    (property "OC_NEWARK" "64T4877" (at 252.73 50.8 0)
-      (effects (font (size 1.27 1.27)) (justify bottom) hide)
-    )
     (property "Supplier" "https://www.digikey.ch/de/products/detail/diodes-incorporated/74AHCT1G32SE-7/2711987" (at 252.73 50.8 0)
