File: pedalboard-hw.kicad_sch (KiCad schematic)
At the start: 0 parts

Commit message: Add Midi & Rotary buttons
Other:
- removed sheet inputs
- added sheet pico (pico.kicad_sch)
Changed lines of the file:
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@@
     )
   )
-  (sheet (at 20.32 59.69) (size 21.59 19.05) (fields_autoplaced)
+  (sheet (at 48.26 25.4) (size 59.69 53.34) (fields_autoplaced)
     (stroke (width 0.1524) (type solid))
     (fill (color 0 0 0 0.0000))
-    (property "Sheetname" "inputs" (at 20.32 58.9784 0)
+    (property "Sheetname" "pico" (at 48.26 24.6884 0)
       (effects (font (size 1.27 1.27)) (justify left bottom))
     )
-    (property "Sheetfile" "inputs.kicad_sch" (at 20.32 79.3246 0)
+    (property "Sheetfile" "pico.kicad_sch" (at 48.26 79.3246 0)
       (effects (font (size 1.27 1.27)) (justify left top))
     )

Commit message: Move leds to pico page
Other:
- removed sheet leds
Changed lines of the file:
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@@
 (kicad_sch (version 20230121) (generator eeschema)
   (paper "A4")
-  (sheet (at 20.32 25.4) (size 20.32 17.78) (fields_autoplaced)
+  (sheet (at 72.39 25.4) (size 59.69 53.34) (fields_autoplaced)
     (stroke (width 0.1524) (type solid))
     (fill (color 0 0 0 0.0000))
-    (property "Sheetname" "leds" (at 20.32 24.6884 0)
+    (property "Sheetname" "pico" (at 72.39 24.6884 0)
       (effects (font (size 1.27 1.27)) (justify left bottom))
     )
-    (property "Sheetfile" "leds.kicad_sch" (at 20.32 43.7646 0)
+    (property "Sheetfile" "pico.kicad_sch" (at 72.39 79.3246 0)
       (effects (font (size 1.27 1.27)) (justify left top))
     )
@@
       )
     )
-  )
-  (sheet (at 48.26 25.4) (size 59.69 53.34) (fields_autoplaced)
-    (stroke (width 0.1524) (type solid))
-    (fill (color 0 0 0 0.0000))
-    (property "Sheetname" "pico" (at 48.26 24.6884 0)
-      (effects (font (size 1.27 1.27)) (justify left bottom))
-    )
-    (property "Sheetfile" "pico.kicad_sch" (at 48.26 79.3246 0)
-      (effects (font (size 1.27 1.27)) (justify left top))
-    )
-    (instances
-      (project "pedalboard-hw"
-        (path "/df521c2a-9827-4355-b809-366f4b88d5d7" (page "3"))
-      )
-    )

Commit message: Add connector for LED extension
Changed lines of the file:
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@@
 (kicad_sch (version 20230121) (generator eeschema)
   (paper "A4")
-  (sheet (at 72.39 25.4) (size 59.69 53.34) (fields_autoplaced)
+  (sheet (at 21.59 25.4) (size 59.69 53.34) (fields_autoplaced)
     (stroke (width 0.1524) (type solid))
     (fill (color 0 0 0 0.0000))
-    (property "Sheetname" "pico" (at 72.39 24.6884 0)
+    (property "Sheetname" "pico" (at 21.59 24.6884 0)
       (effects (font (size 1.27 1.27)) (justify left bottom))
     )
-    (property "Sheetfile" "pico.kicad_sch" (at 72.39 79.3246 0)
+    (property "Sheetfile" "pico.kicad_sch" (at 21.59 79.3246 0)
       (effects (font (size 1.27 1.27)) (justify left top))
     )

Commit message: Initial Audio placement
Other:
- sheet pico renamed MIDI
- added sheet Audio (audio.kicad_sch)
Changed lines of the file:
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@@
 (kicad_sch (version 20230121) (generator eeschema)
   (paper "A4")
+  (sheet (at 120.65 25.4) (size 66.04 53.34) (fields_autoplaced)
+    (stroke (width 0.1524) (type solid))
+    (fill (color 0 0 0 0.0000))
+    (property "Sheetname" "Audio" (at 120.65 24.6884 0)
+      (effects (font (size 1.27 1.27)) (justify left bottom))
+    )
+    (property "Sheetfile" "audio.kicad_sch" (at 120.65 79.3246 0)
+      (effects (font (size 1.27 1.27)) (justify left top))
+    )
+    (instances
+      (project "pedalboard-hw"
+        (path "/df521c2a-9827-4355-b809-366f4b88d5d7" (page "3"))
+      )
+    )
+  )
   (sheet (at 21.59 25.4) (size 59.69 53.34) (fields_autoplaced)
     (stroke (width 0.1524) (type solid))
     (fill (color 0 0 0 0.0000))
-    (property "Sheetname" "pico" (at 21.59 24.6884 0)
+    (property "Sheetname" "MIDI" (at 21.59 24.6884 0)
       (effects (font (size 1.27 1.27)) (justify left bottom))
     )

Commit message: Connect the USB between the processors
Other:
- sheet Audio ports: added USB_DM, USB_DP, USB_GND, V_BUS; removed none
- sheet MIDI ports: added GND, USB_DM, USB_DP, VBUS; removed none
Changed lines of the file:
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@@
 (kicad_sch (version 20230121) (generator eeschema)
   (paper "A4")
+  (wire (pts (xy 81.28 38.1) (xy 120.65 38.1))
+    (stroke (width 0) (type default))
+  )
+  (wire (pts (xy 81.28 41.91) (xy 120.65 41.91))
+    (stroke (width 0) (type default))
+  )
+  (wire (pts (xy 81.28 30.48) (xy 120.65 30.48))
+    (stroke (width 0) (type default))
+  )
+  (wire (pts (xy 81.28 34.29) (xy 120.65 34.29))
+    (stroke (width 0) (type default))
+  )
   (sheet (at 120.65 25.4) (size 66.04 53.34) (fields_autoplaced)
     (stroke (width 0.1524) (type solid))
@@
     (property "Sheetfile" "audio.kicad_sch" (at 120.65 79.3246 0)
       (effects (font (size 1.27 1.27)) (justify left top))
+    )
+    (pin "USB_GND" input (at 120.65 41.91 180)
+      (effects (font (size 1.27 1.27)) (justify left))
+    )
+    (pin "V_BUS" input (at 120.65 30.48 180)
+      (effects (font (size 1.27 1.27)) (justify left))
+    )
+    (pin "USB_DP" input (at 120.65 34.29 180)
+      (effects (font (size 1.27 1.27)) (justify left))
+    )
+    (pin "USB_DM" input (at 120.65 38.1 180)
+      (effects (font (size 1.27 1.27)) (justify left))
     )
     (instances
@@
       (effects (font (size 1.27 1.27)) (justify left top))
     )
+    (pin "USB_DM" input (at 81.28 38.1 0)
+      (effects (font (size 1.27 1.27)) (justify right))
+    )
+    (pin "GND" input (at 81.28 41.91 0)
+      (effects (font (size 1.27 1.27)) (justify right))
+    )
+    (pin "USB_DP" input (at 81.28 34.29 0)
+      (effects (font (size 1.27 1.27)) (justify right))
+    )
+    (pin "VBUS" input (at 81.28 30.48 0)
+      (effects (font (size 1.27 1.27)) (justify right))
+    )
     (instances

Commit message: Connect USB
Other:
- sheet Audio ports: added USB_DN; removed USB_DM
- sheet MIDI ports: added USB_DN; removed USB_DM
Changed lines of the file:
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@@
       (effects (font (size 1.27 1.27)) (justify left))
     )
-    (pin "USB_DM" input (at 120.65 38.1 180)
+    (pin "USB_DN" input (at 120.65 38.1 180)
       (effects (font (size 1.27 1.27)) (justify left))
     )
@@
       (effects (font (size 1.27 1.27)) (justify left top))
     )
-    (pin "USB_DM" input (at 81.28 38.1 0)
+    (pin "USB_DN" input (at 81.28 38.1 0)
       (effects (font (size 1.27 1.27)) (justify right))
     )

Commit message: Set Title Block on schematics
Other:
- title: (none) -> Open Pedalboard
Changed lines of the file:
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@@
 (kicad_sch (version 20230121) (generator eeschema)
   (paper "A4")
+  (title_block
+    (title "Open Pedalboard")
+    (date "2023-03-12")
+    (rev "0.1")
+    (comment 1 "Source Code: https://github.com/pedalboard/pedalboard-hw")
+    (comment 2 "License: CERN Open Hardware Licence Version 2 - Permissive")
+  )
   (wire (pts (xy 81.28 38.1) (xy 120.65 38.1))
     (stroke (width 0) (type default))
