File: pedalboard-hw.kicad_sch (KiCad schematic)
At the start: 3 parts

Commit message: Add footprint for level converter
Parts:
- removed H8: MountingHole, MountingHole:MountingHole_2.7mm_M2.5_DIN965, symbol Mechanical:MountingHole
Changed lines of the file:
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@@
-    )
-  )
-  (symbol (lib_id "Mechanical:MountingHole") (at 62.23 167.64 0) (unit 1)
-    (in_bom yes) (on_board yes) (dnp no) (fields_autoplaced)
-    (property "Reference" "H8" (at 64.77 167.005 0)
-      (effects (font (size 1.27 1.27)) (justify left))
-    )
-    (property "Value" "MountingHole" (at 64.77 169.545 0)
-      (effects (font (size 1.27 1.27)) (justify left))
-    )
-    (property "Footprint" "MountingHole:MountingHole_2.7mm_M2.5_DIN965" (at 62.23 167.64 0)
-      (effects (font (size 1.27 1.27)) hide)
-    )
-    (property "Datasheet" "~" (at 62.23 167.64 0)
-      (effects (font (size 1.27 1.27)) hide)
-    )
-    (instances
-      (project "pedalboard-hw"
-        (path "/df521c2a-9827-4355-b809-366f4b88d5d7"
-          (reference "H8") (unit 1)
-        )
-      )
     )
   )

Commit message: Add fiducials for p&p
Parts:
- added FID1, FID2: Fiducial, Fiducial:Fiducial_1.5mm_Mask3mm, symbol Mechanical:Fiducial
Changed lines of the file:
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@@
+    )
+  )
+  (symbol (lib_id "Mechanical:Fiducial") (at 74.93 186.69 0) (unit 1)
+    (in_bom yes) (on_board yes) (dnp no) (fields_autoplaced)
+    (property "Reference" "FID2" (at 77.47 185.42 0)
+      (effects (font (size 1.27 1.27)) (justify left))
+    )
+    (property "Value" "Fiducial" (at 77.47 187.96 0)
+      (effects (font (size 1.27 1.27)) (justify left))
+    )
+    (property "Footprint" "Fiducial:Fiducial_1.5mm_Mask3mm" (at 74.93 186.69 0)
+      (effects (font (size 1.27 1.27)) hide)
+    )
+    (property "Datasheet" "~" (at 74.93 186.69 0)
+      (effects (font (size 1.27 1.27)) hide)
+    )
+    (instances
+      (project "pedalboard-hw"
+        (path "/df521c2a-9827-4355-b809-366f4b88d5d7"
+          (reference "FID2") (unit 1)
+        )
+      )
+    )
+  )
+  (symbol (lib_id "Mechanical:Fiducial") (at 45.72 186.69 0) (unit 1)
+    (in_bom yes) (on_board yes) (dnp no) (fields_autoplaced)
+    (property "Reference" "FID1" (at 48.26 185.42 0)
+      (effects (font (size 1.27 1.27)) (justify left))
+    )
+    (property "Value" "Fiducial" (at 48.26 187.96 0)
+      (effects (font (size 1.27 1.27)) (justify left))
+    )
+    (property "Footprint" "Fiducial:Fiducial_1.5mm_Mask3mm" (at 45.72 186.69 0)
+      (effects (font (size 1.27 1.27)) hide)
+    )
+    (property "Datasheet" "~" (at 45.72 186.69 0)
+      (effects (font (size 1.27 1.27)) hide)
+    )
+    (instances
+      (project "pedalboard-hw"
+        (path "/df521c2a-9827-4355-b809-366f4b88d5d7"
+          (reference "FID1") (unit 1)
+        )
+      )
     )
   )

Commit message: Initial Revision of CM4
Other:
- added sheet Connectivity (connect.kicad_sch)
- sheet Audio ports: added none; removed USB_DN, USB_DP, USB_GND, VBUS
- sheet MIDI ports: added none; removed GND, VBUS
Changed lines of the file:
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@@
     (comment 2 "License: CERN Open Hardware Licence Version 2 - Permissive")
-  )
-  (wire (pts (xy 81.28 30.48) (xy 120.65 30.48))
-    (stroke (width 0) (type default))
   )
   (wire (pts (xy 60.96 78.74) (xy 60.96 88.9))
@@
   (wire (pts (xy 81.28 59.69) (xy 120.65 59.69))
     (stroke (width 0) (type default))
-  )
-  (wire (pts (xy 81.28 38.1) (xy 120.65 38.1))
-    (stroke (width 0) (type default))
-  )
-  (wire (pts (xy 81.28 41.91) (xy 120.65 41.91))
-    (stroke (width 0) (type default))
-  )
-  (wire (pts (xy 81.28 34.29) (xy 120.65 34.29))
-    (stroke (width 0) (type default))
-  )
-  (label "VBUS" (at 99.06 30.48 0) (fields_autoplaced)
-    (effects (font (size 1.27 1.27)) (justify left bottom))
   )
   (symbol (lib_id "Mechanical:MountingHole") (at 74.93 167.64 0) (unit 1)
@@
       (effects (font (size 1.27 1.27)) (justify left top))
     )
-    (pin "USB_GND" input (at 120.65 41.91 180)
-      (effects (font (size 1.27 1.27)) (justify left))
-    )
-    (pin "VBUS" input (at 120.65 30.48 180)
-      (effects (font (size 1.27 1.27)) (justify left))
-    )
-    (pin "USB_DP" input (at 120.65 34.29 180)
-      (effects (font (size 1.27 1.27)) (justify left))
-    )
-    (pin "USB_DN" input (at 120.65 38.1 180)
-      (effects (font (size 1.27 1.27)) (justify left))
-    )
     (pin "INT_MIDI_TX" input (at 120.65 59.69 180)
       (effects (font (size 1.27 1.27)) (justify left))
@@
       (effects (font (size 1.27 1.27)) (justify right))
     )
-    (pin "GND" input (at 81.28 41.91 0)
-      (effects (font (size 1.27 1.27)) (justify right))
-    )
     (pin "USB_DP" input (at 81.28 34.29 0)
-      (effects (font (size 1.27 1.27)) (justify right))
-    )
-    (pin "VBUS" input (at 81.28 30.48 0)
       (effects (font (size 1.27 1.27)) (justify right))
     )
@@
       )
     )
+  )
+  (sheet (at 203.2 25.4) (size 68.58 52.07) (fields_autoplaced)
+    (stroke (width 0.1524) (type solid))
+    (fill (color 0 0 0 0.0000))
+    (property "Sheetname" "Connectivity" (at 203.2 24.6884 0)
+      (effects (font (size 1.27 1.27)) (justify left bottom))
+    )
+    (property "Sheetfile" "connect.kicad_sch" (at 203.2 78.0546 0)
+      (effects (font (size 1.27 1.27)) (justify left top))
+    )
+    (instances
+      (project "pedalboard-hw"
+        (path "/df521c2a-9827-4355-b809-366f4b88d5d7" (page "6"))
+      )
+    )

Commit message: Route the USB connection
Other:
- sheet Connectivity ports: added USB2_N, USB2_P; removed none
Changed lines of the file:
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@@
     (comment 2 "License: CERN Open Hardware Licence Version 2 - Permissive")
   )
+  (wire (pts (xy 99.06 15.24) (xy 234.95 15.24))
+    (stroke (width 0) (type default))
+  )
+  (wire (pts (xy 99.06 34.29) (xy 99.06 15.24))
+    (stroke (width 0) (type default))
+  )
   (wire (pts (xy 60.96 78.74) (xy 60.96 88.9))
     (stroke (width 0) (type default))
@@
     (stroke (width 0) (type default))
   )
+  (wire (pts (xy 234.95 15.24) (xy 234.95 25.4))
+    (stroke (width 0) (type default))
+  )
+  (wire (pts (xy 227.33 25.4) (xy 227.33 19.05))
+    (stroke (width 0) (type default))
+  )
+  (wire (pts (xy 101.6 19.05) (xy 101.6 38.1))
+    (stroke (width 0) (type default))
+  )
+  (wire (pts (xy 81.28 34.29) (xy 99.06 34.29))
+    (stroke (width 0) (type default))
+  )
+  (wire (pts (xy 101.6 38.1) (xy 81.28 38.1))
+    (stroke (width 0) (type default))
+  )
+  (wire (pts (xy 227.33 19.05) (xy 101.6 19.05))
+    (stroke (width 0) (type default))
+  )
   (symbol (lib_id "Mechanical:MountingHole") (at 74.93 167.64 0) (unit 1)
     (in_bom yes) (on_board yes) (dnp no) (fields_autoplaced)
@@
       (effects (font (size 1.27 1.27)) (justify left top))
     )
-    (instances
+    (pin "USB2_N" input (at 227.33 25.4 90)
+      (effects (font (size 1.27 1.27)) (justify right))
+    )
+    (pin "USB2_P" input (at 234.95 25.4 90)
+      (effects (font (size 1.27 1.27)) (justify right))
+    )
+    (instances

Commit message: Squashed commit of the following:
commit 3fa4ca4d3c5ea62d251efd6d8a974a8ccaef8e6e
Author: Christof Laenzlinger <6319634+laenzlinger@users.noreply.github.com>
Date:   Thu Oct 19 01:43:32 2023 +0200

    Cleanup Silkscreen

commit 95b56afabf9d984d42b570e7dd0e9dc0995e2e0a
Author: Christof Laenzlinger <6319634+laenzlinger@users.noreply.github.com>
Date:   Thu Oct 19 01:37:16 2023 +0200

    Fix ERC and DRC

commit bd76d654c6e0ce2e50bc4bd0303c6b77f3cbeef5
Author: Christof Laenzlinger <6319634+laenzlinger@users.noreply.github.com>
Date:   Thu Oct 19 01:10:46 2023 +0200

    Fix ERC and DRC

commit a0cad1f8b96ac3ca8d87a02e21e40253cfdda0dd
Author: Christof Laenzlinger <6319634+laenzlinger@users.noreply.github.com>
Date:   Thu Oct 19 00:58:14 2023 +0200

    WIP: RP2040 exclude some ERC

commit aeacecf4f2a59ac45e4cb0fbeccc0331a4cb4d99
Author: Christof Laenzlinger <6319634+laenzlinger@users.noreply.github.com>
Date:   Thu Oct 19 00:55:06 2023 +0200

    WIP: RP2040 fix some DRC

commit 55081b7c6b5280d6d649d8c8080d9d887e1852bb
Author: Christof Laenzlinger <6319634+laenzlinger@users.noreply.github.com>
Date:   Thu Oct 19 00:52:29 2023 +0200

    WIP: RP2040 fix some ERC

commit 2468d2f1c68ab1f6ddb7b14c98ba6057067ac39a
Author: Christof Laenzlinger <6319634+laenzlinger@users.noreply.github.com>
Date:   Thu Oct 19 00:43:48 2023 +0200

    WIP: RP2040 fix DRC

commit f8e5d8cf744338d5751e8d0879dfe651a07f16d8
Author: Christof Laenzlinger <6319634+laenzlinger@users.noreply.github.com>
Date:   Wed Oct 18 18:38:41 2023 +0200

    WIP: RP2040 native
Other:
- sheet Power Supply ports: added USB_DN, USB_DP; removed none
Changed lines of the file:
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@@
     (comment 2 "License: CERN Open Hardware Licence Version 2 - Permissive")
   )
-  (wire (pts (xy 99.06 15.24) (xy 234.95 15.24))
+  (junction (at 194.31 19.05) (diameter 0) (color 0 0 0 0)
+  )
+  (junction (at 189.23 15.24) (diameter 0) (color 0 0 0 0)
+  )
+  (wire (pts (xy 99.06 15.24) (xy 189.23 15.24))
     (stroke (width 0) (type default))
   )
@@
     (stroke (width 0) (type default))
   )
+  (wire (pts (xy 186.69 100.33) (xy 194.31 100.33))
+    (stroke (width 0) (type default))
+  )
+  (wire (pts (xy 194.31 19.05) (xy 101.6 19.05))
+    (stroke (width 0) (type default))
+  )
   (wire (pts (xy 81.28 59.69) (xy 120.65 59.69))
     (stroke (width 0) (type default))
   )
   (wire (pts (xy 234.95 15.24) (xy 234.95 25.4))
+    (stroke (width 0) (type default))
+  )
+  (wire (pts (xy 189.23 15.24) (xy 234.95 15.24))
     (stroke (width 0) (type default))
   )
@@
     (stroke (width 0) (type default))
   )
+  (wire (pts (xy 186.69 96.52) (xy 189.23 96.52))
+    (stroke (width 0) (type default))
+  )
   (wire (pts (xy 101.6 38.1) (xy 81.28 38.1))
     (stroke (width 0) (type default))
   )
-  (wire (pts (xy 227.33 19.05) (xy 101.6 19.05))
+  (wire (pts (xy 227.33 19.05) (xy 194.31 19.05))
+    (stroke (width 0) (type default))
+  )
+  (wire (pts (xy 194.31 100.33) (xy 194.31 19.05))
+    (stroke (width 0) (type default))
+  )
+  (wire (pts (xy 189.23 96.52) (xy 189.23 15.24))
     (stroke (width 0) (type default))
   )
@@
       (effects (font (size 1.27 1.27)) (justify left top))
     )
+    (pin "USB_DP" input (at 186.69 96.52 0)
+      (effects (font (size 1.27 1.27)) (justify right))
+    )
+    (pin "USB_DN" input (at 186.69 100.33 0)
+      (effects (font (size 1.27 1.27)) (justify right))
+    )
     (instances

Commit message: Geographical re-annotate
Parts:
- renumbered H7 to H1, H9 to H3
Changed lines of the file:
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@@
   (symbol (lib_id "Mechanical:MountingHole") (at 74.93 167.64 0) (unit 1)
     (in_bom yes) (on_board yes) (dnp no) (fields_autoplaced)
-    (property "Reference" "H9" (at 77.47 167.005 0)
+    (property "Reference" "H3" (at 77.47 167.005 0)
       (effects (font (size 1.27 1.27)) (justify left))
     )
@@
       (project "pedalboard-hw"
         (path "/df521c2a-9827-4355-b809-366f4b88d5d7"
-          (reference "H9") (unit 1)
+          (reference "H3") (unit 1)
         )
       )
@@
   (symbol (lib_id "Mechanical:MountingHole") (at 45.72 167.64 0) (unit 1)
     (in_bom yes) (on_board yes) (dnp no) (fields_autoplaced)
-    (property "Reference" "H7" (at 48.26 167.005 0)
+    (property "Reference" "H1" (at 48.26 167.005 0)
       (effects (font (size 1.27 1.27)) (justify left))
     )
@@
       (project "pedalboard-hw"
         (path "/df521c2a-9827-4355-b809-366f4b88d5d7"
-          (reference "H7") (unit 1)
+          (reference "H1") (unit 1)
         )
       )
