File: pedalboard-hw.kicad_sch (KiCad schematic)
At the start: 7 parts

Commit message: Add two more mounting holes
Parts:
- added H14, H15: MountingHole, MountingHole:MountingHole_2.7mm_M2.5_DIN965, symbol Mechanical:MountingHole
Changed lines of the file:
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@@
+    )
+  )
+  (symbol (lib_id "Mechanical:MountingHole") (at 45.72 177.8 0) (unit 1)
+    (in_bom no) (on_board yes) (dnp no) (fields_autoplaced)
+    (property "Reference" "H14" (at 48.26 177.165 0)
+      (effects (font (size 1.27 1.27)) (justify left))
+    )
+    (property "Value" "MountingHole" (at 48.26 179.705 0)
+      (effects (font (size 1.27 1.27)) (justify left))
+    )
+    (property "Footprint" "MountingHole:MountingHole_2.7mm_M2.5_DIN965" (at 45.72 177.8 0)
+      (effects (font (size 1.27 1.27)) hide)
+    )
+    (property "Datasheet" "~" (at 45.72 177.8 0)
+      (effects (font (size 1.27 1.27)) hide)
+    )
+    (property "Sim.Enable" "0" (at 45.72 177.8 0)
+      (effects (font (size 1.27 1.27)) hide)
+    )
+    (instances
+      (project "pedalboard-hw"
+        (path "/df521c2a-9827-4355-b809-366f4b88d5d7"
+          (reference "H14") (unit 1)
+        )
+      )
     )
   )
@@
         )
       )
+    )
+  )
+  (symbol (lib_id "Mechanical:MountingHole") (at 74.93 177.8 0) (unit 1)
+    (in_bom no) (on_board yes) (dnp no) (fields_autoplaced)
+    (property "Reference" "H15" (at 77.47 177.165 0)
+      (effects (font (size 1.27 1.27)) (justify left))
+    )
+    (property "Value" "MountingHole" (at 77.47 179.705 0)
+      (effects (font (size 1.27 1.27)) (justify left))
+    )
+    (property "Footprint" "MountingHole:MountingHole_2.7mm_M2.5_DIN965" (at 74.93 177.8 0)
+      (effects (font (size 1.27 1.27)) hide)
+    )
+    (property "Datasheet" "~" (at 74.93 177.8 0)
+      (effects (font (size 1.27 1.27)) hide)
+    )
+    (property "Sim.Enable" "0" (at 74.93 177.8 0)
+      (effects (font (size 1.27 1.27)) hide)
+    )
+    (instances
+      (project "pedalboard-hw"
+        (path "/df521c2a-9827-4355-b809-366f4b88d5d7"
+          (reference "H15") (unit 1)
+        )
+      )

Commit message: One more mounting whole
Parts:
- added H16: MountingHole, MountingHole:MountingHole_2.7mm_M2.5_DIN965, symbol Mechanical:MountingHole
Changed lines of the file:
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@@
+	)
+	(symbol
+		(lib_id "Mechanical:MountingHole")
+		(at 60.96 172.72 0)
+		(unit 1)
+		(exclude_from_sim yes)
+		(in_bom no)
+		(on_board yes)
+		(dnp no)
+		(fields_autoplaced yes)
+		(property "Reference" "H16"
+			(at 63.5 172.085 0)
+			(effects
+				(font
+					(size 1.27 1.27)
+				)
+				(justify left)
+			)
+		)
+		(property "Value" "MountingHole"
+			(at 63.5 174.625 0)
+			(effects
+				(font
+					(size 1.27 1.27)
+				)
+				(justify left)
+			)
+		)
+		(property "Footprint" "MountingHole:MountingHole_2.7mm_M2.5_DIN965"
+			(at 60.96 172.72 0)
+			(effects
+				(font
+					(size 1.27 1.27)
+				)
+				(hide yes)
+			)
+		)
+		(property "Datasheet" "~"
+			(at 60.96 172.72 0)
+			(effects
+				(font
+					(size 1.27 1.27)
+				)
+				(hide yes)
+			)
+		)
+		(property "Description" ""
+			(at 60.96 172.72 0)
+			(effects
+				(font
+					(size 1.27 1.27)
+				)
+				(hide yes)
+			)
+		)
+		(instances
+			(project "pedalboard-hw"
+				(path "/df521c2a-9827-4355-b809-366f4b88d5d7"
+					(reference "H16")
+					(unit 1)
+				)
+			)
+		)
 	)
 	(symbol

Commit message: First routing. Still many issues
Other:
- sheet Audio ports: added CM4_3V, nEXTRST; removed none
- sheet Connectivity ports: added CM4_3V, nEXTRST; removed none
Changed lines of the file:
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@@
+	(wire
+		(pts
+			(xy 186.69 41.91) (xy 203.2 41.91)
+		)
+		(stroke
+			(width 0)
+			(type default)
+		)
+	)
 	(wire
 		(pts
@@
 		(pts
 			(xy 81.28 55.88) (xy 120.65 55.88)
+		)
+		(stroke
+			(width 0)
+			(type default)
+		)
+	)
+	(wire
+		(pts
+			(xy 186.69 52.07) (xy 203.2 52.07)
 		)
 		(stroke
@@
 			)
 		)
+		(pin "CM4_3V" input
+			(at 186.69 41.91 0)
+			(effects
+				(font
+					(size 1.27 1.27)
+				)
+				(justify right)
+			)
+		)
+		(pin "nEXTRST" input
+			(at 186.69 52.07 0)
+			(effects
+				(font
+					(size 1.27 1.27)
+				)
+				(justify right)
+			)
+		)
 		(instances
 			(project "pedalboard-hw"
@@
 			)
 		)
+		(pin "CM4_3V" input
+			(at 203.2 41.91 180)
+			(effects
+				(font
+					(size 1.27 1.27)
+				)
+				(justify left)
+			)
+		)
+		(pin "nEXTRST" input
+			(at 203.2 52.07 180)
+			(effects
+				(font
+					(size 1.27 1.27)
+				)
+				(justify left)
+			)
+		)

Commit message: Remove unused connection
Other:
- sheet Power Supply ports: added none; removed USB_DN, USB_DP
Changed lines of the file:
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@@
 		(comment 3 "Git commit hash: ${GIT_HASH}")
 	)
-	(junction
-		(at 194.31 19.05)
-		(diameter 0)
-		(color 0 0 0 0)
-	)
-	(junction
-		(at 189.23 15.24)
-		(diameter 0)
-		(color 0 0 0 0)
-	)
-	(wire
-		(pts
-			(xy 99.06 15.24) (xy 189.23 15.24)
+	(wire
+		(pts
+			(xy 99.06 15.24) (xy 234.95 15.24)
 		)
 		(stroke
@@
 	(wire
 		(pts
-			(xy 186.69 100.33) (xy 194.31 100.33)
-		)
-		(stroke
-			(width 0)
-			(type default)
-		)
-	)
-	(wire
-		(pts
-			(xy 194.31 19.05) (xy 101.6 19.05)
+			(xy 101.6 19.05) (xy 227.33 19.05)
 		)
 		(stroke
@@
 	(wire
 		(pts
-			(xy 189.23 15.24) (xy 234.95 15.24)
-		)
-		(stroke
-			(width 0)
-			(type default)
-		)
-	)
-	(wire
-		(pts
 			(xy 227.33 25.4) (xy 227.33 19.05)
 		)
@@
 	(wire
 		(pts
-			(xy 186.69 96.52) (xy 189.23 96.52)
-		)
-		(stroke
-			(width 0)
-			(type default)
-		)
-	)
-	(wire
-		(pts
 			(xy 101.6 38.1) (xy 81.28 38.1)
-		)
-		(stroke
-			(width 0)
-			(type default)
-		)
-	)
-	(wire
-		(pts
-			(xy 227.33 19.05) (xy 194.31 19.05)
-		)
-		(stroke
-			(width 0)
-			(type default)
-		)
-	)
-	(wire
-		(pts
-			(xy 194.31 100.33) (xy 194.31 19.05)
-		)
-		(stroke
-			(width 0)
-			(type default)
-		)
-	)
-	(wire
-		(pts
-			(xy 189.23 96.52) (xy 189.23 15.24)
 		)
 		(stroke
@@
 			)
 		)
-		(pin "USB_DP" input
-			(at 186.69 96.52 0)
-			(effects
-				(font
-					(size 1.27 1.27)
-				)
-				(justify right)
-			)
-		)
-		(pin "USB_DN" input
-			(at 186.69 100.33 0)
-			(effects
-				(font
-					(size 1.27 1.27)
-				)
-				(justify right)
-			)
-		)

Commit message: Rename label
Other:
- sheet Connectivity ports: added USB_RP_N, USB_RP_P; removed USB2_N, USB2_P
- sheet MIDI ports: added USB_RP_N, USB_RP_P; removed USB_DN, USB_DP
Changed lines of the file:
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@@
 			)
 		)
-		(pin "USB_DN" input
+		(pin "USB_RP_N" input
 			(at 81.28 38.1 0)
 			(effects
@@
 			)
 		)
-		(pin "USB_DP" input
+		(pin "USB_RP_P" input
 			(at 81.28 34.29 0)
 			(effects
@@
 			)
 		)
-		(pin "USB2_N" input
+		(pin "USB_RP_N" input
 			(at 227.33 25.4 90)
 			(effects
@@
 			)
 		)
-		(pin "USB2_P" input
+		(pin "USB_RP_P" input
 			(at 234.95 25.4 90)
 			(effects
