File: pico.kicad_sch (KiCad schematic)
At the start: 51 parts, among them J1 MIDI_OUT, J15 MIDI IN/OUT, J16 MIDI OUT J, J17 MIDI IN J, J2 MIDI_IN, J3 EXP, J4 RGB_LED_EXT, J5 Pico USB TP, SW1 D, SW2 E, SW3 F, SW4 A, SW5 B, SW6 C, SW7 VOL Rotary, SW8 GAIN Rotary, U1 Pico, U2 H11L1

Commit message: Add footprint for MIDI plugs in own library
Parts:
- J1, J2: footprint Audio_Module:CP-2350 -> Pedalboard Library:CP-2350
Changed lines of the file:
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@@
       (effects (font (size 1.27 1.27)))
     )
-    (property "Footprint" "Audio_Module:CP-2350" (at 31.75 93.98 0)
+    (property "Footprint" "Pedalboard Library:CP-2350" (at 31.75 93.98 0)
       (effects (font (size 1.27 1.27)) hide)
     )
@@
       (effects (font (size 1.27 1.27)))
     )
-    (property "Footprint" "Audio_Module:CP-2350" (at 35.56 46.99 0)
-      (effects (font (size 1.27 1.27)) hide)
-    )
+    (property "Footprint" "Pedalboard Library:CP-2350" (at 35.56 46.99 0)
+      (effects (font (size 1.27 1.27)) hide)
+    )

Commit message: After testing the LEDs update the footprint
Parts:
- D1: footprint LED_THT:LED_D5.0mm-NeoPixel -> Pedalboard Library:LED_D5.0mm-NeoPixel
- D10, D2, D3, D4, D5, D6, D7, D8, D9: footprint LED_THT:LED_D5.0mm-NeoPixel -> Pedalboard Library:LED_D5.0mm-NeoPixel; Supplier https://www.digikey.ch/en/products/detail/adafruit-industri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 -> https://www.digikey.ch/de/products/detail/sparkfun-electron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
Changed lines of the file:
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@@
       (effects (font (size 1.27 1.27)))
     )
-    (property "Footprint" "LED_THT:LED_D5.0mm-NeoPixel" (at 203.2 132.08 0)
-      (effects (font (size 1.27 1.27)) (justify left top) hide)
-    )
-    (property "Datasheet" "https://www.adafruit.com/product/1938" (at 204.47 133.985 0)
-      (effects (font (size 1.27 1.27)) (justify left top) hide)
-    )
-    (property "Supplier" "https://www.digikey.ch/en/products/detail/adafruit-industries-llc/1938/6827082" (at 201.93 124.46 0)
+    (property "Footprint" "Pedalboard Library:LED_D5.0mm-NeoPixel" (at 203.2 132.08 0)
+      (effects (font (size 1.27 1.27)) (justify left top) hide)
+    )
+    (property "Datasheet" "https://cdn.sparkfun.com/datasheets/Components/LED/COM-12877.pdf" (at 204.47 133.985 0)
+      (effects (font (size 1.27 1.27)) (justify left top) hide)
+    )
+    (property "Supplier" "https://www.digikey.ch/de/products/detail/sparkfun-electronics/COM-12986/5673799" (at 201.93 124.46 0)
       (effects (font (size 1.27 1.27)) hide)
     )
@@
       (effects (font (size 1.27 1.27)))
     )
-    (property "Footprint" "LED_THT:LED_D5.0mm-NeoPixel" (at 227.33 160.02 0)
-      (effects (font (size 1.27 1.27)) (justify left top) hide)
-    )
-    (property "Datasheet" "https://www.adafruit.com/product/1938" (at 228.6 161.925 0)
-      (effects (font (size 1.27 1.27)) (justify left top) hide)
-    )
-    (property "Supplier" "https://www.digikey.ch/en/products/detail/adafruit-industries-llc/1938/6827082" (at 226.06 152.4 0)
+    (property "Footprint" "Pedalboard Library:LED_D5.0mm-NeoPixel" (at 227.33 160.02 0)
+      (effects (font (size 1.27 1.27)) (justify left top) hide)
+    )
+    (property "Datasheet" "https://cdn.sparkfun.com/datasheets/Components/LED/COM-12877.pdf" (at 228.6 161.925 0)
+      (effects (font (size 1.27 1.27)) (justify left top) hide)
+    )
+    (property "Supplier" "https://www.digikey.ch/de/products/detail/sparkfun-electronics/COM-12986/5673799" (at 226.06 152.4 0)
       (effects (font (size 1.27 1.27)) hide)
     )
@@
       (effects (font (size 1.27 1.27)))
     )
-    (property "Footprint" "LED_THT:LED_D5.0mm-NeoPixel" (at 227.33 99.06 0)
-      (effects (font (size 1.27 1.27)) (justify left top) hide)
-    )
-    (property "Datasheet" "https://www.adafruit.com/product/1938" (at 228.6 100.965 0)
-      (effects (font (size 1.27 1.27)) (justify left top) hide)
-    )
-    (property "Supplier" "https://www.digikey.ch/en/products/detail/adafruit-industries-llc/1938/6827082" (at 226.06 91.44 0)
+    (property "Footprint" "Pedalboard Library:LED_D5.0mm-NeoPixel" (at 227.33 99.06 0)
+      (effects (font (size 1.27 1.27)) (justify left top) hide)
+    )
+    (property "Datasheet" "https://cdn.sparkfun.com/datasheets/Components/LED/COM-12877.pdf" (at 228.6 100.965 0)
+      (effects (font (size 1.27 1.27)) (justify left top) hide)
+    )
+    (property "Supplier" "https://www.digikey.ch/de/products/detail/sparkfun-electronics/COM-12986/5673799" (at 226.06 91.44 0)
       (effects (font (size 1.27 1.27)) hide)
     )
@@
       (effects (font (size 1.27 1.27)))
     )
-    (property "Footprint" "LED_THT:LED_D5.0mm-NeoPixel" (at 273.05 99.06 0)
-      (effects (font (size 1.27 1.27)) (justify left top) hide)
-    )
-    (property "Datasheet" "https://www.adafruit.com/product/1938" (at 274.32 100.965 0)
-      (effects (font (size 1.27 1.27)) (justify left top) hide)
-    )
-    (property "Supplier" "https://www.digikey.ch/en/products/detail/adafruit-industries-llc/1938/6827082" (at 271.78 91.44 0)
+    (property "Footprint" "Pedalboard Library:LED_D5.0mm-NeoPixel" (at 273.05 99.06 0)
+      (effects (font (size 1.27 1.27)) (justify left top) hide)
+    )
+    (property "Datasheet" "https://cdn.sparkfun.com/datasheets/Components/LED/COM-12877.pdf" (at 274.32 100.965 0)
+      (effects (font (size 1.27 1.27)) (justify left top) hide)
+    )
+    (property "Supplier" "https://www.digikey.ch/de/products/detail/sparkfun-electronics/COM-12986/5673799" (at 271.78 91.44 0)
       (effects (font (size 1.27 1.27)) hide)
     )
@@
       (effects (font (size 1.27 1.27)))
     )
-    (property "Footprint" "LED_THT:LED_D5.0mm-NeoPixel" (at 227.33 132.08 0)
-      (effects (font (size 1.27 1.27)) (justify left top) hide)
-    )
-    (property "Datasheet" "https://www.adafruit.com/product/1938" (at 228.6 133.985 0)
-      (effects (font (size 1.27 1.27)) (justify left top) hide)
-    )
-    (property "Supplier" "https://www.digikey.ch/en/products/detail/adafruit-industries-llc/1938/6827082" (at 226.06 124.46 0)
+    (property "Footprint" "Pedalboard Library:LED_D5.0mm-NeoPixel" (at 227.33 132.08 0)
+      (effects (font (size 1.27 1.27)) (justify left top) hide)
+    )
+    (property "Datasheet" "https://cdn.sparkfun.com/datasheets/Components/LED/COM-12877.pdf" (at 228.6 133.985 0)
+      (effects (font (size 1.27 1.27)) (justify left top) hide)
+    )
+    (property "Supplier" "https://www.digikey.ch/de/products/detail/sparkfun-electronics/COM-12986/5673799" (at 226.06 124.46 0)
       (effects (font (size 1.27 1.27)) hide)
     )
@@
       (effects (font (size 1.27 1.27)))
     )
-    (property "Footprint" "LED_THT:LED_D5.0mm-NeoPixel" (at 251.46 99.06 0)
-      (effects (font (size 1.27 1.27)) (justify left top) hide)
-    )
-    (property "Datasheet" "https://www.adafruit.com/product/1938" (at 252.73 100.965 0)
-      (effects (font (size 1.27 1.27)) (justify left top) hide)
-    )
-    (property "Supplier" "https://www.digikey.ch/en/products/detail/adafruit-industries-llc/1938/6827082" (at 250.19 91.44 0)
+    (property "Footprint" "Pedalboard Library:LED_D5.0mm-NeoPixel" (at 251.46 99.06 0)
+      (effects (font (size 1.27 1.27)) (justify left top) hide)
+    )
+    (property "Datasheet" "https://cdn.sparkfun.com/datasheets/Components/LED/COM-12877.pdf" (at 252.73 100.965 0)
+      (effects (font (size 1.27 1.27)) (justify left top) hide)
+    )
+    (property "Supplier" "https://www.digikey.ch/de/products/detail/sparkfun-electronics/COM-12986/5673799" (at 250.19 91.44 0)
       (effects (font (size 1.27 1.27)) hide)
     )
@@
       (effects (font (size 1.27 1.27)))
     )
-    (property "Footprint" "LED_THT:LED_D5.0mm-NeoPixel" (at 203.2 99.06 0)
+    (property "Footprint" "Pedalboard Library:LED_D5.0mm-NeoPixel" (at 203.2 99.06 0)
       (effects (font (size 1.27 1.27)) (justify left top) hide)
     )
@@
       (effects (font (size 1.27 1.27)))
     )
-    (property "Footprint" "LED_THT:LED_D5.0mm-NeoPixel" (at 251.46 132.08 0)
-      (effects (font (size 1.27 1.27)) (justify left top) hide)
-    )
-    (property "Datasheet" "https://www.adafruit.com/product/1938" (at 252.73 133.985 0)
-      (effects (font (size 1.27 1.27)) (justify left top) hide)
-    )
-    (property "Supplier" "https://www.digikey.ch/en/products/detail/adafruit-industries-llc/1938/6827082" (at 250.19 124.46 0)
+    (property "Footprint" "Pedalboard Library:LED_D5.0mm-NeoPixel" (at 251.46 132.08 0)
+      (effects (font (size 1.27 1.27)) (justify left top) hide)
+    )
+    (property "Datasheet" "https://cdn.sparkfun.com/datasheets/Components/LED/COM-12877.pdf" (at 252.73 133.985 0)
+      (effects (font (size 1.27 1.27)) (justify left top) hide)
+    )
+    (property "Supplier" "https://www.digikey.ch/de/products/detail/sparkfun-electronics/COM-12986/5673799" (at 250.19 124.46 0)
       (effects (font (size 1.27 1.27)) hide)
     )
@@
       (effects (font (size 1.27 1.27)))
     )
-    (property "Footprint" "LED_THT:LED_D5.0mm-NeoPixel" (at 201.93 160.02 0)
-      (effects (font (size 1.27 1.27)) (justify left top) hide)
-    )
-    (property "Datasheet" "https://www.adafruit.com/product/1938" (at 203.2 161.925 0)
-      (effects (font (size 1.27 1.27)) (justify left top) hide)
-    )
-    (property "Supplier" "https://www.digikey.ch/en/products/detail/adafruit-industries-llc/1938/6827082" (at 200.66 152.4 0)
+    (property "Footprint" "Pedalboard Library:LED_D5.0mm-NeoPixel" (at 201.93 160.02 0)
+      (effects (font (size 1.27 1.27)) (justify left top) hide)
+    )
+    (property "Datasheet" "https://cdn.sparkfun.com/datasheets/Components/LED/COM-12877.pdf" (at 203.2 161.925 0)
+      (effects (font (size 1.27 1.27)) (justify left top) hide)
+    )
+    (property "Supplier" "https://www.digikey.ch/de/products/detail/sparkfun-electronics/COM-12986/5673799" (at 200.66 152.4 0)
       (effects (font (size 1.27 1.27)) hide)
     )
@@
       (effects (font (size 1.27 1.27)))
     )
-    (property "Footprint" "LED_THT:LED_D5.0mm-NeoPixel" (at 251.46 160.02 0)
-      (effects (font (size 1.27 1.27)) (justify left top) hide)
-    )
-    (property "Datasheet" "https://www.adafruit.com/product/1938" (at 252.73 161.925 0)
-      (effects (font (size 1.27 1.27)) (justify left top) hide)
-    )
-    (property "Supplier" "https://www.digikey.ch/en/products/detail/adafruit-industries-llc/1938/6827082" (at 250.19 152.4 0)
-      (effects (font (size 1.27 1.27)) hide)
-    )
+    (property "Footprint" "Pedalboard Library:LED_D5.0mm-NeoPixel" (at 251.46 160.02 0)
+      (effects (font (size 1.27 1.27)) (justify left top) hide)
+    )
+    (property "Datasheet" "https://cdn.sparkfun.com/datasheets/Components/LED/COM-12877.pdf" (at 252.73 161.925 0)
+      (effects (font (size 1.27 1.27)) (justify left top) hide)
+    )
+    (property "Supplier" "https://www.digikey.ch/de/products/detail/sparkfun-electronics/COM-12986/5673799" (at 250.19 152.4 0)
+      (effects (font (size 1.27 1.27)) hide)
+    )

Commit message: Fix some pcb errors
Parts:
- J2: Supplier https://www.digikey.ch/de/products/detail/cui-devices/SDS-5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 -> https://www.digikey.ch/de/products/detail/switchcraft-inc/5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
- L2, L3, L4, L5: Supplier https://www.digikey.de/en/products/detail/fair-rite-product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 -> https://www.digikey.ch/en/products/detail/fair-rite-product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
Changed lines of the file:
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@@
       (effects (font (size 1.27 1.27)) hide)
     )
-    (property "Supplier" "https://www.digikey.de/en/products/detail/fair-rite-products-corp/2743005111/8599429" (at 52.07 91.44 0)
+    (property "Supplier" "https://www.digikey.ch/en/products/detail/fair-rite-products-corp/2743005111/8599429" (at 52.07 91.44 0)
       (effects (font (size 1.27 1.27)) hide)
     )
@@
       (effects (font (size 1.27 1.27)) hide)
     )
-    (property "Supplier" "https://www.digikey.de/en/products/detail/fair-rite-products-corp/2743005111/8599429" (at 168.91 29.21 0)
+    (property "Supplier" "https://www.digikey.ch/en/products/detail/fair-rite-products-corp/2743005111/8599429" (at 168.91 29.21 0)
       (effects (font (size 1.27 1.27)) hide)
     )
@@
       (effects (font (size 1.27 1.27)) hide)
     )
-    (property "Datasheet" "https://www.cuidevices.com/product/resource/sds-j.pdf" (at 31.75 93.98 0)
-      (effects (font (size 1.27 1.27)) hide)
-    )
-    (property "Supplier" "https://www.digikey.ch/de/products/detail/cui-devices/SDS-50J/97033" (at 31.75 93.98 0)
+    (property "Datasheet" "https://www.switchcraft.com/assets/1/24/57PC5F_CD.pdf?5023" (at 31.75 93.98 0)
+      (effects (font (size 1.27 1.27)) hide)
+    )
+    (property "Supplier" "https://www.digikey.ch/de/products/detail/switchcraft-inc/57PC5F/275385" (at 31.75 93.98 0)
       (effects (font (size 1.27 1.27)) hide)
     )
@@
       (effects (font (size 1.27 1.27)) hide)
     )
-    (property "Supplier" "https://www.digikey.de/en/products/detail/fair-rite-products-corp/2743005111/8599429" (at 43.18 35.56 0)
+    (property "Supplier" "https://www.digikey.ch/en/products/detail/fair-rite-products-corp/2743005111/8599429" (at 43.18 35.56 0)
       (effects (font (size 1.27 1.27)) hide)
     )
@@
       (effects (font (size 1.27 1.27)) hide)
     )
-    (property "Supplier" "https://www.digikey.de/en/products/detail/fair-rite-products-corp/2743005111/8599429" (at 21.59 38.1 0)
-      (effects (font (size 1.27 1.27)) hide)
-    )
+    (property "Supplier" "https://www.digikey.ch/en/products/detail/fair-rite-products-corp/2743005111/8599429" (at 21.59 38.1 0)
+      (effects (font (size 1.27 1.27)) hide)
+    )

Commit message: Add Footprint for Audio Jacks
Parts:
- J3: footprint Connector_Audio:Jack_6.35mm_Neutrik_NMJ6HCD2_Horizontal -> Pedalboard Library:Jack_6.35mm_Horizontal
Changed lines of the file:
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@@
       (effects (font (size 1.27 1.27)) (justify right))
     )
-    (property "Footprint" "Connector_Audio:Jack_6.35mm_Neutrik_NMJ6HCD2_Horizontal" (at 243.84 52.07 0)
+    (property "Footprint" "Pedalboard Library:Jack_6.35mm_Horizontal" (at 243.84 52.07 0)
       (effects (font (size 1.27 1.27)) hide)
     )

Commit message: Add Footprint for Audio Jacksg
Parts:
- SW1, SW2, SW3, SW4, SW5, SW6: footprint Button_Switch_THT:SW_PUSH-12mm_Wuerth-430476085716 -> Pedalboard Library:SW_PUSH-12mm_Wuerth-430476085716
Changed lines of the file:
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@@
       (effects (font (size 1.27 1.27)))
     )
-    (property "Footprint" "Button_Switch_THT:SW_PUSH-12mm_Wuerth-430476085716" (at 60.96 168.91 0)
+    (property "Footprint" "Pedalboard Library:SW_PUSH-12mm_Wuerth-430476085716" (at 60.96 168.91 0)
       (effects (font (size 1.27 1.27)) hide)
     )
@@
       (effects (font (size 1.27 1.27)))
     )
-    (property "Footprint" "Button_Switch_THT:SW_PUSH-12mm_Wuerth-430476085716" (at 104.14 168.91 0)
+    (property "Footprint" "Pedalboard Library:SW_PUSH-12mm_Wuerth-430476085716" (at 104.14 168.91 0)
       (effects (font (size 1.27 1.27)) hide)
     )
@@
       (effects (font (size 1.27 1.27)))
     )
-    (property "Footprint" "Button_Switch_THT:SW_PUSH-12mm_Wuerth-430476085716" (at 60.96 151.13 0)
+    (property "Footprint" "Pedalboard Library:SW_PUSH-12mm_Wuerth-430476085716" (at 60.96 151.13 0)
       (effects (font (size 1.27 1.27)) hide)
     )
@@
       (effects (font (size 1.27 1.27)))
     )
-    (property "Footprint" "Button_Switch_THT:SW_PUSH-12mm_Wuerth-430476085716" (at 104.14 151.13 0)
+    (property "Footprint" "Pedalboard Library:SW_PUSH-12mm_Wuerth-430476085716" (at 104.14 151.13 0)
       (effects (font (size 1.27 1.27)) hide)
     )
@@
       (effects (font (size 1.27 1.27)))
     )
-    (property "Footprint" "Button_Switch_THT:SW_PUSH-12mm_Wuerth-430476085716" (at 144.78 167.64 0)
+    (property "Footprint" "Pedalboard Library:SW_PUSH-12mm_Wuerth-430476085716" (at 144.78 167.64 0)
       (effects (font (size 1.27 1.27)) hide)
     )
@@
       (effects (font (size 1.27 1.27)))
     )
-    (property "Footprint" "Button_Switch_THT:SW_PUSH-12mm_Wuerth-430476085716" (at 144.78 151.13 0)
-      (effects (font (size 1.27 1.27)) hide)
-    )
+    (property "Footprint" "Pedalboard Library:SW_PUSH-12mm_Wuerth-430476085716" (at 144.78 151.13 0)
+      (effects (font (size 1.27 1.27)) hide)
+    )

Commit message: Move Rotary encoder to project library
Parts:
- SW7, SW8: footprint Rotary_Encoder:RotaryEncoder_Alps_EC11E-Switch_Vertical_H20mm_CircularMountingHoles -> Pedalboard Library:RotaryEncoder_Alps_EC11E-Switch_Vertical_H20mm_CircularMountingHoles
Changed lines of the file:
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@@
       (effects (font (size 1.27 1.27)))
     )
-    (property "Footprint" "Rotary_Encoder:RotaryEncoder_Alps_EC11E-Switch_Vertical_H20mm_CircularMountingHoles" (at 120.65 121.666 0)
+    (property "Footprint" "Pedalboard Library:RotaryEncoder_Alps_EC11E-Switch_Vertical_H20mm_CircularMountingHoles" (at 120.65 121.666 0)
       (effects (font (size 1.27 1.27)) hide)
     )
@@
       (effects (font (size 1.27 1.27)))
     )
-    (property "Footprint" "Rotary_Encoder:RotaryEncoder_Alps_EC11E-Switch_Vertical_H20mm_CircularMountingHoles" (at 67.31 121.666 0)
+    (property "Footprint" "Pedalboard Library:RotaryEncoder_Alps_EC11E-Switch_Vertical_H20mm_CircularMountingHoles" (at 67.31 121.666 0)
       (effects (font (size 1.27 1.27)) hide)
     )
