File: pico.kicad_sch (KiCad schematic)
At the start: 39 parts, among them J1 MIDI_OUT, J15 MIDI IN/OUT, J16 MIDI OUT J, J17 MIDI IN J, J2 MIDI_IN, J3 EXP, J5 Pico USB TP, SW1 D, SW2 E, SW3 F, SW4 A, SW5 B, SW6 C, SW7 VOL Rotary, SW8 GAIN Rotary, U1 Pico, U2 H11L1

Commit message: Use SMD components for MIDI
Parts:
- removed R2: 470, Resistor_THT:R_Axial_DIN0207_L6.3mm_D2.5mm_P10.16mm_Horizontal, symbol Device:R
- removed U2: H11L1, Package_DIP:DIP-6_W7.62mm_LongPads, symbol Isolator:H11L1
- added U2: TLP2761, Package_SO:SO-6L_10x3.84mm_P1.27mm, symbol Isolator:TLP2761
- C1, C12: footprint Capacitor_THT:C_Disc_D3.0mm_W1.6mm_P2.50mm -> Capacitor_SMD:C_0805_2012Metric; Supplier https://www.digikey.ch/en/products/detail/vishay-beyschlag-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 -> https://www.digikey.ch/de/products/detail/kyocera-avx/KGM21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
- D11: value 1N4148 -> SM4007; footprint Diode_THT:D_DO-35_SOD27_P7.62mm_Horizontal -> Diode_SMD:D_SOD-123F; Supplier https://www.digikey.ch/en/products/detail/onsemi/1N4148/458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 -> https://www.digikey.ch/de/products/detail/micro-commercial-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
- L1, L2, L3, L4, L5: value 103_100MHz -> 120_100MHz; footprint Inductor_THT:L_Axial_L6.6mm_D2.7mm_P10.16mm_Horizontal_Vishay_IM-2 -> Inductor_SMD:L_0603_1608Metric; Supplier https://www.digikey.ch/en/products/detail/fair-rite-product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 -> https://www.digikey.ch/de/products/detail/murata-electronic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
- R1, R3, R4: footprint Resistor_THT:R_Axial_DIN0207_L6.3mm_D2.5mm_P10.16mm_Horizontal -> Resistor_SMD:R_0805_2012Metric; Supplier https://www.digikey.ch/de/products/detail/koa-speer-electro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 -> https://www.digikey.ch/de/products/detail/stackpole-electro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
Connections:
- net +3.3V: now also U2.6 (VDD)
- net EXT_MIDI_RX: now also U2.5 (VO)
- net GND: now also U2.4 (GND)
- net at D11.2 (A), L2.2: now also U2.3 (K)
- net at D11.1 (K), R1.2: now also U2.1 (A)
Other:
- moved on the sheet: L1, R1

Commit message: Replace Schotky Diode with SMD part
Parts:
- D13: value 1N5817 -> SS34HF; footprint Diode_THT:D_DO-41_SOD81_P10.16mm_Horizontal -> Diode_SMD:D_SMA; Supplier https://www.digikey.ch/en/products/detail/onsemi/1N5817RLG/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 -> https://www.digikey.ch/de/products/detail/comchip-technolog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
Changed lines of the file:
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@@
       (effects (font (size 1.27 1.27)))
     )
-    (property "Value" "1N5817" (at 196.5325 34.29 0)
+    (property "Value" "SS34HF" (at 196.5325 34.29 0)
       (effects (font (size 1.27 1.27)))
     )
-    (property "Footprint" "Diode_THT:D_DO-41_SOD81_P10.16mm_Horizontal" (at 196.85 41.275 0)
+    (property "Footprint" "Diode_SMD:D_SMA" (at 196.85 41.275 0)
       (effects (font (size 1.27 1.27)) hide)
     )
-    (property "Datasheet" "https://www.onsemi.com/pdf/datasheet/1n5817-d.pdf" (at 196.85 36.83 0)
+    (property "Datasheet" "https://www.comchiptech.com/admin/files/product/20190514101641.pdf" (at 196.85 36.83 0)
       (effects (font (size 1.27 1.27)) hide)
     )
-    (property "Supplier" "https://www.digikey.ch/en/products/detail/onsemi/1N5817RLG/807254" (at 196.85 36.83 0)
+    (property "Supplier" "https://www.digikey.ch/de/products/detail/comchip-technology/SS34-HF/10279693" (at 196.85 36.83 0)
       (effects (font (size 1.27 1.27)) hide)
     )

Commit message: Replace buttons with SMD part
Parts:
- SW1, SW2, SW3, SW4, SW5, SW6: footprint Pedalboard Library:SW_PUSH-12mm_Wuerth-430476085716 -> Button_Switch_SMD:SW_SPST_B3S-1000; Supplier https://www.digikey.ch/de/products/detail/w%C3%BCrth-elektr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 -> https://www.digikey.ch/de/products/detail/omron-electronics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
Changed lines of the file:
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@@
       (effects (font (size 1.27 1.27)))
     )
-    (property "Footprint" "Pedalboard Library:SW_PUSH-12mm_Wuerth-430476085716" (at 93.98 168.91 0)
-      (effects (font (size 1.27 1.27)) hide)
-    )
-    (property "Datasheet" "https://www.we-online.com/components/products/datasheet/430466043726.pdf" (at 93.98 168.91 0)
-      (effects (font (size 1.27 1.27)) hide)
-    )
-    (property "Supplier" "https://www.digikey.ch/de/products/detail/w%C3%BCrth-elektronik/430466043726/5209037" (at 93.98 173.99 0)
+    (property "Footprint" "Button_Switch_SMD:SW_SPST_B3S-1000" (at 93.98 168.91 0)
+      (effects (font (size 1.27 1.27)) hide)
+    )
+    (property "Datasheet" "https://omronfs.omron.com/en_US/ecb/products/pdf/en-b3s.pdf" (at 93.98 168.91 0)
+      (effects (font (size 1.27 1.27)) hide)
+    )
+    (property "Supplier" "https://www.digikey.ch/de/products/detail/omron-electronics-inc-emc-div/B3S-1000P/368390" (at 93.98 173.99 0)
       (effects (font (size 1.27 1.27)) hide)
     )
@@
       (effects (font (size 1.27 1.27)))
     )
-    (property "Footprint" "Pedalboard Library:SW_PUSH-12mm_Wuerth-430476085716" (at 125.73 168.91 0)
-      (effects (font (size 1.27 1.27)) hide)
-    )
-    (property "Datasheet" "https://www.we-online.com/components/products/datasheet/430466043726.pdf" (at 125.73 168.91 0)
-      (effects (font (size 1.27 1.27)) hide)
-    )
-    (property "Supplier" "https://www.digikey.ch/de/products/detail/w%C3%BCrth-elektronik/430466043726/5209037" (at 125.73 173.99 0)
+    (property "Footprint" "Button_Switch_SMD:SW_SPST_B3S-1000" (at 125.73 168.91 0)
+      (effects (font (size 1.27 1.27)) hide)
+    )
+    (property "Datasheet" "https://omronfs.omron.com/en_US/ecb/products/pdf/en-b3s.pdf" (at 125.73 168.91 0)
+      (effects (font (size 1.27 1.27)) hide)
+    )
+    (property "Supplier" "https://www.digikey.ch/de/products/detail/omron-electronics-inc-emc-div/B3S-1000P/368390" (at 125.73 173.99 0)
       (effects (font (size 1.27 1.27)) hide)
     )
@@
       (effects (font (size 1.27 1.27)))
     )
-    (property "Footprint" "Pedalboard Library:SW_PUSH-12mm_Wuerth-430476085716" (at 93.98 151.13 0)
-      (effects (font (size 1.27 1.27)) hide)
-    )
-    (property "Datasheet" "https://www.we-online.com/components/products/datasheet/430466043726.pdf" (at 93.98 151.13 0)
-      (effects (font (size 1.27 1.27)) hide)
-    )
-    (property "Supplier" "https://www.digikey.ch/de/products/detail/w%C3%BCrth-elektronik/430466043726/5209037" (at 93.98 156.21 0)
+    (property "Footprint" "Button_Switch_SMD:SW_SPST_B3S-1000" (at 93.98 151.13 0)
+      (effects (font (size 1.27 1.27)) hide)
+    )
+    (property "Datasheet" "https://omronfs.omron.com/en_US/ecb/products/pdf/en-b3s.pdf" (at 93.98 151.13 0)
+      (effects (font (size 1.27 1.27)) hide)
+    )
+    (property "Supplier" "https://www.digikey.ch/de/products/detail/omron-electronics-inc-emc-div/B3S-1000P/368390" (at 93.98 156.21 0)
       (effects (font (size 1.27 1.27)) hide)
     )
@@
       (effects (font (size 1.27 1.27)))
     )
-    (property "Footprint" "Pedalboard Library:SW_PUSH-12mm_Wuerth-430476085716" (at 125.73 151.13 0)
-      (effects (font (size 1.27 1.27)) hide)
-    )
-    (property "Datasheet" "https://www.we-online.com/components/products/datasheet/430466043726.pdf" (at 125.73 151.13 0)
-      (effects (font (size 1.27 1.27)) hide)
-    )
-    (property "Supplier" "https://www.digikey.ch/de/products/detail/w%C3%BCrth-elektronik/430466043726/5209037" (at 125.73 156.21 0)
+    (property "Footprint" "Button_Switch_SMD:SW_SPST_B3S-1000" (at 125.73 151.13 0)
+      (effects (font (size 1.27 1.27)) hide)
+    )
+    (property "Datasheet" "https://omronfs.omron.com/en_US/ecb/products/pdf/en-b3s.pdf" (at 125.73 151.13 0)
+      (effects (font (size 1.27 1.27)) hide)
+    )
+    (property "Supplier" "https://www.digikey.ch/de/products/detail/omron-electronics-inc-emc-div/B3S-1000P/368390" (at 125.73 156.21 0)
       (effects (font (size 1.27 1.27)) hide)
     )
@@
       (effects (font (size 1.27 1.27)))
     )
-    (property "Footprint" "Pedalboard Library:SW_PUSH-12mm_Wuerth-430476085716" (at 157.48 167.64 0)
-      (effects (font (size 1.27 1.27)) hide)
-    )
-    (property "Datasheet" "https://www.we-online.com/components/products/datasheet/430466043726.pdf" (at 157.48 167.64 0)
-      (effects (font (size 1.27 1.27)) hide)
-    )
-    (property "Supplier" "https://www.digikey.ch/de/products/detail/w%C3%BCrth-elektronik/430466043726/5209037" (at 157.48 172.72 0)
+    (property "Footprint" "Button_Switch_SMD:SW_SPST_B3S-1000" (at 157.48 167.64 0)
+      (effects (font (size 1.27 1.27)) hide)
+    )
+    (property "Datasheet" "https://omronfs.omron.com/en_US/ecb/products/pdf/en-b3s.pdf" (at 157.48 167.64 0)
+      (effects (font (size 1.27 1.27)) hide)
+    )
+    (property "Supplier" "https://www.digikey.ch/de/products/detail/omron-electronics-inc-emc-div/B3S-1000P/368390" (at 157.48 172.72 0)
       (effects (font (size 1.27 1.27)) hide)
     )
@@
       (effects (font (size 1.27 1.27)))
     )
-    (property "Footprint" "Pedalboard Library:SW_PUSH-12mm_Wuerth-430476085716" (at 157.48 151.13 0)
-      (effects (font (size 1.27 1.27)) hide)
-    )
-    (property "Datasheet" "https://www.we-online.com/components/products/datasheet/430466043726.pdf" (at 157.48 151.13 0)
-      (effects (font (size 1.27 1.27)) hide)
-    )
-    (property "Supplier" "https://www.digikey.ch/de/products/detail/w%C3%BCrth-elektronik/430466043726/5209037" (at 157.48 156.21 0)
-      (effects (font (size 1.27 1.27)) hide)
-    )
+    (property "Footprint" "Button_Switch_SMD:SW_SPST_B3S-1000" (at 157.48 151.13 0)
+      (effects (font (size 1.27 1.27)) hide)
+    )
+    (property "Datasheet" "https://omronfs.omron.com/en_US/ecb/products/pdf/en-b3s.pdf" (at 157.48 151.13 0)
+      (effects (font (size 1.27 1.27)) hide)
+    )
+    (property "Supplier" "https://www.digikey.ch/de/products/detail/omron-electronics-inc-emc-div/B3S-1000P/368390" (at 157.48 156.21 0)
+      (effects (font (size 1.27 1.27)) hide)
+    )

Commit message: Route SMD parts
Parts:
- J15: symbol Connector_Generic:Conn_02x03_Top_Bottom -> Connector_Generic:Conn_02x03_Odd_Even
Connections:
- net GND: now also J15.4 (Pin_4); no longer J15.5 (Pin_5)
- net at J17.R, J17.RN, J2.4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: now also J15.5 (Pin_5); no longer J15.3 (Pin_3)
- net at C1.1, J17.S, J2.2: now also J15.3 (Pin_3); no longer J15.2 (Pin_2)
- net at J1.5, J16.T, J16.TN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: now also J15.2 (Pin_2); no longer J15.4 (Pin_4)
Changed lines of the file:
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@@
     )
   )
-  (symbol (lib_id "Connector_Generic:Conn_02x03_Top_Bottom") (at 19.05 71.12 90) (unit 1)
+  (symbol (lib_id "Connector_Generic:Conn_02x03_Odd_Even") (at 19.05 71.12 90) (unit 1)
     (in_bom yes) (on_board yes) (dnp no) (fields_autoplaced)
     (property "Reference" "J15" (at 24.13 69.215 90)
@@
       (effects (font (size 1.27 1.27)) hide)
     )
-    (property "Datasheet" "https://www.we-online.com/components/products/datasheet/6130xx21021.pdf" (at 19.05 71.12 0)
+    (property "Datasheet" "~" (at 19.05 71.12 0)
       (effects (font (size 1.27 1.27)) hide)
     )

Commit message: use solder jumpers instead of own nasty fuses
Parts:
- removed F2, F3: ~, Pedalboard Library:Trace_Fuse, symbol Device:Fuse_Small
- added JP3, JP4: SJP, Jumper:SolderJumper-2_P1.3mm_Bridged_RoundedPad1.0x1.5mm, symbol Jumper:SolderJumper_2_Bridged
Connections:
- net INT_MIDI_RX: now also JP4.1 (A)
- net INT_MIDI_TX: now also JP3.1 (A)
- net at U1.11 (GPIO8): now also JP3.2 (B)
- net at U1.12 (GPIO9): now also JP4.2 (B)
Changed lines of the file:
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@@
-    (stroke (width 0) (type default))
-  )
-  (wire (pts (xy 109.22 64.77) (xy 101.6 64.77))
     (stroke (width 0) (type default))
   )
@@
     (stroke (width 0) (type default))
   )
-  (wire (pts (xy 109.22 67.31) (xy 101.6 67.31))
+  (wire (pts (xy 101.6 67.31) (xy 106.68 67.31))
     (stroke (width 0) (type default))
   )
@@
   )
   (wire (pts (xy 35.56 31.75) (xy 33.02 31.75))
+    (stroke (width 0) (type default))
+  )
+  (wire (pts (xy 106.68 64.77) (xy 101.6 64.77))
     (stroke (width 0) (type default))
   )
@@
     )
   )
+  (symbol (lib_id "Jumper:SolderJumper_2_Bridged") (at 110.49 67.31 0) (unit 1)
+    (in_bom yes) (on_board yes) (dnp no)
+    (property "Reference" "JP4" (at 115.57 68.58 0)
+      (effects (font (size 1.27 1.27)))
+    )
+    (property "Value" "SJP" (at 105.41 66.04 0)
+      (effects (font (size 1.27 1.27)))
+    )
+    (property "Footprint" "Jumper:SolderJumper-2_P1.3mm_Bridged_RoundedPad1.0x1.5mm" (at 110.49 67.31 0)
+      (effects (font (size 1.27 1.27)) hide)
+    )
+    (property "Datasheet" "~" (at 110.49 67.31 0)
+      (effects (font (size 1.27 1.27)) hide)
+    )
+    (pin "1")
+    (pin "2")
+    (instances
+      (project "pedalboard-hw"
+        (path "/df521c2a-9827-4355-b809-366f4b88d5d7/d36964e5-9373-47ae-95a7-088f8df77199"
+          (reference "JP4") (unit 1)
+        )
+      )
+    )
+  )
   (symbol (lib_id "Switch:SW_Omron_B3FS") (at 93.98 173.99 0) (unit 1)
     (in_bom yes) (on_board yes) (dnp no) (fields_autoplaced)
@@
         (path "/df521c2a-9827-4355-b809-366f4b88d5d7/d36964e5-9373-47ae-95a7-088f8df77199"
           (reference "SW4") (unit 1)
-        )
-      )
-    )
-  )
-  (symbol (lib_id "Device:Fuse_Small") (at 111.76 64.77 0) (unit 1)
-    (in_bom yes) (on_board yes) (dnp no)
-    (property "Reference" "F2" (at 114.3 63.5 0)
-      (effects (font (size 1.27 1.27)))
-    )
-    (property "Value" "~" (at 119.38 63.5 0)
-      (effects (font (size 1.27 1.27)))
-    )
-    (property "Footprint" "Pedalboard Library:Trace_Fuse" (at 111.76 64.77 0)
-      (effects (font (size 1.27 1.27)) hide)
-    )
-    (property "Datasheet" "~" (at 111.76 64.77 0)
-      (effects (font (size 1.27 1.27)) hide)
-    )
-    (pin "1")
-    (pin "2")
-    (instances
-      (project "pedalboard-hw"
-        (path "/df521c2a-9827-4355-b809-366f4b88d5d7/d36964e5-9373-47ae-95a7-088f8df77199"
-          (reference "F2") (unit 1)
         )
       )
@@
     )
   )
+  (symbol (lib_id "Jumper:SolderJumper_2_Bridged") (at 110.49 64.77 0) (unit 1)
+    (in_bom yes) (on_board yes) (dnp no)
+    (property "Reference" "JP3" (at 115.57 66.04 0)
+      (effects (font (size 1.27 1.27)))
+    )
+    (property "Value" "SJP" (at 105.41 63.5 0)
+      (effects (font (size 1.27 1.27)))
+    )
+    (property "Footprint" "Jumper:SolderJumper-2_P1.3mm_Bridged_RoundedPad1.0x1.5mm" (at 110.49 64.77 0)
+      (effects (font (size 1.27 1.27)) hide)
+    )
+    (property "Datasheet" "~" (at 110.49 64.77 0)
+      (effects (font (size 1.27 1.27)) hide)
+    )
+    (pin "1")
+    (pin "2")
+    (instances
+      (project "pedalboard-hw"
+        (path "/df521c2a-9827-4355-b809-366f4b88d5d7/d36964e5-9373-47ae-95a7-088f8df77199"
+          (reference "JP3") (unit 1)
+        )
+      )
+    )
+  )
   (symbol (lib_id "Switch:SW_Omron_B3FS") (at 125.73 156.21 0) (unit 1)
     (in_bom yes) (on_board yes) (dnp no) (fields_autoplaced)
@@
         )
       )
-    )
-  )
-  (symbol (lib_id "Device:Fuse_Small") (at 111.76 67.31 0) (unit 1)
-    (in_bom yes) (on_board yes) (dnp no)
-    (property "Reference" "F3" (at 114.3 66.04 0)
-      (effects (font (size 1.27 1.27)))
-    )
-    (property "Value" "~" (at 119.38 53.34 0)
-      (effects (font (size 1.27 1.27)))
-    )
-    (property "Footprint" "Pedalboard Library:Trace_Fuse" (at 111.76 67.31 0)
-      (effects (font (size 1.27 1.27)) hide)
-    )
-    (property "Datasheet" "~" (at 111.76 67.31 0)
-      (effects (font (size 1.27 1.27)) hide)
-    )
-    (pin "1")
-    (pin "2")
-    (instances
-      (project "pedalboard-hw"
-        (path "/df521c2a-9827-4355-b809-366f4b88d5d7/d36964e5-9373-47ae-95a7-088f8df77199"
-          (reference "F3") (unit 1)
-        )
-      )

Commit message: Use 12x12mm tactile buttons (SMD)
Parts:
- SW1, SW2, SW3, SW4, SW5, SW6: footprint Button_Switch_SMD:SW_SPST_B3S-1000 -> Pedalboard Library:SW_PUSH-12mm_Wuerth; Supplier https://www.digikey.ch/de/products/detail/omron-electronics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 -> https://www.digikey.ch/de/products/detail/w%C3%BCrth-elektr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
Changed lines of the file:
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@@
       (effects (font (size 1.27 1.27)))
     )
-    (property "Footprint" "Button_Switch_SMD:SW_SPST_B3S-1000" (at 93.98 168.91 0)
-      (effects (font (size 1.27 1.27)) hide)
-    )
-    (property "Datasheet" "https://omronfs.omron.com/en_US/ecb/products/pdf/en-b3s.pdf" (at 93.98 168.91 0)
-      (effects (font (size 1.27 1.27)) hide)
-    )
-    (property "Supplier" "https://www.digikey.ch/de/products/detail/omron-electronics-inc-emc-div/B3S-1000P/368390" (at 93.98 173.99 0)
+    (property "Footprint" "Pedalboard Library:SW_PUSH-12mm_Wuerth" (at 93.98 168.91 0)
+      (effects (font (size 1.27 1.27)) hide)
+    )
+    (property "Datasheet" "https://www.we-online.com/components/products/datasheet/430172043816.pdf" (at 93.98 168.91 0)
+      (effects (font (size 1.27 1.27)) hide)
+    )
+    (property "Supplier" "https://www.digikey.ch/de/products/detail/w%C3%BCrth-elektronik/430162043826/9950802" (at 93.98 173.99 0)
       (effects (font (size 1.27 1.27)) hide)
     )
@@
       (effects (font (size 1.27 1.27)))
     )
-    (property "Footprint" "Button_Switch_SMD:SW_SPST_B3S-1000" (at 125.73 168.91 0)
-      (effects (font (size 1.27 1.27)) hide)
-    )
-    (property "Datasheet" "https://omronfs.omron.com/en_US/ecb/products/pdf/en-b3s.pdf" (at 125.73 168.91 0)
-      (effects (font (size 1.27 1.27)) hide)
-    )
-    (property "Supplier" "https://www.digikey.ch/de/products/detail/omron-electronics-inc-emc-div/B3S-1000P/368390" (at 125.73 173.99 0)
+    (property "Footprint" "Pedalboard Library:SW_PUSH-12mm_Wuerth" (at 125.73 168.91 0)
+      (effects (font (size 1.27 1.27)) hide)
+    )
+    (property "Datasheet" "https://www.we-online.com/components/products/datasheet/430172043816.pdf" (at 125.73 168.91 0)
+      (effects (font (size 1.27 1.27)) hide)
+    )
+    (property "Supplier" "https://www.digikey.ch/de/products/detail/w%C3%BCrth-elektronik/430162043826/9950802" (at 125.73 173.99 0)
       (effects (font (size 1.27 1.27)) hide)
     )
@@
       (effects (font (size 1.27 1.27)))
     )
-    (property "Footprint" "Button_Switch_SMD:SW_SPST_B3S-1000" (at 93.98 151.13 0)
-      (effects (font (size 1.27 1.27)) hide)
-    )
-    (property "Datasheet" "https://omronfs.omron.com/en_US/ecb/products/pdf/en-b3s.pdf" (at 93.98 151.13 0)
-      (effects (font (size 1.27 1.27)) hide)
-    )
-    (property "Supplier" "https://www.digikey.ch/de/products/detail/omron-electronics-inc-emc-div/B3S-1000P/368390" (at 93.98 156.21 0)
+    (property "Footprint" "Pedalboard Library:SW_PUSH-12mm_Wuerth" (at 93.98 151.13 0)
+      (effects (font (size 1.27 1.27)) hide)
+    )
+    (property "Datasheet" "https://www.we-online.com/components/products/datasheet/430172043816.pdf" (at 93.98 151.13 0)
+      (effects (font (size 1.27 1.27)) hide)
+    )
+    (property "Supplier" "https://www.digikey.ch/de/products/detail/w%C3%BCrth-elektronik/430162043826/9950802" (at 93.98 156.21 0)
       (effects (font (size 1.27 1.27)) hide)
     )
@@
       (effects (font (size 1.27 1.27)))
     )
-    (property "Footprint" "Button_Switch_SMD:SW_SPST_B3S-1000" (at 125.73 151.13 0)
-      (effects (font (size 1.27 1.27)) hide)
-    )
-    (property "Datasheet" "https://omronfs.omron.com/en_US/ecb/products/pdf/en-b3s.pdf" (at 125.73 151.13 0)
-      (effects (font (size 1.27 1.27)) hide)
-    )
-    (property "Supplier" "https://www.digikey.ch/de/products/detail/omron-electronics-inc-emc-div/B3S-1000P/368390" (at 125.73 156.21 0)
+    (property "Footprint" "Pedalboard Library:SW_PUSH-12mm_Wuerth" (at 125.73 151.13 0)
+      (effects (font (size 1.27 1.27)) hide)
+    )
+    (property "Datasheet" "https://www.we-online.com/components/products/datasheet/430172043816.pdf" (at 125.73 151.13 0)
+      (effects (font (size 1.27 1.27)) hide)
+    )
+    (property "Supplier" "https://www.digikey.ch/de/products/detail/w%C3%BCrth-elektronik/430162043826/9950802" (at 125.73 156.21 0)
       (effects (font (size 1.27 1.27)) hide)
     )
@@
       (effects (font (size 1.27 1.27)))
     )
-    (property "Footprint" "Button_Switch_SMD:SW_SPST_B3S-1000" (at 157.48 167.64 0)
-      (effects (font (size 1.27 1.27)) hide)
-    )
-    (property "Datasheet" "https://omronfs.omron.com/en_US/ecb/products/pdf/en-b3s.pdf" (at 157.48 167.64 0)
-      (effects (font (size 1.27 1.27)) hide)
-    )
-    (property "Supplier" "https://www.digikey.ch/de/products/detail/omron-electronics-inc-emc-div/B3S-1000P/368390" (at 157.48 172.72 0)
+    (property "Footprint" "Pedalboard Library:SW_PUSH-12mm_Wuerth" (at 157.48 167.64 0)
+      (effects (font (size 1.27 1.27)) hide)
+    )
+    (property "Datasheet" "https://www.we-online.com/components/products/datasheet/430172043816.pdf" (at 157.48 167.64 0)
+      (effects (font (size 1.27 1.27)) hide)
+    )
+    (property "Supplier" "https://www.digikey.ch/de/products/detail/w%C3%BCrth-elektronik/430162043826/9950802" (at 157.48 172.72 0)
       (effects (font (size 1.27 1.27)) hide)
     )
@@
       (effects (font (size 1.27 1.27)))
     )
-    (property "Footprint" "Button_Switch_SMD:SW_SPST_B3S-1000" (at 157.48 151.13 0)
-      (effects (font (size 1.27 1.27)) hide)
-    )
-    (property "Datasheet" "https://omronfs.omron.com/en_US/ecb/products/pdf/en-b3s.pdf" (at 157.48 151.13 0)
-      (effects (font (size 1.27 1.27)) hide)
-    )
-    (property "Supplier" "https://www.digikey.ch/de/products/detail/omron-electronics-inc-emc-div/B3S-1000P/368390" (at 157.48 156.21 0)
-      (effects (font (size 1.27 1.27)) hide)
-    )
+    (property "Footprint" "Pedalboard Library:SW_PUSH-12mm_Wuerth" (at 157.48 151.13 0)
+      (effects (font (size 1.27 1.27)) hide)
+    )
+    (property "Datasheet" "https://www.we-online.com/components/products/datasheet/430172043816.pdf" (at 157.48 151.13 0)
+      (effects (font (size 1.27 1.27)) hide)
+    )
+    (property "Supplier" "https://www.digikey.ch/de/products/detail/w%C3%BCrth-elektronik/430162043826/9950802" (at 157.48 156.21 0)
+      (effects (font (size 1.27 1.27)) hide)
+    )

Commit message: JST connector for MIDI
Parts:
- removed J15: MIDI IN/OUT, Connector_PinHeader_2.54mm:PinHeader_2x03_P2.54mm_Horizontal, symbol Connector_Generic:Conn_02x03_Odd_Even
- added J24, J25: Conn_01x03_Pin, Connector_JST:JST_XH_B3B-XH-A_1x03_P2.50mm_Vertical, symbol Connector:Conn_01x03_Pin
Connections:
- net GND: now also J25.2 (Pin_2)
- net at J17.T, J17.TN, J2.5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: now also J24.3 (Pin_3)
- net at J17.R, J17.RN, J2.4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: now also J24.1 (Pin_1)
- net at C1.1, J17.S, J2.2: now also J24.2 (Pin_2)
- net at J1.4, J16.R, J16.RN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: now also J25.1 (Pin_1)
- net at J1.5, J16.T, J16.TN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: now also J25.3 (Pin_3)
Other:
- moved on the sheet: H1

Commit message: Resize PCB
Parts:
- J24, J25: value Conn_01x03_Pin -> EXT-MIDI
Changed lines of the file:
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@@
       (effects (font (size 1.27 1.27)) (justify right))
     )
-    (property "Value" "Conn_01x03_Pin" (at 54.61 72.39 0)
+    (property "Value" "EXT-MIDI" (at 54.61 72.39 0)
       (effects (font (size 1.27 1.27)) (justify right))
     )
@@
       (effects (font (size 1.27 1.27)) (justify right))
     )
-    (property "Value" "Conn_01x03_Pin" (at 48.26 132.08 0)
+    (property "Value" "EXT-MIDI" (at 48.26 132.08 0)
       (effects (font (size 1.27 1.27)) (justify right))
     )
