File: pico.kicad_sch (KiCad schematic)
At the start: 60 parts, among them J1 DIN5, J2 Conn_01x02, J2 Jack 3.5mm, J23 JST XH 3, J24 JST XH 3, J3 DIN5, J4 Jack 3.5mm, J6 Debug, J7 Jack 6.35mm, J9 Jack 6.35mm, SW1 Rotary, SW2 Rotary, SW3 Tactile, SW4 Tactile, SW5 Tactile, SW6 Tactile, SW7 Tactile, SW8 Tactile, U1 TLP2761, U2 W25Q128JVS, U3 RP2040, Y1 ABLS-12.000MHZ-B4-T

Commit message: Fix USB Boot mode bug
Connections:
- net QSPI_SCLK: no longer R1.2
- net QSPI_SS: now also R1.2
Other:
- moved on the sheet: J2, R1
Changed lines of the file:
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@@
     (stroke (width 0) (type default))
   )
-  (wire (pts (xy 87.63 38.1) (xy 92.71 38.1))
+  (wire (pts (xy 85.09 38.1) (xy 92.71 38.1))
     (stroke (width 0) (type default))
   )
@@
     (stroke (width 0) (type default))
   )
-  (wire (pts (xy 92.71 38.1) (xy 92.71 53.34))
+  (wire (pts (xy 92.71 38.1) (xy 92.71 41.91))
     (stroke (width 0) (type default))
   )
@@
     (stroke (width 0) (type default))
   )
-  (wire (pts (xy 87.63 40.64) (xy 88.9 40.64))
+  (wire (pts (xy 85.09 40.64) (xy 88.9 40.64))
     (stroke (width 0) (type default))
   )
@@
     (stroke (width 0) (type default))
   )
-  (wire (pts (xy 92.71 58.42) (xy 92.71 59.69))
-    (stroke (width 0) (type default))
-  )
   (wire (pts (xy 24.13 167.64) (xy 35.56 167.64))
     (stroke (width 0) (type default))
@@
     (stroke (width 0) (type default))
   )
-  (wire (pts (xy 95.25 50.8) (xy 105.41 50.8))
+  (wire (pts (xy 92.71 50.8) (xy 105.41 50.8))
     (stroke (width 0) (type default))
   )
@@
     (stroke (width 0) (type default))
   )
+  (wire (pts (xy 92.71 50.8) (xy 92.71 46.99))
+    (stroke (width 0) (type default))
+  )
   (wire (pts (xy 39.37 91.44) (xy 46.99 91.44))
     (stroke (width 0) (type default))
@@
     (effects (font (size 1.27 1.27)) (justify right bottom))
   )
-  (label "QSPI_SCLK" (at 96.52 59.69 0) (fields_autoplaced)
+  (label "QSPI_SCLK" (at 92.71 59.69 0) (fields_autoplaced)
     (effects (font (size 1.27 1.27)) (justify left bottom))
   )
@@
     )
   )
-  (symbol (lib_id "Connector_Generic:Conn_01x02") (at 82.55 38.1 0) (mirror y) (unit 1)
+  (symbol (lib_id "Connector_Generic:Conn_01x02") (at 80.01 38.1 0) (mirror y) (unit 1)
     (in_bom yes) (on_board yes) (dnp no)
-    (property "Reference" "J2" (at 81.28 34.29 0)
+    (property "Reference" "J2" (at 78.74 34.29 0)
       (effects (font (size 1.27 1.27)))
     )
-    (property "Value" "Conn_01x02" (at 81.28 44.45 0)
+    (property "Value" "Conn_01x02" (at 78.74 44.45 0)
       (effects (font (size 1.27 1.27)))
     )
-    (property "Footprint" "Connector_PinHeader_2.54mm:PinHeader_1x02_P2.54mm_Vertical" (at 82.55 38.1 0)
+    (property "Footprint" "Connector_PinHeader_2.54mm:PinHeader_1x02_P2.54mm_Vertical" (at 80.01 38.1 0)
       (effects (font (size 1.27 1.27)) hide)
     )
-    (property "Datasheet" "~" (at 82.55 38.1 0)
+    (property "Datasheet" "~" (at 80.01 38.1 0)
       (effects (font (size 1.27 1.27)) hide)
     )
@@
     )
   )
-  (symbol (lib_id "Device:R_Small") (at 92.71 55.88 0) (unit 1)
+  (symbol (lib_id "Device:R_Small") (at 92.71 44.45 0) (unit 1)
     (in_bom yes) (on_board yes) (dnp no)
-    (property "Reference" "R1" (at 87.4522 55.88 90)
+    (property "Reference" "R1" (at 87.4522 44.45 90)
       (effects (font (size 1.27 1.27)))
     )
-    (property "Value" "1K" (at 89.7636 55.88 90)
+    (property "Value" "1K" (at 89.7636 44.45 90)
       (effects (font (size 1.27 1.27)))
     )
-    (property "Footprint" "Resistor_SMD:R_0805_2012Metric" (at 90.932 55.88 90)
+    (property "Footprint" "Resistor_SMD:R_0805_2012Metric" (at 90.932 44.45 90)
       (effects (font (size 1.27 1.27)) hide)
     )
-    (property "Datasheet" "https://www.seielect.com/catalog/sei-rncp.pdf" (at 92.71 55.88 0)
+    (property "Datasheet" "https://www.seielect.com/catalog/sei-rncp.pdf" (at 92.71 44.45 0)
       (effects (font (size 1.27 1.27)) hide)
     )
-    (property "Supplier" "https://www.digikey.ch/de/products/detail/stackpole-electronics-inc/RNCP0805FTD1K00/2240229" (at 92.71 55.88 0)
+    (property "Supplier" "https://www.digikey.ch/de/products/detail/stackpole-electronics-inc/RNCP0805FTD1K00/2240229" (at 92.71 44.45 0)
       (effects (font (size 1.27 1.27)) hide)
     )

Commit message: Use PSU design based on CM4IO V5 board
Parts:
- R1: value 33 -> 33R
- R2: value 10 -> 10R
- R3, R4: value 27 -> 27R
- R3: value 220 -> 220R
Changed lines of the file:
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@@
       (effects (font (size 1.27 1.27)) (justify left))
     )
-    (property "Value" "33" (at 24.13 29.845 0)
+    (property "Value" "33R" (at 24.13 29.845 0)
       (effects (font (size 1.27 1.27)) (justify left))
     )
@@
       (effects (font (size 1.27 1.27)))
     )
-    (property "Value" "10" (at 46.99 24.13 90)
+    (property "Value" "10R" (at 46.99 24.13 90)
       (effects (font (size 1.27 1.27)))
     )
@@
       (effects (font (size 1.27 1.27)))
     )
-    (property "Value" "27" (at 243.84 52.9336 90)
+    (property "Value" "27R" (at 243.84 52.9336 90)
       (effects (font (size 1.27 1.27)))
     )
@@
       (effects (font (size 1.27 1.27)))
     )
-    (property "Value" "220" (at 44.45 78.74 90)
+    (property "Value" "220R" (at 44.45 78.74 90)
       (effects (font (size 1.27 1.27)))
     )
@@
       (effects (font (size 1.27 1.27)))
     )
-    (property "Value" "27" (at 243.84 60.5536 90)
-      (effects (font (size 1.27 1.27)))
-    )
+    (property "Value" "27R" (at 243.84 60.5536 90)
+      (effects (font (size 1.27 1.27)))
+    )

Commit message: Update References
Parts:
- renumbered J2 to J1, J1 to J2, J4 to J3, J3 to J4, J7 to J5, JP2 to JP1, JP1 to JP2, L2 to L1, L4 to L2, L1 to L4, R3 to R1, R1 to R3

Commit message: Add tactile button for USB boot
Parts:
- removed J2: Conn_01x02, Connector_PinHeader_2.54mm:PinHeader_1x02_P2.54mm_Vertical, symbol Connector_Generic:Conn_01x02
- added SW9: Tactile, Button_Switch_SMD:SW_SPST_B3U-1000P, symbol Switch:SW_Omron_B3FS
Connections:
- net GND: now also SW9.1
- net ~{USB_BOOT}: now also SW9.2
Changed lines of the file:
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@@
     (stroke (width 0) (type default))
   )
+  (wire (pts (xy 80.01 46.99) (xy 88.9 46.99))
+    (stroke (width 0) (type default))
+  )
   (wire (pts (xy 163.83 180.34) (xy 163.83 191.77))
     (stroke (width 0) (type default))
@@
     (stroke (width 0) (type default))
   )
-  (wire (pts (xy 85.09 38.1) (xy 92.71 38.1))
-    (stroke (width 0) (type default))
-  )
   (wire (pts (xy 167.64 20.32) (xy 167.64 22.86))
     (stroke (width 0) (type default))
@@
     (stroke (width 0) (type default))
   )
-  (wire (pts (xy 92.71 38.1) (xy 92.71 41.91))
+  (wire (pts (xy 92.71 30.48) (xy 92.71 41.91))
     (stroke (width 0) (type default))
   )
@@
     (stroke (width 0) (type default))
   )
-  (wire (pts (xy 85.09 40.64) (xy 88.9 40.64))
-    (stroke (width 0) (type default))
-  )
   (wire (pts (xy 228.6 121.92) (xy 243.84 121.92))
     (stroke (width 0) (type default))
@@
     (stroke (width 0) (type default))
   )
+  (wire (pts (xy 88.9 46.99) (xy 88.9 50.8))
+    (stroke (width 0) (type default))
+  )
   (wire (pts (xy 234.95 55.88) (xy 241.3 55.88))
     (stroke (width 0) (type default))
@@
     (stroke (width 0) (type default))
   )
+  (wire (pts (xy 80.01 30.48) (xy 92.71 30.48))
+    (stroke (width 0) (type default))
+  )
   (wire (pts (xy 22.86 173.99) (xy 54.61 173.99))
     (stroke (width 0) (type default))
@@
     (stroke (width 0) (type default))
   )
+  (wire (pts (xy 80.01 36.83) (xy 80.01 30.48))
+    (stroke (width 0) (type default))
+  )
   (wire (pts (xy 35.56 31.75) (xy 33.02 31.75))
     (stroke (width 0) (type default))
@@
     (stroke (width 0) (type default))
   )
-  (wire (pts (xy 88.9 40.64) (xy 88.9 41.91))
-    (stroke (width 0) (type default))
-  )
   (wire (pts (xy 87.63 109.22) (xy 87.63 119.38))
     (stroke (width 0) (type default))
@@
     (effects (font (size 1.27 1.27)) (justify left bottom))
   )
-  (label "~{USB_BOOT}" (at 87.63 38.1 0) (fields_autoplaced)
+  (label "~{USB_BOOT}" (at 82.55 30.48 0) (fields_autoplaced)
     (effects (font (size 1.27 1.27)) (justify left bottom))
   )
@@
     )
   )
-  (symbol (lib_id "Connector_Generic:Conn_01x02") (at 80.01 38.1 0) (mirror y) (unit 1)
-    (in_bom yes) (on_board yes) (dnp no)
-    (property "Reference" "J2" (at 78.74 34.29 0)
-      (effects (font (size 1.27 1.27)))
-    )
-    (property "Value" "Conn_01x02" (at 78.74 44.45 0)
-      (effects (font (size 1.27 1.27)))
-    )
-    (property "Footprint" "Connector_PinHeader_2.54mm:PinHeader_1x02_P2.54mm_Vertical" (at 80.01 38.1 0)
-      (effects (font (size 1.27 1.27)) hide)
-    )
-    (property "Datasheet" "~" (at 80.01 38.1 0)
-      (effects (font (size 1.27 1.27)) hide)
-    )
-    (pin "1")
-    (pin "2")
-    (instances
-      (project "RP2040_minimal"
-        (path "/aa156aab-bead-4c71-9076-01087371a0f1"
-          (reference "J2") (unit 1)
-        )
-      )
-      (project "pedalboard-hw"
-        (path "/df521c2a-9827-4355-b809-366f4b88d5d7/d36964e5-9373-47ae-95a7-088f8df77199"
-          (reference "J11") (unit 1)
-        )
-      )
-    )
-  )
   (symbol (lib_id "Device:C_Small") (at 237.49 25.4 0) (unit 1)
     (in_bom yes) (on_board yes) (dnp no)
@@
     )
   )
+  (symbol (lib_id "Switch:SW_Omron_B3FS") (at 80.01 41.91 90) (unit 1)
+    (in_bom yes) (on_board yes) (dnp no)
+    (property "Reference" "SW9" (at 73.66 41.91 0)
+      (effects (font (size 1.27 1.27)))
+    )
+    (property "Value" "Tactile" (at 76.2 41.91 0)
+      (effects (font (size 1.27 1.27)))
+    )
+    (property "Footprint" "Button_Switch_SMD:SW_SPST_B3U-1000P" (at 74.93 41.91 0)
+      (effects (font (size 1.27 1.27)) hide)
+    )
+    (property "Datasheet" "https://omronfs.omron.com/en_US/ecb/products/pdf/en-b3u.pdf" (at 74.93 41.91 0)
+      (effects (font (size 1.27 1.27)) hide)
+    )
+    (property "Supplier" "https://www.digikey.ch/en/products/detail/omron-electronics-inc-emc-div/B3U-1000P/1534338" (at 80.01 41.91 0)
+      (effects (font (size 1.27 1.27)) hide)
+    )
+    (property "Notes" "Boot" (at 80.01 41.91 0)
+      (effects (font (size 1.27 1.27)) hide)
+    )
+    (pin "1")
+    (pin "2")
+    (instances
+      (project "pedalboard-hw"
+        (path "/df521c2a-9827-4355-b809-366f4b88d5d7/d36964e5-9373-47ae-95a7-088f8df77199"
+          (reference "SW9") (unit 1)
+        )
+      )
+    )
+  )
   (symbol (lib_id "Mechanical:MountingHole") (at 148.59 170.18 0) (unit 1)
     (in_bom yes) (on_board yes) (dnp no) (fields_autoplaced)
@@
     )
   )
-  (symbol (lib_id "power:GND") (at 88.9 41.91 0) (unit 1)
+  (symbol (lib_id "power:GND") (at 88.9 50.8 0) (mirror y) (unit 1)
     (in_bom yes) (on_board yes) (dnp no)
-    (property "Reference" "#PWR02" (at 88.9 48.26 0)
+    (property "Reference" "#PWR02" (at 88.9 57.15 0)
       (effects (font (size 1.27 1.27)) hide)
     )
-    (property "Value" "GND" (at 89.027 46.3042 0)
+    (property "Value" "GND" (at 88.773 55.1942 0)
       (effects (font (size 1.27 1.27)))
     )
-    (property "Footprint" "" (at 88.9 41.91 0)
+    (property "Footprint" "" (at 88.9 50.8 0)
       (effects (font (size 1.27 1.27)) hide)
     )
-    (property "Datasheet" "" (at 88.9 41.91 0)
+    (property "Datasheet" "" (at 88.9 50.8 0)
       (effects (font (size 1.27 1.27)) hide)
     )

Commit message: Add tactile button for reset (RP2040)
Parts:
- added SW10: Tactile, Button_Switch_SMD:SW_SPST_B3U-1000P, symbol Switch:SW_Omron_B3FS
- SW9: now not fitted
Connections:
- net GND: now also SW10.1
- net at U3.26 (RUN): now also SW10.2
- no-connect marks 20 -> 19
Changed lines of the file:
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@@
   (junction (at 105.41 50.8) (diameter 0) (color 0 0 0 0)
   )
+  (junction (at 134.62 142.24) (diameter 0) (color 0 0 0 0)
+  )
   (junction (at 266.7 132.08) (diameter 0) (color 0 0 0 0)
   )
@@
   (no_connect (at 228.6 96.52))
   (no_connect (at 228.6 139.7))
-  (no_connect (at 165.1 124.46))
   (no_connect (at 228.6 129.54))
   (no_connect (at 267.97 154.94))
@@
     (stroke (width 0) (type default))
   )
-  (wire (pts (xy 80.01 46.99) (xy 88.9 46.99))
-    (stroke (width 0) (type default))
-  )
   (wire (pts (xy 163.83 180.34) (xy 163.83 191.77))
     (stroke (width 0) (type default))
@@
     (stroke (width 0) (type default))
   )
+  (wire (pts (xy 134.62 142.24) (xy 140.97 142.24))
+    (stroke (width 0) (type default))
+  )
   (wire (pts (xy 127 38.1) (xy 127 40.64))
     (stroke (width 0) (type default))
@@
     (stroke (width 0) (type default))
   )
-  (wire (pts (xy 92.71 30.48) (xy 92.71 41.91))
+  (wire (pts (xy 92.71 34.29) (xy 92.71 41.91))
     (stroke (width 0) (type default))
   )
@@
     (stroke (width 0) (type default))
   )
+  (wire (pts (xy 140.97 135.89) (xy 140.97 142.24))
+    (stroke (width 0) (type default))
+  )
   (wire (pts (xy 49.53 26.67) (xy 59.69 26.67))
     (stroke (width 0) (type default))
@@
     (stroke (width 0) (type default))
   )
+  (wire (pts (xy 140.97 124.46) (xy 165.1 124.46))
+    (stroke (width 0) (type default))
+  )
   (wire (pts (xy 267.97 157.48) (xy 259.08 157.48))
     (stroke (width 0) (type default))
@@
     (stroke (width 0) (type default))
   )
+  (wire (pts (xy 80.01 34.29) (xy 92.71 34.29))
+    (stroke (width 0) (type default))
+  )
   (wire (pts (xy 43.18 97.79) (xy 43.18 86.36))
     (stroke (width 0) (type default))
@@
     (stroke (width 0) (type default))
   )
-  (wire (pts (xy 88.9 46.99) (xy 88.9 50.8))
+  (wire (pts (xy 80.01 46.99) (xy 80.01 50.8))
     (stroke (width 0) (type default))
   )
@@
     (stroke (width 0) (type default))
   )
-  (wire (pts (xy 80.01 30.48) (xy 92.71 30.48))
-    (stroke (width 0) (type default))
-  )
   (wire (pts (xy 22.86 173.99) (xy 54.61 173.99))
     (stroke (width 0) (type default))
@@
     (stroke (width 0) (type default))
   )
+  (wire (pts (xy 134.62 146.05) (xy 134.62 142.24))
+    (stroke (width 0) (type default))
+  )
   (wire (pts (xy 259.08 149.86) (xy 267.97 149.86))
     (stroke (width 0) (type default))
@@
     (stroke (width 0) (type default))
   )
-  (wire (pts (xy 80.01 36.83) (xy 80.01 30.48))
+  (wire (pts (xy 80.01 36.83) (xy 80.01 34.29))
     (stroke (width 0) (type default))
   )
@@
     (stroke (width 0) (type default))
   )
+  (wire (pts (xy 140.97 124.46) (xy 140.97 125.73))
+    (stroke (width 0) (type default))
+  )
   (wire (pts (xy 151.13 81.28) (xy 165.1 81.28))
     (stroke (width 0) (type default))
@@
     (effects (font (size 1.27 1.27)) (justify left bottom))
   )
-  (label "~{USB_BOOT}" (at 82.55 30.48 0) (fields_autoplaced)
+  (label "~{USB_BOOT}" (at 81.28 34.29 0) (fields_autoplaced)
     (effects (font (size 1.27 1.27)) (justify left bottom))
   )
@@
     )
   )
-  (symbol (lib_id "power:GND") (at 134.62 142.24 0) (unit 1)
+  (symbol (lib_id "power:GND") (at 134.62 146.05 0) (unit 1)
     (in_bom yes) (on_board yes) (dnp no) (fields_autoplaced)
-    (property "Reference" "#PWR058" (at 134.62 148.59 0)
+    (property "Reference" "#PWR058" (at 134.62 152.4 0)
       (effects (font (size 1.27 1.27)) hide)
     )
-    (property "Value" "GND" (at 134.62 147.32 0)
+    (property "Value" "GND" (at 134.62 151.13 0)
       (effects (font (size 1.27 1.27)))
     )
-    (property "Footprint" "" (at 134.62 142.24 0)
+    (property "Footprint" "" (at 134.62 146.05 0)
       (effects (font (size 1.27 1.27)) hide)
     )
-    (property "Datasheet" "" (at 134.62 142.24 0)
+    (property "Datasheet" "" (at 134.62 146.05 0)
       (effects (font (size 1.27 1.27)) hide)
     )
@@
     )
   )
+  (symbol (lib_id "Switch:SW_Omron_B3FS") (at 140.97 130.81 90) (unit 1)
+    (in_bom yes) (on_board yes) (dnp yes)
+    (property "Reference" "SW10" (at 134.62 130.81 0)
+      (effects (font (size 1.27 1.27)))
+    )
+    (property "Value" "Tactile" (at 137.16 130.81 0)
+      (effects (font (size 1.27 1.27)))
+    )
+    (property "Footprint" "Button_Switch_SMD:SW_SPST_B3U-1000P" (at 135.89 130.81 0)
+      (effects (font (size 1.27 1.27)) hide)
+    )
+    (property "Datasheet" "https://omronfs.omron.com/en_US/ecb/products/pdf/en-b3u.pdf" (at 135.89 130.81 0)
+      (effects (font (size 1.27 1.27)) hide)
+    )
+    (property "Supplier" "https://www.digikey.ch/en/products/detail/omron-electronics-inc-emc-div/B3U-1000P/1534338" (at 140.97 130.81 0)
+      (effects (font (size 1.27 1.27)) hide)
+    )
+    (property "Notes" "Boot" (at 140.97 130.81 0)
+      (effects (font (size 1.27 1.27)) hide)
+    )
+    (pin "1")
+    (pin "2")
+    (instances
+      (project "pedalboard-hw"
+        (path "/df521c2a-9827-4355-b809-366f4b88d5d7/d36964e5-9373-47ae-95a7-088f8df77199"
+          (reference "SW10") (unit 1)
+        )
+      )
+    )
+  )
   (symbol (lib_id "power:+3V3") (at 120.65 29.21 0) (unit 1)
     (in_bom yes) (on_board yes) (dnp no)
@@
   )
   (symbol (lib_id "Switch:SW_Omron_B3FS") (at 80.01 41.91 90) (unit 1)
-    (in_bom yes) (on_board yes) (dnp no)
+    (in_bom yes) (on_board yes) (dnp yes)
     (property "Reference" "SW9" (at 73.66 41.91 0)
       (effects (font (size 1.27 1.27)))
@@
     )
   )
-  (symbol (lib_id "power:GND") (at 88.9 50.8 0) (mirror y) (unit 1)
+  (symbol (lib_id "power:GND") (at 80.01 50.8 0) (mirror y) (unit 1)
     (in_bom yes) (on_board yes) (dnp no)
-    (property "Reference" "#PWR02" (at 88.9 57.15 0)
+    (property "Reference" "#PWR02" (at 80.01 57.15 0)
       (effects (font (size 1.27 1.27)) hide)
     )
-    (property "Value" "GND" (at 88.773 55.1942 0)
+    (property "Value" "GND" (at 79.883 55.1942 0)
       (effects (font (size 1.27 1.27)))
     )
-    (property "Footprint" "" (at 88.9 50.8 0)
+    (property "Footprint" "" (at 80.01 50.8 0)
       (effects (font (size 1.27 1.27)) hide)
     )
-    (property "Datasheet" "" (at 88.9 50.8 0)
+    (property "Datasheet" "" (at 80.01 50.8 0)
       (effects (font (size 1.27 1.27)) hide)
     )

Commit message: Cleanup part list
Parts:
- C1, C11, C12, C13, C15, C16, C5, C6, C7, C9: Notes 50V/10% -> 10% 16V Ceramic Capacitor X7R
- J23, J24: Notes EXT-MIDI -> (none)
- R2: Notes (none) -> Resistor 10R 1% 63mW
- SW10: Notes Boot -> Reset
Changed lines of the file:
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@@
       (effects (font (size 1.27 1.27)) hide)
     )
-    (property "Notes" "50V/10%" (at 167.64 25.4 0)
+    (property "Notes" "10% 16V Ceramic Capacitor X7R" (at 167.64 25.4 0)
       (effects (font (size 1.27 1.27)) hide)
     )
@@
       (effects (font (size 1.27 1.27)) hide)
     )
-    (property "Notes" "50V/10%" (at 217.17 25.4 0)
+    (property "Notes" "10% 16V Ceramic Capacitor X7R" (at 217.17 25.4 0)
       (effects (font (size 1.27 1.27)) hide)
     )
@@
       (effects (font (size 1.27 1.27)) hide)
     )
-    (property "Notes" "EXT-MIDI" (at 66.04 68.58 0)
+    (property "Notes" "" (at 66.04 68.58 0)
       (effects (font (size 1.27 1.27)) hide)
     )
@@
       (effects (font (size 1.27 1.27)) hide)
     )
-    (property "Notes" "50V/10%" (at 267.97 25.4 0)
+    (property "Notes" "10% 16V Ceramic Capacitor X7R" (at 267.97 25.4 0)
       (effects (font (size 1.27 1.27)) hide)
     )
@@
       (effects (font (size 1.27 1.27)) hide)
     )
-    (property "Notes" "50V/10%" (at 43.18 101.6 0)
+    (property "Notes" "10% 16V Ceramic Capacitor X7R" (at 43.18 101.6 0)
       (effects (font (size 1.27 1.27)) hide)
     )
@@
       (effects (font (size 1.27 1.27)) hide)
     )
-    (property "Notes" "Boot" (at 140.97 130.81 0)
+    (property "Notes" "Reset" (at 140.97 130.81 0)
       (effects (font (size 1.27 1.27)) hide)
     )
@@
       (effects (font (size 1.27 1.27)) hide)
     )
-    (property "Notes" "50V/10%" (at 237.49 25.4 0)
+    (property "Notes" "10% 16V Ceramic Capacitor X7R" (at 237.49 25.4 0)
       (effects (font (size 1.27 1.27)) hide)
     )
@@
       (effects (font (size 1.27 1.27)) hide)
     )
-    (property "Notes" "50V/10%" (at 156.21 25.4 0)
+    (property "Notes" "10% 16V Ceramic Capacitor X7R" (at 156.21 25.4 0)
       (effects (font (size 1.27 1.27)) hide)
     )
@@
     )
     (property "Supplier" "https://www.digikey.ch/de/products/detail/stackpole-electronics-inc/RNCP0805FTD10R0/2240197" (at 46.99 26.67 0)
+      (effects (font (size 1.27 1.27)) hide)
+    )
+    (property "Notes" "Resistor 10R 1% 63mW" (at 46.99 26.67 0)
       (effects (font (size 1.27 1.27)) hide)
     )
@@
       (effects (font (size 1.27 1.27)) hide)
     )
-    (property "Notes" "50V/10%" (at 227.33 25.4 0)
+    (property "Notes" "10% 16V Ceramic Capacitor X7R" (at 227.33 25.4 0)
       (effects (font (size 1.27 1.27)) hide)
     )
@@
       (effects (font (size 1.27 1.27)) hide)
     )
-    (property "Notes" "50V/10%" (at 247.65 25.4 0)
+    (property "Notes" "10% 16V Ceramic Capacitor X7R" (at 247.65 25.4 0)
       (effects (font (size 1.27 1.27)) hide)
     )
@@
       (effects (font (size 1.27 1.27)) hide)
     )
-    (property "Notes" "50V/10%" (at 257.81 25.4 0)
+    (property "Notes" "10% 16V Ceramic Capacitor X7R" (at 257.81 25.4 0)
       (effects (font (size 1.27 1.27)) hide)
     )
@@
       (effects (font (size 1.27 1.27)) hide)
     )
-    (property "Notes" "50V/10%" (at 127 35.56 0)
+    (property "Notes" "10% 16V Ceramic Capacitor X7R" (at 127 35.56 0)
       (effects (font (size 1.27 1.27)) hide)
     )
@@
       (effects (font (size 1.27 1.27)) hide)
     )
-    (property "Notes" "EXT-MIDI" (at 62.23 127 0)
-      (effects (font (size 1.27 1.27)) hide)
-    )
+    (property "Notes" "" (at 62.23 127 0)
+      (effects (font (size 1.27 1.27)) hide)
+    )

Commit message: Fix buttons
Parts:
- SW10, SW9: value Tactile -> Micro Button
- SW3, SW4, SW5, SW6, SW7, SW8: value Tactile -> Tactile Button
Changed lines of the file:
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@@
       (effects (font (size 1.27 1.27)))
     )
-    (property "Value" "Tactile" (at 102.87 177.8 0)
+    (property "Value" "Tactile Button" (at 102.87 177.8 0)
       (effects (font (size 1.27 1.27)))
     )
@@
       (effects (font (size 1.27 1.27)))
     )
-    (property "Value" "Tactile" (at 132.08 177.8 0)
+    (property "Value" "Tactile Button" (at 132.08 177.8 0)
       (effects (font (size 1.27 1.27)))
     )
@@
       (effects (font (size 1.27 1.27)))
     )
-    (property "Value" "Tactile" (at 102.87 162.56 0)
+    (property "Value" "Tactile Button" (at 102.87 162.56 0)
       (effects (font (size 1.27 1.27)))
     )
@@
       (effects (font (size 1.27 1.27)))
     )
-    (property "Value" "Tactile" (at 137.16 130.81 0)
+    (property "Value" "Micro Button" (at 137.16 130.81 0)
       (effects (font (size 1.27 1.27)))
     )
@@
       (effects (font (size 1.27 1.27)))
     )
-    (property "Value" "Tactile" (at 132.08 162.56 0)
+    (property "Value" "Tactile Button" (at 132.08 162.56 0)
       (effects (font (size 1.27 1.27)))
     )
@@
       (effects (font (size 1.27 1.27)))
     )
-    (property "Value" "Tactile" (at 158.75 176.53 0)
+    (property "Value" "Tactile Button" (at 158.75 176.53 0)
       (effects (font (size 1.27 1.27)))
     )
@@
       (effects (font (size 1.27 1.27)))
     )
-    (property "Value" "Tactile" (at 158.75 162.56 0)
+    (property "Value" "Tactile Button" (at 158.75 162.56 0)
       (effects (font (size 1.27 1.27)))
     )
@@
       (effects (font (size 1.27 1.27)))
     )
-    (property "Value" "Tactile" (at 76.2 41.91 0)
-      (effects (font (size 1.27 1.27)))
-    )
+    (property "Value" "Micro Button" (at 76.2 41.91 0)
+      (effects (font (size 1.27 1.27)))
+    )
