File: pico.kicad_sch (KiCad schematic)
At the start: 61 parts, among them J1 Jack 3.5mm, J2 DIN5, J23 JST XH 3, J24 JST XH 3, J3 Jack 3.5mm, J4 DIN5, J5 Jack 6.35mm, J6 Debug, J9 Jack 6.35mm, SW1 Rotary, SW10 Micro Button, SW2 Rotary, SW3 Tactile Button, SW4 Tactile Button, SW5 Tactile Button, SW6 Tactile Button, SW7 Tactile Button, SW8 Tactile Button, SW9 Micro Button, U1 TLP2761, U2 W25Q128JVS, U3 RP2040, Y1 ABLS-12.000MHZ-B4-T

Commit message: Add Stemma Connector for displays
Parts:
- added J28: stemma, Connector_JST:JST_PH_B4B-PH-SM4-TB_1x04-1MP_P2.00mm_Vertical, symbol Connector:Conn_01x04_Pin
Connections:
- net +3V3: now also J28.3 (Pin_3)
- net GND: now also J28.4 (Pin_4)
- net I2C_SDA: now reaches U3.36 (GPIO24)
- net I2C_SDA: now also J28.2 (Pin_2)
- net I2C_SCL: now reaches U3.37 (GPIO25)
- net I2C_SCL: now also J28.1 (Pin_1)
- no-connect marks 19 -> 17
Other:
- moved on the sheet: J5, J9, R4, R5
