File: psu.kicad_sch (KiCad schematic)
At the start: 21 parts, among them J13 Barrel_Jack_MountingPin, Q1 FDS4435BZ, U12 TPS54331

Commit message: Squashed commit of the following:
commit 3fa4ca4d3c5ea62d251efd6d8a974a8ccaef8e6e
Author: Christof Laenzlinger <6319634+laenzlinger@users.noreply.github.com>
Date:   Thu Oct 19 01:43:32 2023 +0200

    Cleanup Silkscreen

commit 95b56afabf9d984d42b570e7dd0e9dc0995e2e0a
Author: Christof Laenzlinger <6319634+laenzlinger@users.noreply.github.com>
Date:   Thu Oct 19 01:37:16 2023 +0200

    Fix ERC and DRC

commit bd76d654c6e0ce2e50bc4bd0303c6b77f3cbeef5
Author: Christof Laenzlinger <6319634+laenzlinger@users.noreply.github.com>
Date:   Thu Oct 19 01:10:46 2023 +0200

    Fix ERC and DRC

commit a0cad1f8b96ac3ca8d87a02e21e40253cfdda0dd
Author: Christof Laenzlinger <6319634+laenzlinger@users.noreply.github.com>
Date:   Thu Oct 19 00:58:14 2023 +0200

    WIP: RP2040 exclude some ERC

commit aeacecf4f2a59ac45e4cb0fbeccc0331a4cb4d99
Author: Christof Laenzlinger <6319634+laenzlinger@users.noreply.github.com>
Date:   Thu Oct 19 00:55:06 2023 +0200

    WIP: RP2040 fix some DRC

commit 55081b7c6b5280d6d649d8c8080d9d887e1852bb
Author: Christof Laenzlinger <6319634+laenzlinger@users.noreply.github.com>
Date:   Thu Oct 19 00:52:29 2023 +0200

    WIP: RP2040 fix some ERC

commit 2468d2f1c68ab1f6ddb7b14c98ba6057067ac39a
Author: Christof Laenzlinger <6319634+laenzlinger@users.noreply.github.com>
Date:   Thu Oct 19 00:43:48 2023 +0200

    WIP: RP2040 fix DRC

commit f8e5d8cf744338d5751e8d0879dfe651a07f16d8
Author: Christof Laenzlinger <6319634+laenzlinger@users.noreply.github.com>
Date:   Wed Oct 18 18:38:41 2023 +0200

    WIP: RP2040 native
Parts:
- added C1, C4: 22u, Capacitor_SMD:C_0805_2012Metric, symbol Device:C
- added D13 (x2): SS34HF, Diode_SMD:D_SMA, symbol Diode:1N5817
- added J1: USB_B_Micro, Connector_USB:USB_Micro-B_Amphenol_10104110_Horizontal, symbol RP2040_minimal-rescue:USB_B_Micro-Connector
- added U1: NCP1117-3.3_SOT223, Package_TO_SOT_SMD:SOT-223-3_TabPin2, symbol Regulator_Linear:NCP1117-3.3_SOT223
Connections:
- net +5VP: now also D13.2 (A)
- net GND: now also C1.2, C4.2, J1.5 (GND), J1.6 (Shield), U1.1 (GND)
- new net +3V3: C4.1, U1.2 (VO)
- new net USB_DN: J1.2 (D-)
- new net USB_DP: J1.3 (D+)
- new net VBUS: D13.2 (A), J1.1 (VBUS)
- new net ored: C1.1, D13.1 (K), D13.1 (K), U1.3 (VI)
- no-connect marks 2 -> 3

Commit message: Add 3d model for USB
Parts:
- J1: footprint Connector_USB:USB_Micro-B_Amphenol_10104110_Horizontal -> Pedalboard Library:USB_Micro-B_Wuerth_614105150721_Vertical
Changed lines of the file:
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@@
       (effects (font (size 1.27 1.27)) (justify right))
     )
-    (property "Footprint" "Connector_USB:USB_Micro-B_Amphenol_10104110_Horizontal" (at 162.56 50.8 0)
+    (property "Footprint" "Pedalboard Library:USB_Micro-B_Wuerth_614105150721_Vertical" (at 162.56 50.8 0)
       (effects (font (size 1.27 1.27)) hide)
     )

Commit message: Add alternative terminal for power
Parts:
- added J26: Screw_Terminal_01x02, TerminalBlock_Phoenix:TerminalBlock_Phoenix_MKDS-1,5-2_1x02_P5.00mm_Horizontal, symbol Connector:Screw_Terminal_01x02
Connections:
- net GND: now also J26.1 (Pin_1)
- net unfused: now also J26.2 (Pin_2)
Changed lines of the file:
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@@
   (junction (at 143.51 120.65) (diameter 0) (color 0 0 0 0)
   )
+  (junction (at 45.72 44.45) (diameter 0) (color 0 0 0 0)
+  )
   (junction (at 173.99 44.45) (diameter 0) (color 0 0 0 0)
   )
@@
   )
   (junction (at 205.74 44.45) (diameter 0) (color 0 0 0 0)
+  )
+  (junction (at 45.72 68.58) (diameter 0) (color 0 0 0 0)
   )
   (junction (at 241.3 44.45) (diameter 0) (color 0 0 0 0)
@@
     (stroke (width 0) (type default))
   )
+  (wire (pts (xy 48.26 44.45) (xy 45.72 44.45))
+    (stroke (width 0) (type default))
+  )
   (wire (pts (xy 99.06 125.73) (xy 100.33 125.73))
     (stroke (width 0) (type default))
@@
     (stroke (width 0) (type default))
   )
+  (wire (pts (xy 35.56 68.58) (xy 45.72 68.58))
+    (stroke (width 0) (type default))
+  )
   (wire (pts (xy 99.06 120.65) (xy 106.68 120.65))
     (stroke (width 0) (type default))
@@
     (stroke (width 0) (type default))
   )
-  (wire (pts (xy 45.72 49.53) (xy 45.72 73.66))
+  (wire (pts (xy 45.72 49.53) (xy 45.72 68.58))
     (stroke (width 0) (type default))
   )
@@
     (stroke (width 0) (type default))
   )
-  (wire (pts (xy 44.45 40.64) (xy 62.23 40.64))
+  (wire (pts (xy 45.72 40.64) (xy 62.23 40.64))
     (stroke (width 0) (type default))
   )
@@
     (stroke (width 0) (type default))
   )
+  (wire (pts (xy 48.26 66.04) (xy 48.26 44.45))
+    (stroke (width 0) (type default))
+  )
   (wire (pts (xy 80.01 40.64) (xy 80.01 52.07))
     (stroke (width 0) (type default))
   )
-  (wire (pts (xy 39.37 44.45) (xy 44.45 44.45))
+  (wire (pts (xy 39.37 44.45) (xy 45.72 44.45))
     (stroke (width 0) (type default))
   )
@@
     (stroke (width 0) (type default))
   )
-  (wire (pts (xy 44.45 44.45) (xy 44.45 40.64))
+  (wire (pts (xy 45.72 44.45) (xy 45.72 40.64))
     (stroke (width 0) (type default))
   )
@@
     (stroke (width 0) (type default))
   )
+  (wire (pts (xy 45.72 68.58) (xy 45.72 73.66))
+    (stroke (width 0) (type default))
+  )
   (wire (pts (xy 73.66 40.64) (xy 80.01 40.64))
     (stroke (width 0) (type default))
@@
   )
   (wire (pts (xy 152.4 119.38) (xy 152.4 120.65))
+    (stroke (width 0) (type default))
+  )
+  (wire (pts (xy 35.56 66.04) (xy 48.26 66.04))
     (stroke (width 0) (type default))
   )
@@
         )
       )
+    )
+  )
+  (symbol (lib_id "Connector:Screw_Terminal_01x02") (at 30.48 68.58 180) (unit 1)
+    (in_bom yes) (on_board yes) (dnp yes) (fields_autoplaced)
+    (property "Reference" "J26" (at 30.48 59.69 0)
+      (effects (font (size 1.27 1.27)))
+    )
+    (property "Value" "Screw_Terminal_01x02" (at 30.48 62.23 0)
+      (effects (font (size 1.27 1.27)))
+    )
+    (property "Footprint" "TerminalBlock_Phoenix:TerminalBlock_Phoenix_MKDS-1,5-2_1x02_P5.00mm_Horizontal" (at 30.48 68.58 0)
+      (effects (font (size 1.27 1.27)) hide)
+    )
+    (property "Datasheet" "~" (at 30.48 68.58 0)
+      (effects (font (size 1.27 1.27)) hide)
+    )
+    (pin "1")
+    (pin "2")
+    (instances
+      (project "pedalboard-hw"
+        (path "/df521c2a-9827-4355-b809-366f4b88d5d7/0d7c87b0-1309-475f-a9d7-edcf3dee5e4e"
+          (reference "J26") (unit 1)
+        )
+      )

Commit message: Geographical re-annotate
Parts:
- renumbered C6 to C2, C13 to C3, C20 to C4, J26 to J5, J13 to J6
Changed lines of the file:
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@@
       (project "pedalboard-hw"
         (path "/df521c2a-9827-4355-b809-366f4b88d5d7/0d7c87b0-1309-475f-a9d7-edcf3dee5e4e"
-          (reference "C12") (unit 1)
+          (reference "C31") (unit 1)
         )
       )
@@
       (project "pedalboard-hw"
         (path "/df521c2a-9827-4355-b809-366f4b88d5d7/0d7c87b0-1309-475f-a9d7-edcf3dee5e4e"
-          (reference "J7") (unit 1)
+          (reference "J10") (unit 1)
         )
       )
@@
   (symbol (lib_id "Connector:Barrel_Jack_Switch") (at 31.75 46.99 0) (mirror x) (unit 1)
     (in_bom yes) (on_board yes) (dnp no)
-    (property "Reference" "J13" (at 41.91 54.61 0)
+    (property "Reference" "J6" (at 41.91 54.61 0)
       (effects (font (size 1.27 1.27)))
     )
@@
       (project "pedalboard-hw"
         (path "/df521c2a-9827-4355-b809-366f4b88d5d7/0d7c87b0-1309-475f-a9d7-edcf3dee5e4e"
-          (reference "J13") (unit 1)
+          (reference "J6") (unit 1)
         )
       )
@@
       (project "pedalboard-hw"
         (path "/df521c2a-9827-4355-b809-366f4b88d5d7/0d7c87b0-1309-475f-a9d7-edcf3dee5e4e"
-          (reference "D7") (unit 1)
+          (reference "D6") (unit 1)
         )
       )
@@
       (project "pedalboard-hw"
         (path "/df521c2a-9827-4355-b809-366f4b88d5d7/0d7c87b0-1309-475f-a9d7-edcf3dee5e4e"
-          (reference "C11") (unit 1)
+          (reference "C25") (unit 1)
         )
       )
@@
         )
         (path "/df521c2a-9827-4355-b809-366f4b88d5d7/0d7c87b0-1309-475f-a9d7-edcf3dee5e4e"
-          (reference "D8") (unit 1)
+          (reference "D5") (unit 1)
         )
       )
@@
       (project "pedalboard-hw"
         (path "/df521c2a-9827-4355-b809-366f4b88d5d7/0d7c87b0-1309-475f-a9d7-edcf3dee5e4e"
-          (reference "C14") (unit 1)
+          (reference "C32") (unit 1)
         )
       )
@@
   (symbol (lib_id "Connector:Screw_Terminal_01x02") (at 30.48 68.58 180) (unit 1)
     (in_bom yes) (on_board yes) (dnp yes) (fields_autoplaced)
-    (property "Reference" "J26" (at 30.48 59.69 0)
+    (property "Reference" "J5" (at 30.48 59.69 0)
       (effects (font (size 1.27 1.27)))
     )
@@
       (project "pedalboard-hw"
         (path "/df521c2a-9827-4355-b809-366f4b88d5d7/0d7c87b0-1309-475f-a9d7-edcf3dee5e4e"
-          (reference "J26") (unit 1)
+          (reference "J5") (unit 1)
         )
       )
@@
       (project "pedalboard-hw"
         (path "/df521c2a-9827-4355-b809-366f4b88d5d7/0d7c87b0-1309-475f-a9d7-edcf3dee5e4e"
-          (reference "C10") (unit 1)
+          (reference "C23") (unit 1)
         )
       )
@@
   (symbol (lib_id "Device:C") (at 80.01 55.88 0) (unit 1)
     (in_bom yes) (on_board yes) (dnp no)
-    (property "Reference" "C6" (at 76.2 53.34 0)
+    (property "Reference" "C2" (at 76.2 53.34 0)
       (effects (font (size 1.27 1.27)) (justify left))
     )
@@
       (project "pedalboard-hw"
         (path "/df521c2a-9827-4355-b809-366f4b88d5d7/0d7c87b0-1309-475f-a9d7-edcf3dee5e4e"
-          (reference "C6") (unit 1)
+          (reference "C2") (unit 1)
         )
       )
@@
   (symbol (lib_id "Device:C_Polarized") (at 96.52 55.88 0) (unit 1)
     (in_bom yes) (on_board yes) (dnp no) (fields_autoplaced)
-    (property "Reference" "C13" (at 100.33 53.721 0)
+    (property "Reference" "C3" (at 100.33 53.721 0)
       (effects (font (size 1.27 1.27)) (justify left))
     )
@@
       (project "pedalboard-hw"
         (path "/df521c2a-9827-4355-b809-366f4b88d5d7/0d7c87b0-1309-475f-a9d7-edcf3dee5e4e"
-          (reference "C13") (unit 1)
+          (reference "C3") (unit 1)
         )
       )
@@
       (project "pedalboard-hw"
         (path "/df521c2a-9827-4355-b809-366f4b88d5d7/0d7c87b0-1309-475f-a9d7-edcf3dee5e4e"
-          (reference "R7") (unit 1)
+          (reference "R12") (unit 1)
         )
       )
@@
       (project "pedalboard-hw"
         (path "/df521c2a-9827-4355-b809-366f4b88d5d7/0d7c87b0-1309-475f-a9d7-edcf3dee5e4e"
-          (reference "C9") (unit 1)
+          (reference "C24") (unit 1)
         )
       )
@@
   (symbol (lib_id "Device:C") (at 73.66 55.88 0) (unit 1)
     (in_bom yes) (on_board yes) (dnp no)
-    (property "Reference" "C20" (at 68.58 53.34 0)
+    (property "Reference" "C4" (at 68.58 53.34 0)
       (effects (font (size 1.27 1.27)) (justify left))
     )
@@
       (project "pedalboard-hw"
         (path "/df521c2a-9827-4355-b809-366f4b88d5d7/0d7c87b0-1309-475f-a9d7-edcf3dee5e4e"
-          (reference "C20") (unit 1)
+          (reference "C4") (unit 1)
         )
       )
@@
       (project "pedalboard-hw"
         (path "/df521c2a-9827-4355-b809-366f4b88d5d7/0d7c87b0-1309-475f-a9d7-edcf3dee5e4e"
-          (reference "C16") (unit 1)
+          (reference "C27") (unit 1)
         )
       )
@@
       (project "pedalboard-hw"
         (path "/df521c2a-9827-4355-b809-366f4b88d5d7/0d7c87b0-1309-475f-a9d7-edcf3dee5e4e"
-          (reference "U6") (unit 1)
+          (reference "U5") (unit 1)
         )
       )
@@
       (project "pedalboard-hw"
         (path "/df521c2a-9827-4355-b809-366f4b88d5d7/0d7c87b0-1309-475f-a9d7-edcf3dee5e4e"
-          (reference "U5") (unit 1)
+          (reference "U6") (unit 1)
         )
       )
@@
       (project "pedalboard-hw"
         (path "/df521c2a-9827-4355-b809-366f4b88d5d7/0d7c87b0-1309-475f-a9d7-edcf3dee5e4e"
-          (reference "C15") (unit 1)
+          (reference "C26") (unit 1)
         )
       )
@@
       (project "pedalboard-hw"
         (path "/df521c2a-9827-4355-b809-366f4b88d5d7/0d7c87b0-1309-475f-a9d7-edcf3dee5e4e"
-          (reference "C7") (unit 1)
+          (reference "C29") (unit 1)
         )
       )
@@
       (project "pedalboard-hw"
         (path "/df521c2a-9827-4355-b809-366f4b88d5d7/0d7c87b0-1309-475f-a9d7-edcf3dee5e4e"
-          (reference "C18") (unit 1)
+          (reference "C19") (unit 1)
         )
       )
@@
         )
         (path "/df521c2a-9827-4355-b809-366f4b88d5d7/0d7c87b0-1309-475f-a9d7-edcf3dee5e4e"
-          (reference "D9") (unit 1)
+          (reference "D8") (unit 1)
         )
       )
@@
       (project "pedalboard-hw"
         (path "/df521c2a-9827-4355-b809-366f4b88d5d7/0d7c87b0-1309-475f-a9d7-edcf3dee5e4e"
-          (reference "C8") (unit 1)
+          (reference "C30") (unit 1)
         )
       )
@@
       (project "pedalboard-hw"
         (path "/df521c2a-9827-4355-b809-366f4b88d5d7/0d7c87b0-1309-475f-a9d7-edcf3dee5e4e"
-          (reference "R8") (unit 1)
+          (reference "R13") (unit 1)
         )
       )
@@
       (project "pedalboard-hw"
         (path "/df521c2a-9827-4355-b809-366f4b88d5d7/0d7c87b0-1309-475f-a9d7-edcf3dee5e4e"
-          (reference "R9") (unit 1)
+          (reference "R14") (unit 1)
         )
       )
@@
       (project "pedalboard-hw"
         (path "/df521c2a-9827-4355-b809-366f4b88d5d7/0d7c87b0-1309-475f-a9d7-edcf3dee5e4e"
-          (reference "C17") (unit 1)
-        )
-      )
+          (reference "C28") (unit 1)
+        )
+      )
