File: psu.kicad_sch (KiCad schematic)
At the start: 38 parts, among them J1 USB_B_Micro, J6 Screw_Terminal_01x02, J7 Barrel_Jack_MountingPin, Q1 FDS4435BZ, U1 NCP1117-3.3_SOT223, U6 AP64501SP-13

Commit message: DNP the USB connector
Parts:
- J1: now not fitted
Changed lines of the file:
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@@
   )
   (symbol (lib_id "pedalboard:USB_B_Micro-Connector") (at 158.75 49.53 0) (unit 1)
-    (in_bom yes) (on_board yes) (dnp no)
+    (in_bom yes) (on_board yes) (dnp yes)
     (property "Reference" "J1" (at 154.94 39.37 0)
       (effects (font (size 1.27 1.27)) (justify right))

Commit message: Show screw terminal instead on 3d view (DNP for jack barrel)
Parts:
- J6: now fitted
- J7: now not fitted
Changed lines of the file:
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@@
   )
   (symbol (lib_id "Connector:Barrel_Jack_Switch") (at 31.75 46.99 0) (mirror x) (unit 1)
-    (in_bom yes) (on_board yes) (dnp no)
+    (in_bom yes) (on_board yes) (dnp yes)
     (property "Reference" "J7" (at 41.91 54.61 0)
       (effects (font (size 1.27 1.27)))
@@
   )
   (symbol (lib_id "Connector:Screw_Terminal_01x02") (at 30.48 68.58 180) (unit 1)
-    (in_bom yes) (on_board yes) (dnp yes) (fields_autoplaced)
+    (in_bom yes) (on_board yes) (dnp no) (fields_autoplaced)
     (property "Reference" "J6" (at 30.48 59.69 0)
       (effects (font (size 1.27 1.27)))

Commit message: Update to V4
Parts:
- renumbered D13 to D4, D13 to D5

Commit message: First version of USB-Hub
Parts:
- removed D4, D5: SS34HF, Diode_SMD:D_SMA, symbol Device:D_Schottky_Small
- removed J1: USB_B_Micro, Pedalboard Library:USB_Micro-B_Wuerth_614105150721_Vertical, symbol pedalboard:USB_B_Micro-Connector
Connections:
- net ored is gone; now on net +5VP: C1.1, U1.3 (VI)
- no-connect marks 2 -> 1

Commit message: Fix symbol warnings
Changed lines of the file:
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@@
 	(wire
 		(pts
-			(xy 42.545 130.81) (xy 42.545 134.62)
+			(xy 48.26 130.81) (xy 48.26 134.62)
 		)
 		(stroke
@@
 	(wire
 		(pts
-			(xy 42.545 130.81) (xy 58.42 130.81)
+			(xy 48.26 130.81) (xy 58.42 130.81)
 		)
 		(stroke
@@
 			)
 		)
-		(property "Description" ""
+		(property "Description" "Power symbol creates a global label with name \"GND\" , ground"
 			(at 135.89 146.05 0)
 			(effects
@@
 			)
 		)
-		(property "Description" ""
+		(property "Description" "Power symbol creates a global label with name \"GND\" , ground"
 			(at 223.52 53.34 0)
 			(effects
@@
 			)
 		)
-		(property "Description" ""
+		(property "Description" "Power symbol creates a global label with name \"GND\" , ground"
 			(at 241.3 54.61 0)
 			(effects
@@
 	)
 	(symbol
-		(lib_name "GND_1")
 		(lib_id "power:GND")
 		(at 45.72 77.47 0)
@@
 			)
 		)
-		(property "Description" ""
+		(property "Description" "Power symbol creates a global label with name \"GND\" , ground"
 			(at 45.72 77.47 0)
 			(effects
@@
 			)
 		)
-		(property "Description" ""
+		(property "Description" "Power symbol creates a global label with name \"GND\" , ground"
 			(at 205.74 54.61 0)
 			(effects
@@
 			)
 		)
-		(property "Description" ""
+		(property "Description" "Power symbol creates a global label with name \"GND\" , ground"
 			(at 245.237 119.38 0)
 			(effects
@@
 			)
 		)
-		(property "Description" ""
+		(property "Description" "Power symbol creates a global label with name \"GND\" , ground"
 			(at 201.295 132.08 0)
 			(effects
@@
 			)
 		)
-		(property "Description" ""
+		(property "Description" "Power symbol creates a global label with name \"+5VP\""
 			(at 254.635 109.22 0)
 			(effects
@@
 	(symbol
 		(lib_id "power:GND")
-		(at 42.545 134.62 0)
+		(at 48.26 134.62 0)
 		(unit 1)
 		(exclude_from_sim no)
@@
 		(dnp no)
 		(property "Reference" "#PWR059"
-			(at 42.545 140.97 0)
+			(at 48.26 140.97 0)
 			(effects
 				(font
@@
 		)
 		(property "Value" "GND"
-			(at 42.672 139.0142 0)
+			(at 48.387 139.0142 0)
 			(effects
 				(font
@@
 		)
 		(property "Footprint" ""
-			(at 42.545 134.62 0)
+			(at 48.26 134.62 0)
 			(effects
 				(font
@@
 		)
 		(property "Datasheet" ""
-			(at 42.545 134.62 0)
+			(at 48.26 134.62 0)
 			(effects
 				(font
@@
 			)
 		)
-		(property "Description" ""
-			(at 42.545 134.62 0)
+		(property "Description" "Power symbol creates a global label with name \"GND\" , ground"
+			(at 48.26 134.62 0)
 			(effects
 				(font
@@
 			)
 		)
-		(property "Description" ""
+		(property "Description" "Power symbol creates a global label with name \"GND\" , ground"
 			(at 201.93 119.38 0)
 			(effects
@@
 			)
 		)
-		(property "Description" ""
+		(property "Description" "Power symbol creates a global label with name \"+3V3\""
 			(at 241.3 43.18 0)
 			(effects
@@
 			)
 		)
-		(property "Description" ""
+		(property "Description" "Power symbol creates a global label with name \"+5VP\""
 			(at 195.58 26.67 0)
 			(effects

Commit message: Fix warngings
Parts:
- C33: symbol Device:CP -> Device:C_Polarized
Other:
- moved on the sheet: C33, TP2, TP3

Commit message: Fix new errors
Changed lines of the file:
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@@
+	)
+	(symbol
+		(lib_id "power:PWR_FLAG")
+		(at 96.52 40.64 0)
+		(unit 1)
+		(exclude_from_sim no)
+		(in_bom yes)
+		(on_board yes)
+		(dnp no)
+		(fields_autoplaced yes)
+		(property "Reference" "#FLG02"
+			(at 96.52 38.735 0)
+			(effects
+				(font
+					(size 1.27 1.27)
+				)
+				(hide yes)
+			)
+		)
+		(property "Value" "PWR_FLAG"
+			(at 96.52 35.56 0)
+			(effects
+				(font
+					(size 1.27 1.27)
+				)
+			)
+		)
+		(property "Footprint" ""
+			(at 96.52 40.64 0)
+			(effects
+				(font
+					(size 1.27 1.27)
+				)
+				(hide yes)
+			)
+		)
+		(property "Datasheet" "~"
+			(at 96.52 40.64 0)
+			(effects
+				(font
+					(size 1.27 1.27)
+				)
+				(hide yes)
+			)
+		)
+		(property "Description" "Special symbol for telling ERC where power comes from"
+			(at 96.52 40.64 0)
+			(effects
+				(font
+					(size 1.27 1.27)
+				)
+				(hide yes)
+			)
+		)
+		(pin "1"
+		)
+		(instances
+			(project ""
+				(path "/df521c2a-9827-4355-b809-366f4b88d5d7/0d7c87b0-1309-475f-a9d7-edcf3dee5e4e"
+					(reference "#FLG02")
+					(unit 1)
+				)
+			)
+		)
 	)
 	(symbol

Commit message: Use stadard KiCAD inductor symbol
Parts:
- L5: symbol pspice:INDUCTOR -> Device:L
Changed lines of the file:
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@@
-	(wire
-		(pts
-			(xy 170.18 109.22) (xy 172.72 109.22)
-		)
-		(stroke
-			(width 0)
-			(type solid)
-		)
-	)
 	(wire
 		(pts
@@
 		)
 	)
+	(wire
+		(pts
+			(xy 167.64 109.22) (xy 172.72 109.22)
+		)
+		(stroke
+			(width 0)
+			(type default)
+		)
+	)
 	(polyline
 		(pts
@@
 	(wire
 		(pts
-			(xy 144.78 109.22) (xy 157.48 109.22)
+			(xy 144.78 109.22) (xy 160.02 109.22)
 		)
 		(stroke
@@
 	)
 	(symbol
-		(lib_id "pspice:INDUCTOR")
-		(at 163.83 109.22 0)
+		(lib_id "Device:L")
+		(at 163.83 109.22 90)
 		(unit 1)
 		(exclude_from_sim no)
@@
 		(dnp no)
 		(property "Reference" "L5"
-			(at 163.83 103.759 0)
+			(at 161.036 111.252 90)
 			(effects
 				(font
@@
 		)
 		(property "Value" "SRN6045TA-3R3Y"
-			(at 163.83 106.0704 0)
-			(effects
-				(font
+			(at 163.83 106.426 90)
+			(effects
+				(font
