File: leds.kicad_sch (KiCad schematic)
At the start: 29 parts, among them J18 LED-Ring, J19 LED-Ring, J20 LED-Ring, J21 LED-Ring, J22 LED-Ring, J23 LED-Ring, J4 RGB_LED_EXT, U3 74AHCT1G32SE-7

Commit message: Use SMD components for MIDI
Parts:
- C10, C11, C2, C3, C4, C5, C6, C7, C8, C9: footprint Capacitor_THT:C_Disc_D3.0mm_W1.6mm_P2.50mm -> Capacitor_SMD:C_0805_2012Metric; Supplier https://www.digikey.ch/en/products/detail/vishay-beyschlag-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 -> https://www.digikey.ch/de/products/detail/kyocera-avx/KGM21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
- R5: footprint Resistor_THT:R_Axial_DIN0207_L6.3mm_D2.5mm_P10.16mm_Horizontal -> Resistor_SMD:R_0805_2012Metric; Supplier https://www.digikey.ch/de/products/detail/koa-speer-electro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 -> https://www.digikey.ch/de/products/detail/stackpole-electro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
- U3: Package SOT-353 Diodes Inc. -> (none); Purchase-URL https://www.snapeda.com/api/url_track_click_mouser/?unipart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 -> (none); SUPPLIER Diodes INC -> (none); SnapEDA_Link https://www.snapeda.com/parts/74AHCT1G32SE-7/Diodes+Inc./vi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 -> (none); Supplier (none) -> https://www.digikey.ch/de/products/detail/diodes-incorporat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

Commit message: Replace LEDs with SMD part
Parts:
- D1, D10, D2, D3, D4, D5, D6, D7, D8, D9: value NEOPIX -> SK6812; footprint Pedalboard Library:LED_D5.0mm-NeoPixel -> LED_SMD:LED_SK6812_PLCC4_5.0x5.0mm_P3.2mm; symbol LED:NeoPixel_THT -> LED:SK6812; Supplier https://www.digikey.ch/de/products/detail/sparkfun-electron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 -> https://www.digikey.ch/de/products/detail/adafruit-industri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
Connections:
- net +5VP: now also D1.3 (VDD), D10.3 (VDD), D2.3 (VDD), D3.3 (VDD), D4.3 (VDD), D5.3 (VDD), D6.3 (VDD), D7.3 (VDD), D8.3 (VDD), D9.3 (VDD); no longer D1.2 (VDD), D10.2 (VDD), D2.2 (VDD), D3.2 (VDD), D4.2 (VDD), D5.2 (VDD), D6.2 (VDD), D7.2 (VDD), D8.2 (VDD), D9.2 (VDD)
- net GND: now also D1.1 (VSS), D10.1 (VSS), D2.1 (VSS), D3.1 (VSS), D4.1 (VSS), D5.1 (VSS), D6.1 (VSS), D7.1 (VSS), D8.1 (VSS), D9.1 (VSS); no longer D1.3 (GND), D10.3 (GND), D2.3 (GND), D3.3 (GND), D4.3 (GND), D5.3 (GND), D6.3 (GND), D7.3 (GND), D8.3 (GND), D9.3 (GND)
- net at D1.4 (DOUT): now also D2.2 (DIN); no longer D2.1 (DIN)
- net at D2.4 (DOUT): now also D3.2 (DIN); no longer D3.1 (DIN)
- net at D5.4 (DOUT), J18.4 (Pin_4), J19.3 (Pin_3): now also D6.2 (DIN); no longer D6.1 (DIN)
- net at D6.4 (DOUT), J19.4 (Pin_4), J20.3 (Pin_3): now also D7.2 (DIN); no longer D7.1 (DIN)
- net at D4.4 (DOUT), J18.3 (Pin_3): now also D5.2 (DIN); no longer D5.1 (DIN)
- net at D7.4 (DOUT), J20.4 (Pin_4), J21.3 (Pin_3): now also D8.2 (DIN); no longer D8.1 (DIN)
- net at D8.4 (DOUT), J21.4 (Pin_4), J22.3 (Pin_3): now also D9.2 (DIN); no longer D9.1 (DIN)
- net at D3.4 (DOUT): now also D4.2 (DIN); no longer D4.1 (DIN)
- net at U3.4 (Y): now also D1.2 (DIN); no longer D1.1 (DIN)
- net at D9.4 (DOUT), J22.4 (Pin_4), J23.3 (Pin_3): now also D10.2 (DIN); no longer D10.1 (DIN)

Commit message: Replace reverse power diode with MOSFET
Parts:
- U3: Check_prices https://www.snapeda.com/parts/74AHCT1G32SE-7/Diodes+Inc./vi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 -> (none)
Changed lines of the file:
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@@
-      (effects (font (size 1.27 1.27)) (justify bottom) hide)
-    )
-    (property "Check_prices" "https://www.snapeda.com/parts/74AHCT1G32SE-7/Diodes+Inc./view-part/?ref=eda" (at 100.33 50.8 0)
       (effects (font (size 1.27 1.27)) (justify bottom) hide)
     )

Commit message: Replace capacitors for PSU with SMD components
Parts:
- R5: value 470 -> 220
Changed lines of the file:
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@@
   (symbol (lib_id "Device:R") (at 66.04 53.34 90) (unit 1)
     (in_bom yes) (on_board yes) (dnp no) (fields_autoplaced)
-    (property "Reference" "R5" (at 66.04 48.26 90)
+    (property "Reference" "R5" (at 66.04 46.99 90)
       (effects (font (size 1.27 1.27)))
     )
-    (property "Value" "470" (at 66.04 50.8 90)
+    (property "Value" "220" (at 66.04 49.53 90)
       (effects (font (size 1.27 1.27)))
     )
@@
         )
         (path "/df521c2a-9827-4355-b809-366f4b88d5d7/539b926e-3ef4-477a-b921-49e2b2b26dfc"
-          (reference "R5") (unit 1)
+          (reference "R4") (unit 1)
         )
       )

Commit message: Fix ERC errors
Parts:
- U3: footprint Package_TO_SOT_SMD:SOT-353_SC-70-5 -> Pedalboard Library:SOT65P210X110-5N
Changed lines of the file:
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@@
         )
         (path "/df521c2a-9827-4355-b809-366f4b88d5d7/539b926e-3ef4-477a-b921-49e2b2b26dfc"
-          (reference "R4") (unit 1)
+          (reference "R5") (unit 1)
         )
       )
@@
       (effects (font (size 1.27 1.27)))
     )
-    (property "Footprint" "Package_TO_SOT_SMD:SOT-353_SC-70-5" (at 100.33 50.8 0)
+    (property "Footprint" "Pedalboard Library:SOT65P210X110-5N" (at 100.33 50.8 0)
       (effects (font (size 1.27 1.27)) (justify bottom) hide)
     )

Commit message: Started to cleanup routing
Parts:
- removed C10, C11, C6, C7, C8, C9: 100nF, Capacitor_SMD:C_0805_2012Metric, symbol Device:C
- removed D10, D5, D6, D7, D8, D9: SK6812, LED_SMD:LED_SK6812_PLCC4_5.0x5.0mm_P3.2mm, symbol LED:SK6812
Other:
- moved on the sheet: J21, J23

Commit message: Resize PCB
Parts:
- J4: footprint Connector_PinHeader_2.54mm:PinHeader_1x03_P2.54mm_Horizontal -> Connector_JST:JST_XH_B3B-XH-A_1x03_P2.50mm_Vertical
Changed lines of the file:
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@@
       (effects (font (size 1.27 1.27)))
     )
-    (property "Footprint" "Connector_PinHeader_2.54mm:PinHeader_1x03_P2.54mm_Horizontal" (at 265.43 143.51 0)
+    (property "Footprint" "Connector_JST:JST_XH_B3B-XH-A_1x03_P2.50mm_Vertical" (at 265.43 143.51 0)
       (effects (font (size 1.27 1.27)) hide)
     )

Commit message: Driver for LED
Parts:
- U3: footprint Pedalboard Library:SOT65P210X110-5N -> SOT-353_SC-70-5
Changed lines of the file:
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@@
       (effects (font (size 1.27 1.27)))
     )
-    (property "Footprint" "Pedalboard Library:SOT65P210X110-5N" (at 100.33 50.8 0)
+    (property "Footprint" "SOT-353_SC-70-5" (at 100.33 50.8 0)
       (effects (font (size 1.27 1.27)) (justify bottom) hide)
     )
