File: leds.kicad_sch (KiCad schematic)
At the start: 15 parts, among them J11 LED-Ring, J13 LED-Ring, J14 LED-Ring, J19 LED-Ring, J21 LED-Ring, J22 LED-Ring, J27 LED-Ring, J4 JST XH 3, J8 LED-Ring, U2 74AHCT1G32SE-7

Commit message: Stemma Spec for LED Out
Parts:
- J4: value JST XH 3 -> STEMMA LED; footprint Connector_JST:JST_XH_B3B-XH-A_1x03_P2.50mm_Vertical -> Connector_JST:JST_PH_B3B-PH-K_1x03_P2.00mm_Vertical
Connections:
- net +5VP: now also J4.2 (Pin_2); no longer J4.3 (Pin_3)
- net at J21.4 (Pin_4): now also J4.3 (Pin_3); no longer J4.2 (Pin_2)
Other:
- moved on the sheet: J4
Changed lines of the file:
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@@
   (junction (at 121.92 151.13) (diameter 0) (color 0 0 0 0)
   )
+  (junction (at 207.01 151.13) (diameter 0) (color 0 0 0 0)
+  )
   (junction (at 157.48 25.4) (diameter 0) (color 0 0 0 0)
   )
   (junction (at 123.19 109.22) (diameter 0) (color 0 0 0 0)
   )
+  (junction (at 76.2 151.13) (diameter 0) (color 0 0 0 0)
+  )
+  (junction (at 146.05 48.26) (diameter 0) (color 0 0 0 0)
+  )
+  (junction (at 123.19 83.82) (diameter 0) (color 0 0 0 0)
+  )
+  (junction (at 121.92 125.73) (diameter 0) (color 0 0 0 0)
+  )
+  (junction (at 146.05 67.31) (diameter 0) (color 0 0 0 0)
+  )
+  (junction (at 166.37 125.73) (diameter 0) (color 0 0 0 0)
+  )
+  (junction (at 77.47 109.22) (diameter 0) (color 0 0 0 0)
+  )
+  (junction (at 76.2 125.73) (diameter 0) (color 0 0 0 0)
+  )
   (junction (at 207.01 125.73) (diameter 0) (color 0 0 0 0)
   )
-  (junction (at 76.2 151.13) (diameter 0) (color 0 0 0 0)
-  )
-  (junction (at 146.05 48.26) (diameter 0) (color 0 0 0 0)
-  )
-  (junction (at 123.19 83.82) (diameter 0) (color 0 0 0 0)
-  )
-  (junction (at 121.92 125.73) (diameter 0) (color 0 0 0 0)
-  )
-  (junction (at 146.05 67.31) (diameter 0) (color 0 0 0 0)
-  )
-  (junction (at 166.37 125.73) (diameter 0) (color 0 0 0 0)
-  )
-  (junction (at 77.47 109.22) (diameter 0) (color 0 0 0 0)
-  )
-  (junction (at 76.2 125.73) (diameter 0) (color 0 0 0 0)
-  )
   (junction (at 166.37 83.82) (diameter 0) (color 0 0 0 0)
   )
@@
   (junction (at 77.47 83.82) (diameter 0) (color 0 0 0 0)
   )
-  (junction (at 207.01 151.13) (diameter 0) (color 0 0 0 0)
-  )
   (junction (at 165.1 33.02) (diameter 0) (color 0 0 0 0)
   )
@@
     (stroke (width 0) (type default))
   )
+  (wire (pts (xy 260.35 151.13) (xy 207.01 151.13))
+    (stroke (width 0) (type default))
+  )
   (wire (pts (xy 119.38 129.54) (xy 119.38 130.81))
     (stroke (width 0) (type default))
@@
     (stroke (width 0) (type default))
   )
-  (wire (pts (xy 255.27 151.13) (xy 260.35 146.05))
-    (stroke (width 0) (type default))
-  )
   (wire (pts (xy 82.55 60.96) (xy 82.55 67.31))
     (stroke (width 0) (type default))
@@
     (stroke (width 0) (type default))
   )
+  (wire (pts (xy 204.47 146.05) (xy 204.47 142.24))
+    (stroke (width 0) (type default))
+  )
   (wire (pts (xy 63.5 87.63) (xy 74.93 87.63))
     (stroke (width 0) (type default))
@@
     (stroke (width 0) (type default))
   )
-  (wire (pts (xy 204.47 143.51) (xy 260.35 143.51))
-    (stroke (width 0) (type default))
-  )
   (wire (pts (xy 121.92 151.13) (xy 166.37 151.13))
     (stroke (width 0) (type default))
@@
     (stroke (width 0) (type default))
   )
-  (wire (pts (xy 255.27 128.27) (xy 260.35 140.97))
-    (stroke (width 0) (type default))
-  )
   (wire (pts (xy 128.27 58.42) (xy 138.43 58.42))
     (stroke (width 0) (type default))
@@
     (stroke (width 0) (type default))
   )
+  (wire (pts (xy 207.01 125.73) (xy 228.6 125.73))
+    (stroke (width 0) (type default))
+  )
   (wire (pts (xy 123.19 109.22) (xy 166.37 109.22))
     (stroke (width 0) (type default))
@@
     (stroke (width 0) (type default))
   )
+  (wire (pts (xy 260.35 146.05) (xy 204.47 146.05))
+    (stroke (width 0) (type default))
+  )
   (wire (pts (xy 77.47 113.03) (xy 77.47 109.22))
     (stroke (width 0) (type default))
@@
     (stroke (width 0) (type default))
   )
-  (wire (pts (xy 255.27 128.27) (xy 255.27 125.73))
-    (stroke (width 0) (type default))
-  )
   (wire (pts (xy 157.48 25.4) (xy 165.1 25.4))
     (stroke (width 0) (type default))
@@
     (stroke (width 0) (type default))
   )
+  (wire (pts (xy 228.6 148.59) (xy 228.6 125.73))
+    (stroke (width 0) (type default))
+  )
   (wire (pts (xy 166.37 125.73) (xy 166.37 129.54))
     (stroke (width 0) (type default))
@@
     (stroke (width 0) (type default))
   )
-  (wire (pts (xy 204.47 142.24) (xy 204.47 143.51))
-    (stroke (width 0) (type default))
-  )
   (wire (pts (xy 208.28 83.82) (xy 208.28 86.36))
     (stroke (width 0) (type default))
@@
     (stroke (width 0) (type default))
   )
-  (wire (pts (xy 207.01 125.73) (xy 255.27 125.73))
-    (stroke (width 0) (type default))
-  )
-  (wire (pts (xy 207.01 151.13) (xy 255.27 151.13))
+  (wire (pts (xy 260.35 148.59) (xy 228.6 148.59))
     (stroke (width 0) (type default))
   )
@@
     )
   )
-  (symbol (lib_id "Connector:Conn_01x03_Pin") (at 265.43 143.51 180) (unit 1)
+  (symbol (lib_id "Connector:Conn_01x03_Pin") (at 265.43 148.59 180) (unit 1)
     (in_bom yes) (on_board yes) (dnp no)
-    (property "Reference" "J4" (at 265.43 148.59 0)
-      (effects (font (size 1.27 1.27)))
-    )
-    (property "Value" "JST XH 3" (at 266.7 135.89 0)
-      (effects (font (size 1.27 1.27)))
-    )
-    (property "Footprint" "Connector_JST:JST_XH_B3B-XH-A_1x03_P2.50mm_Vertical" (at 265.43 143.51 0)
-      (effects (font (size 1.27 1.27)) hide)
-    )
-    (property "Datasheet" "https://app.adam-tech.com/products/download/data_sheet/240508/25sh-b-xx-ts-data-sheet.pdf" (at 265.43 143.51 0)
-      (effects (font (size 1.27 1.27)) hide)
-    )
-    (property "Supplier" "https://www.digikey.ch/de/products/detail/adam-tech/25SH-B-03-TS/9830417" (at 265.43 143.51 0)
-      (effects (font (size 1.27 1.27)) hide)
-    )
-    (property "Notes" "" (at 265.43 143.51 0)
-      (effects (font (size 1.27 1.27)) hide)
-    )
+    (property "Reference" "J4" (at 265.43 153.67 0)
+      (effects (font (size 1.27 1.27)))
+    )
+    (property "Value" "STEMMA LED" (at 266.7 140.97 0)
+      (effects (font (size 1.27 1.27)))
+    )
+    (property "Footprint" "Connector_JST:JST_PH_B3B-PH-K_1x03_P2.00mm_Vertical" (at 265.43 148.59 0)
+      (effects (font (size 1.27 1.27)) hide)
+    )
+    (property "Datasheet" "https://app.adam-tech.com/products/download/data_sheet/240508/25sh-b-xx-ts-data-sheet.pdf" (at 265.43 148.59 0)
+      (effects (font (size 1.27 1.27)) hide)
+    )
+    (property "Supplier" "https://www.digikey.ch/de/products/detail/adam-tech/25SH-B-03-TS/9830417" (at 265.43 148.59 0)
+      (effects (font (size 1.27 1.27)) hide)
+    )
+    (property "Notes" "" (at 265.43 148.59 0)
+      (effects (font (size 1.27 1.27)) hide)
+    )

Commit message: Geographical Reannotate
Parts:
- renumbered J11 to J10, J27 to J13, J13 to J15, J14 to J17, J19 to J21, J21 to J23, J22 to J24, J8 to J9, U2 to U1
Changed lines of the file:
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@@
         )
         (path "/df521c2a-9827-4355-b809-366f4b88d5d7/539b926e-3ef4-477a-b921-49e2b2b26dfc"
-          (reference "D3") (unit 1)
+          (reference "D2") (unit 1)
         )
       )
@@
   (symbol (lib_id "Connector_Generic:Conn_02x02_Odd_Even") (at 123.19 91.44 270) (unit 1)
     (in_bom yes) (on_board yes) (dnp no) (fields_autoplaced)
-    (property "Reference" "J13" (at 125.73 92.075 90)
+    (property "Reference" "J15" (at 125.73 92.075 90)
       (effects (font (size 1.27 1.27)) (justify left))
     )
@@
       (project "pedalboard-hw"
         (path "/df521c2a-9827-4355-b809-366f4b88d5d7/539b926e-3ef4-477a-b921-49e2b2b26dfc"
-          (reference "J13") (unit 1)
+          (reference "J15") (unit 1)
         )
       )
@@
         )
         (path "/df521c2a-9827-4355-b809-366f4b88d5d7/539b926e-3ef4-477a-b921-49e2b2b26dfc"
-          (reference "D4") (unit 1)
+          (reference "D3") (unit 1)
         )
       )
@@
   (symbol (lib_id "Connector_Generic:Conn_02x02_Odd_Even") (at 166.37 92.71 270) (unit 1)
     (in_bom yes) (on_board yes) (dnp no) (fields_autoplaced)
-    (property "Reference" "J22" (at 168.91 93.345 90)
+    (property "Reference" "J24" (at 168.91 93.345 90)
       (effects (font (size 1.27 1.27)) (justify left))
     )
@@
       (project "pedalboard-hw"
         (path "/df521c2a-9827-4355-b809-366f4b88d5d7/539b926e-3ef4-477a-b921-49e2b2b26dfc"
-          (reference "J22") (unit 1)
+          (reference "J24") (unit 1)
         )
       )
@@
         )
         (path "/df521c2a-9827-4355-b809-366f4b88d5d7/539b926e-3ef4-477a-b921-49e2b2b26dfc"
-          (reference "C12") (unit 1)
+          (reference "C11") (unit 1)
         )
       )
@@
         )
         (path "/df521c2a-9827-4355-b809-366f4b88d5d7/539b926e-3ef4-477a-b921-49e2b2b26dfc"
-          (reference "J26") (unit 1)
+          (reference "J28") (unit 1)
         )
       )
@@
   (symbol (lib_id "Connector_Generic:Conn_02x02_Odd_Even") (at 76.2 134.62 270) (unit 1)
     (in_bom yes) (on_board yes) (dnp no) (fields_autoplaced)
-    (property "Reference" "J14" (at 78.74 135.255 90)
+    (property "Reference" "J17" (at 78.74 135.255 90)
       (effects (font (size 1.27 1.27)) (justify left))
     )
@@
       (project "pedalboard-hw"
         (path "/df521c2a-9827-4355-b809-366f4b88d5d7/539b926e-3ef4-477a-b921-49e2b2b26dfc"
-          (reference "J14") (unit 1)
+          (reference "J17") (unit 1)
         )
       )
@@
         )
         (path "/df521c2a-9827-4355-b809-366f4b88d5d7/539b926e-3ef4-477a-b921-49e2b2b26dfc"
-          (reference "R6") (unit 1)
+          (reference "R7") (unit 1)
         )
       )
@@
   (symbol (lib_id "Connector_Generic:Conn_02x02_Odd_Even") (at 166.37 134.62 270) (unit 1)
     (in_bom yes) (on_board yes) (dnp no) (fields_autoplaced)
-    (property "Reference" "J8" (at 168.91 135.255 90)
+    (property "Reference" "J9" (at 168.91 135.255 90)
       (effects (font (size 1.27 1.27)) (justify left))
     )
@@
       (project "pedalboard-hw"
         (path "/df521c2a-9827-4355-b809-366f4b88d5d7/539b926e-3ef4-477a-b921-49e2b2b26dfc"
-          (reference "J8") (unit 1)
+          (reference "J9") (unit 1)
         )
       )
@@
   (symbol (lib_id "Connector_Generic:Conn_02x02_Odd_Even") (at 121.92 135.89 270) (unit 1)
     (in_bom yes) (on_board yes) (dnp no) (fields_autoplaced)
-    (property "Reference" "J11" (at 124.46 136.525 90)
+    (property "Reference" "J10" (at 124.46 136.525 90)
       (effects (font (size 1.27 1.27)) (justify left))
     )
@@
       (project "pedalboard-hw"
         (path "/df521c2a-9827-4355-b809-366f4b88d5d7/539b926e-3ef4-477a-b921-49e2b2b26dfc"
-          (reference "J11") (unit 1)
+          (reference "J10") (unit 1)
         )
       )
@@
   (symbol (lib_id "Connector_Generic:Conn_02x02_Odd_Even") (at 207.01 134.62 270) (unit 1)
     (in_bom yes) (on_board yes) (dnp no) (fields_autoplaced)
-    (property "Reference" "J21" (at 209.55 135.255 90)
+    (property "Reference" "J23" (at 209.55 135.255 90)
       (effects (font (size 1.27 1.27)) (justify left))
     )
@@
       (project "pedalboard-hw"
         (path "/df521c2a-9827-4355-b809-366f4b88d5d7/539b926e-3ef4-477a-b921-49e2b2b26dfc"
-          (reference "J21") (unit 1)
+          (reference "J23") (unit 1)
         )
       )
@@
   (symbol (lib_id "Connector_Generic:Conn_02x02_Odd_Even") (at 77.47 92.71 270) (unit 1)
     (in_bom yes) (on_board yes) (dnp no) (fields_autoplaced)
-    (property "Reference" "J27" (at 80.01 93.345 90)
+    (property "Reference" "J13" (at 80.01 93.345 90)
       (effects (font (size 1.27 1.27)) (justify left))
     )
@@
       (project "pedalboard-hw"
         (path "/df521c2a-9827-4355-b809-366f4b88d5d7/539b926e-3ef4-477a-b921-49e2b2b26dfc"
-          (reference "J27") (unit 1)
+          (reference "J13") (unit 1)
         )
       )
@@
   (symbol (lib_id "pedalboard:74AHCT1G32SE-7") (at 100.33 50.8 0) (unit 1)
     (in_bom yes) (on_board yes) (dnp no) (fields_autoplaced)
-    (property "Reference" "U2" (at 100.33 38.1 0)
+    (property "Reference" "U1" (at 100.33 38.1 0)
       (effects (font (size 1.27 1.27)))
     )
@@
       (project "pedalboard-hw"
         (path "/df521c2a-9827-4355-b809-366f4b88d5d7/539b926e-3ef4-477a-b921-49e2b2b26dfc"
-          (reference "U2") (unit 1)
+          (reference "U1") (unit 1)
         )
       )
@@
   (symbol (lib_id "Connector_Generic:Conn_02x02_Odd_Even") (at 208.28 91.44 270) (unit 1)
     (in_bom yes) (on_board yes) (dnp no) (fields_autoplaced)
-    (property "Reference" "J19" (at 210.82 92.075 90)
+    (property "Reference" "J21" (at 210.82 92.075 90)
       (effects (font (size 1.27 1.27)) (justify left))
     )
@@
       (project "pedalboard-hw"
         (path "/df521c2a-9827-4355-b809-366f4b88d5d7/539b926e-3ef4-477a-b921-49e2b2b26dfc"
-          (reference "J19") (unit 1)
-        )
-      )
+          (reference "J21") (unit 1)
+        )
+      )

Commit message: Improve BOM
Parts:
- J4: Supplier https://www.digikey.ch/de/products/detail/adam-tech/25SH-B-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 -> https://www.digikey.com/en/products/detail/jst-sales-americ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
Changed lines of the file:
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@@
       (effects (font (size 1.27 1.27)) hide)
     )
-    (property "Datasheet" "https://app.adam-tech.com/products/download/data_sheet/240508/25sh-b-xx-ts-data-sheet.pdf" (at 265.43 148.59 0)
+    (property "Datasheet" "https://www.jst-mfg.com/product/pdf/eng/ePH.pdf" (at 265.43 148.59 0)
       (effects (font (size 1.27 1.27)) hide)
     )
-    (property "Supplier" "https://www.digikey.ch/de/products/detail/adam-tech/25SH-B-03-TS/9830417" (at 265.43 148.59 0)
+    (property "Supplier" "https://www.digikey.com/en/products/detail/jst-sales-america-inc/B3B-PH-K-S/926612" (at 265.43 148.59 0)
       (effects (font (size 1.27 1.27)) hide)
     )

Commit message: Improve BOM (JST)
Parts:
- J4: value STEMMA LED -> JST PH 3
Changed lines of the file:
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@@
       (effects (font (size 1.27 1.27)))
     )
-    (property "Value" "STEMMA LED" (at 266.7 140.97 0)
+    (property "Value" "JST PH 3" (at 266.7 140.97 0)
       (effects (font (size 1.27 1.27)))
     )

Commit message: DNP LED out
Parts:
- J4: now not fitted
Changed lines of the file:
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@@
   )
   (symbol (lib_id "Connector:Conn_01x03_Pin") (at 265.43 148.59 180) (unit 1)
-    (in_bom yes) (on_board yes) (dnp no)
+    (in_bom yes) (on_board yes) (dnp yes)
     (property "Reference" "J4" (at 265.43 153.67 0)
       (effects (font (size 1.27 1.27)))
