File: connect.kicad_sch (KiCad schematic)
At the start: 1 part

Commit message: Improve BOM: Same components have same value
Parts:
- Module1: value ComputeModule4-CM4 -> CM4
Changed lines of the file:
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@@
       (effects (font (size 1.27 1.27)))
     )
-    (property "Value" "ComputeModule4-CM4" (at 119.38 29.21 0)
+    (property "Value" "CM4" (at 119.38 29.21 0)
       (effects (font (size 1.27 1.27)))
     )

Commit message: Cleanup Supplier link for CM4
Parts:
- Module1: Supplier https://www.digikey.ch/de/products/detail/hirose-electric-co-ltd/DF40C-100DS-0-4V-51/1969476?utm_adgroup=Connectors%2C%20Interconnects&utm_source=google&utm_medium=cpc&utm_campaign=Dynamic%20Search_DE_Product&utm_term=&productid=&utm_content=Connectors%2C%20Interconnects&utm_id=go_cmp-225090269_adg-23739644429_ad-668713893261_dsa-40817298870_dev-c_ext-_prd-_sig-EAIaIQobChMIkc2bqtWCggMV_4RoCR2sgwV-EAAYASAAEgLIUvD_BwE&gclid=EAIaIQobChMIkc2bqtWCggMV_4RoCR2sgwV-EAAYASAAEgLIUvD_BwE -> https://www.digikey.ch/de/products/detail/hirose-electric-co-ltd/DF40C-100DS-0-4V-51/1969476
Changed lines of the file:
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@@
       (effects (font (size 1.27 1.27)) hide)
     )
-    (property "Supplier" "https://www.digikey.ch/de/products/detail/hirose-electric-co-ltd/DF40C-100DS-0-4V-51/1969476?utm_adgroup=Connectors%2C%20Interconnects&utm_source=google&utm_medium=cpc&utm_campaign=Dynamic%20Search_DE_Product&utm_term=&productid=&utm_content=Connectors%2C%20Interconnects&utm_id=go_cmp-225090269_adg-23739644429_ad-668713893261_dsa-40817298870_dev-c_ext-_prd-_sig-EAIaIQobChMIkc2bqtWCggMV_4RoCR2sgwV-EAAYASAAEgLIUvD_BwE&gclid=EAIaIQobChMIkc2bqtWCggMV_4RoCR2sgwV-EAAYASAAEgLIUvD_BwE" (at -20.32 100.33 0)
+    (property "Supplier" "https://www.digikey.ch/de/products/detail/hirose-electric-co-ltd/DF40C-100DS-0-4V-51/1969476" (at -20.32 100.33 0)
       (effects (font (size 1.27 1.27)) hide)
     )

Commit message: Use CM4 of symbol library
Parts:
- Module1: symbol pedalboard:ComputeModule4-CM4 -> pedalboard:CM4
Changed lines of the file:
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@@
     )
   )
-  (symbol (lib_id "pedalboard:ComputeModule4-CM4") (at -20.32 100.33 0) (unit 2)
+  (symbol (lib_id "pedalboard:CM4") (at -20.32 100.33 0) (unit 2)
     (in_bom yes) (on_board yes) (dnp no) (fields_autoplaced)
     (property "Reference" "Module1" (at 119.38 26.67 0)
