File: connect.kicad_sch (KiCad schematic)
At the start: 1 part

Commit message: Update to V4
Parts:
- renumbered Module1 to CM1

Commit message: First version of USB-Hub
Parts:
- added C11, C25: 27p, Capacitor_SMD:C_0805_2012Metric, symbol Device:C_Small
- added C38, C39, C40, C41, C42: 10u, Capacitor_SMD:C_0805_2012Metric, symbol Device:C_Small
- added C43: 100u, Capacitor_Tantalum_SMD:CP_EIA-7343-31_Kemet-D, symbol Device:CP
- added J10: USB_A_Stacked, symbol Connector:USB_A_Stacked
- added J9: USB_OTG, symbol Connector:USB_OTG
- added R22, R23: 2K2, Resistor_SMD:R_0805_2012Metric, symbol Device:R_Small
- added R24: 12K, Resistor_SMD:R_0805_2012Metric, symbol Device:R_Small
- added R25, R26, R27, R28, R29: 36K, Resistor_SMD:R_0805_2012Metric, symbol Device:R_Small
- added U10: AP2553W6, Package_TO_SOT_SMD:SOT-23-6, symbol pedalboard:AP2553W6
- added U8: FSUSB42MUX, Package_SO:MSOP-10_3x3mm_P0.5mm, symbol Interface_USB:FSUSB42MUX
- added U9: USB2514B_Bi, Package_DFN_QFN:QFN-36-1EP_6x6mm_P0.5mm_EP3.7x3.7mm, symbol Interface_USB:USB2514B_Bi
- added Y1: Crystal_Small, Crystal:Crystal_SMD_HC49-SD, symbol Device:Crystal_Small
Connections:
- net GND: now also C11.2, C25.2, C38.2, C39.2, C40.2, C41.2, C42.2, C43.2, J10.4 (GND1), J10.8 (GND2), J10.9 (Shield), J9.5 (GND), J9.6 (Shield), R23.2, R24.2, R25.2, R26.2, R27.2, R28.2, R29.1, U10.2 (GND), U8.10 (~{OE}), U8.5 (GND), U9.37 (VSS); no longer CM1.101 (USB_OTG_ID)
- net USB2_N: now also U9.8 (USBDM_DN4/PRT_DIS_M4); no longer CM1.103 (USB2_N)
- net USB2_P: now also U9.9 (USBDP_DN4/PRT_DIS_P4); no longer CM1.105 (USB2_P)
- new net: C25.1, U9.32 (XTALOUT), Y1.2
- new net: R26.1, U9.22 (SDA/SMBDATA/NON_REM1)
- new net: R22.2, U8.2 (SEL)
- new net: CM1.105 (USB2_P), U8.3 (D+)
- new net: CM1.103 (USB2_N), U8.4 (D-)
- new net: U8.6 (HSD1-), U9.30 (USBDM_UP)
- new net: U8.7 (HSD1+), U9.31 (USBDP_UP)
- new net: J9.2 (D-), U8.8 (HSD2-)
- new net: J9.3 (D+), U8.9 (HSD2+)
- new net: R24.1, U9.35 (RBIAS)
- new net: CM1.101 (USB_OTG_ID), J9.1 (VBUS), R22.1, R23.1
- new net: R27.1, U9.28 (SUSP_IND/LOCAL_PWR/NON_REM0)
- new net: J10.2 (D1-), U9.1 (USBDM_DN1/PRT_DIS_M1)
- new net: J10.3 (D1+), U9.2 (USBDP_DN1/PRT_DIS_P1)
- new net: J10.6 (D2-), U9.3 (USBDM_DN2/PRT_DIS_M2)
- new net: J10.7 (D2+), U9.4 (USBDP_DN2/PRT_DIS_P2)
- new net: U10.3 (EN), U9.12 (PRTPWR1/BC_EN1)
- new net: R29.2, U10.5 (ILIM)
- new net: C11.1, U9.33 (XTALIN/CLKIN), Y1.1
- new net: R25.1, U9.24 (SCL/SMBCLK/CFG_SEL0)
- new net: R28.1, U9.25 (HS_IND/CFG_SEL1)
- new net +5VP: C38.1, U10.1 (IN)
- new net CM4_3V: U8.1 (VCC), U9.10 (VDDA33), U9.15 (VDD33), U9.23 (VDD33), U9.27 (VBUS_DET), U9.29 (VDDA33), U9.36 (VDDA33), U9.5 (VDDA33)
- new net VBUS: C39.1, C40.1, C41.1, C42.1, C43.1, J10.1 (VBUS1), J10.5 (VBUS2), U10.6 (OUT)
- new net nEXTRST: U9.26 (RESET_N)
- new net nOSC1: U10.4 (nFault), U9.13 (OCS_N1), U9.17 (OCS_N2), U9.19 (OCS_N3), U9.21 (OCS_N4)
- no-connect marks 67 -> 74
Other:
- note removed: "USB_OTG_ID is tied to GND. See Chapter 2.4"
- moved on the sheet: CM1B

Commit message: Make space for USB hub
Parts:
- C11, C25: value 27p -> 18p
- J10: footprint (none) -> Connector_USB:USB_A_CUI_UJ2-ADH-TH_Horizontal_Stacked
- J9: footprint (none) -> Connector_USB:USB_Micro-B_Amphenol_10103594-0001LF_Horizontal
- Y1: footprint Crystal:Crystal_SMD_HC49-SD -> Crystal:Crystal_SMD_5032-2Pin_5.0x3.2mm
Other:
- moved on the sheet: J9
Changed lines of the file:
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@@
 	)
 	(no_connect
-		(at 224.79 48.26)
+		(at 224.79 44.45)
 	)
 	(no_connect
@@
 	(wire
 		(pts
-			(xy 87.63 102.87) (xy 91.44 102.87)
+			(xy 234.95 49.53) (xy 234.95 53.34)
 		)
 		(stroke
@@
 	(wire
 		(pts
-			(xy 219.71 68.58) (xy 219.71 69.85)
+			(xy 87.63 102.87) (xy 91.44 102.87)
 		)
 		(stroke
@@
 	(wire
 		(pts
-			(xy 24.13 102.87) (xy 24.13 110.49)
+			(xy 219.71 68.58) (xy 219.71 69.85)
 		)
 		(stroke
@@
 	(wire
 		(pts
-			(xy 24.13 148.59) (xy 24.13 157.48)
+			(xy 24.13 102.87) (xy 24.13 110.49)
 		)
 		(stroke
@@
 	(wire
 		(pts
-			(xy 214.63 39.37) (xy 214.63 43.18)
+			(xy 24.13 148.59) (xy 24.13 157.48)
 		)
 		(stroke
@@
 	(wire
 		(pts
-			(xy 212.09 45.72) (xy 224.79 45.72)
-		)
-		(stroke
-			(width 0)
-			(type default)
-		)
-	)
-	(wire
-		(pts
 			(xy 130.81 133.35) (xy 157.48 133.35)
 		)
@@
 	(wire
 		(pts
-			(xy 199.39 41.91) (xy 212.09 41.91)
+			(xy 199.39 41.91) (xy 224.79 41.91)
 		)
 		(stroke
@@
 	(wire
 		(pts
-			(xy 199.39 39.37) (xy 214.63 39.37)
+			(xy 199.39 39.37) (xy 224.79 39.37)
 		)
 		(stroke
@@
 	(wire
 		(pts
-			(xy 214.63 43.18) (xy 224.79 43.18)
-		)
-		(stroke
-			(width 0)
-			(type default)
-		)
-	)
-	(wire
-		(pts
 			(xy 213.36 123.19) (xy 243.84 123.19)
 		)
@@
 	(wire
 		(pts
-			(xy 219.71 38.1) (xy 224.79 38.1)
+			(xy 219.71 34.29) (xy 224.79 34.29)
 		)
 		(stroke
@@
 	(wire
 		(pts
-			(xy 219.71 19.05) (xy 219.71 38.1)
+			(xy 219.71 19.05) (xy 219.71 34.29)
 		)
 		(stroke
@@
 	(wire
 		(pts
-			(xy 212.09 41.91) (xy 212.09 45.72)
-		)
-		(stroke
-			(width 0)
-			(type default)
-		)
-	)
-	(wire
-		(pts
-			(xy 232.41 53.34) (xy 234.95 53.34)
-		)
-		(stroke
-			(width 0)
-			(type default)
-		)
-	)
-	(wire
-		(pts
 			(xy 120.65 121.92) (xy 128.27 121.92)
 		)
@@
 	(wire
 		(pts
+			(xy 232.41 49.53) (xy 232.41 53.34)
+		)
+		(stroke
+			(width 0)
+			(type default)
+		)
+	)
+	(wire
+		(pts
 			(xy 260.35 80.01) (xy 264.16 80.01)
 		)
@@
 	(wire
 		(pts
+			(xy 234.95 53.34) (xy 232.41 53.34)
+		)
+		(stroke
+			(width 0)
+			(type default)
+		)
+	)
+	(wire
+		(pts
 			(xy 273.05 80.01) (xy 278.13 80.01)
 		)
@@
 			)
 		)
-		(property "Value" "27p"
+		(property "Value" "18p"
 			(at 131.191 120.523 0)
 			(effects
@@
 			)
 		)
-		(property "Footprint" ""
+		(property "Footprint" "Connector_USB:USB_A_CUI_UJ2-ADH-TH_Horizontal_Stacked"
 			(at 265.43 121.92 0)
 			(effects
@@
 			)
 		)
-		(property "Footprint" "Crystal:Crystal_SMD_HC49-SD"
+		(property "Footprint" "Crystal:Crystal_SMD_5032-2Pin_5.0x3.2mm"
 			(at 120.65 113.03 0)
 			(effects
@@
 			)
 		)
-		(property "Value" "27p"
+		(property "Value" "18p"
 			(at 117.221 120.523 0)
 			(effects
@@
 	(symbol
 		(lib_id "Connector:USB_OTG")
-		(at 232.41 43.18 0)
+		(at 232.41 39.37 0)
 		(mirror y)
 		(unit 1)
@@
 		(dnp no)
 		(property "Reference" "J9"
-			(at 232.41 30.48 0)
+			(at 232.41 26.67 0)
 			(effects
 				(font
@@
 		)
 		(property "Value" "USB_OTG"
-			(at 232.41 33.02 0)
+			(at 232.41 29.21 0)
 			(effects
 				(font
@@
 			)
 		)
-		(property "Footprint" ""
-			(at 228.6 44.45 0)
+		(property "Footprint" "Connector_USB:USB_Micro-B_Amphenol_10103594-0001LF_Horizontal"
+			(at 228.6 40.64 0)
 			(effects
 				(font
@@
 		)
 		(property "Datasheet" "~"
-			(at 228.6 44.45 0)
+			(at 228.6 40.64 0)
 			(effects
 				(font
@@
 		)
 		(property "Description" "USB mini/micro connector"
-			(at 232.41 43.18 0)
+			(at 232.41 39.37 0)
 			(effects
 				(font

Commit message: First routing. Still many issues
Parts:
- removed J10: USB_A_Stacked, Connector_USB:USB_A_CUI_UJ2-ADH-TH_Horizontal_Stacked, symbol Connector:USB_A_Stacked
- added C44, C45: 10u, Capacitor_SMD:C_0805_2012Metric, symbol Device:C_Small
- added C46, C47, C48, C49: 100n, Capacitor_SMD:C_0805_2012Metric, symbol Device:C_Small
- added J10: USB_A, Connector_USB:USB_A_Molex_67643_Horizontal, symbol Connector:USB_A
Connections:
- net CM4_3V: now also C44.1, C45.1, C46.1, C47.1, C48.1, C49.1
- net GND: now also C44.2, C45.2, C46.2, C47.2, C48.2, C49.2, J10.4 (GND), J10.5 (Shield)
- net USB2_N: now also U9.1 (USBDM_DN1/PRT_DIS_M1); no longer U9.8 (USBDM_DN4/PRT_DIS_M4)
- net USB2_P: now also U9.2 (USBDP_DN1/PRT_DIS_P1); no longer U9.9 (USBDP_DN4/PRT_DIS_P4)
- net VBUS: now also J10.1 (VBUS)
- net nOSC1: no longer U9.19 (OCS_N3), U9.21 (OCS_N4)
- net USB_CM_P: now reaches CM1.105 (USB2_P), U8.3 (D+)
- net USB_CM_N: now reaches CM1.103 (USB2_N), U8.4 (D-)
- net USB_UP_N: now reaches U8.6 (HSD1-), U9.30 (USBDM_UP)
- net USB_UP_P: now reaches U8.7 (HSD1+), U9.31 (USBDP_UP)
- net USB_OTG_N: now reaches J9.2 (D-), U8.8 (HSD2-)
- net USB_OTG_P: now reaches J9.3 (D+), U8.9 (HSD2+)
- net USB_OUT_N: now reaches U9.3 (USBDM_DN2/PRT_DIS_M2)
- net USB_OUT_N: now also J10.2 (D-)
- net USB_OUT_P: now reaches U9.4 (USBDP_DN2/PRT_DIS_P2)
- net USB_OUT_P: now also J10.3 (D+)
- no-connect marks 74 -> 79

Commit message: Fix all errors
Parts:
- U8: footprint Package_SO:MSOP-10_3x3mm_P0.5mm -> Package_SO:TSSOP-10_3x3mm_P0.5mm
Changed lines of the file:
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@@
 			)
 		)
-		(property "Footprint" "Package_SO:MSOP-10_3x3mm_P0.5mm"
+		(property "Footprint" "Package_SO:TSSOP-10_3x3mm_P0.5mm"
 			(at 189.23 64.77 0)
 			(effects

Commit message: Switch top layer from +5V to GND
Connections:
- net at U8.2 (SEL): now also CM1.101 (USB_OTG_ID), R22.1, R23.1; no longer R22.2
- new net: J9.1 (VBUS), R22.2
Changed lines of the file:
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@@
 	)
 	(junction
-		(at 158.75 34.29)
-		(diameter 0)
-		(color 0 0 0 0)
-	)
-	(junction
 		(at 91.44 148.59)
 		(diameter 0)
@@
 	)
 	(junction
+		(at 158.75 34.29)
+		(diameter 0)
+		(color 0 0 0 0)
+	)
+	(junction
 		(at 180.34 69.85)
 		(diameter 0)
@@
 	(wire
 		(pts
-			(xy 158.75 34.29) (xy 158.75 19.05)
-		)
-		(stroke
-			(width 0)
-			(type default)
-		)
-	)
-	(wire
-		(pts
 			(xy 254 80.01) (xy 254 78.74)
 		)
@@
 	(wire
 		(pts
-			(xy 165.1 49.53) (xy 158.75 49.53)
+			(xy 158.75 49.53) (xy 179.07 49.53)
 		)
 		(stroke
@@
 	(wire
 		(pts
+			(xy 158.75 19.05) (xy 158.75 24.13)
+		)
+		(stroke
+			(width 0)
+			(type default)
+		)
+	)
+	(wire
+		(pts
 			(xy 62.23 186.69) (xy 71.12 186.69)
 		)
@@
 	(wire
 		(pts
-			(xy 170.18 49.53) (xy 179.07 49.53)
-		)
-		(stroke
-			(width 0)
-			(type default)
-		)
-	)
-	(wire
-		(pts
 			(xy 243.84 105.41) (xy 262.89 105.41)
 		)
@@
 	(wire
 		(pts
+			(xy 158.75 29.21) (xy 158.75 34.29)
+		)
+		(stroke
+			(width 0)
+			(type default)
+		)
+	)
+	(wire
+		(pts
 			(xy 71.12 173.99) (xy 71.12 177.8)
 		)
@@
 	(symbol
 		(lib_id "Device:R_Small")
-		(at 167.64 49.53 90)
+		(at 158.75 26.67 180)
 		(unit 1)
 		(exclude_from_sim no)
@@
 		(fields_autoplaced yes)
 		(property "Reference" "R22"
-			(at 167.64 44.45 90)
+			(at 161.29 25.3999 0)
 			(effects
 				(font
 					(size 1.27 1.27)
 				)
+				(justify right)
 			)
 		)
 		(property "Value" "2K2"
-			(at 167.64 46.99 90)
+			(at 161.29 27.9399 0)
 			(effects
 				(font
 					(size 1.27 1.27)
 				)
+				(justify right)
 			)
 		)
 		(property "Footprint" "Resistor_SMD:R_0805_2012Metric"
-			(at 167.64 51.308 90)
+			(at 160.528 26.67 90)
 			(effects
 				(font
@@
 		)
 		(property "Datasheet" "https://www.seielect.com/catalog/sei-rncp.pdf"
-			(at 167.64 49.53 0)
+			(at 158.75 26.67 0)
 			(effects
 				(font
@@
 		)
 		(property "Description" ""
-			(at 167.64 49.53 0)
+			(at 158.75 26.67 0)
 			(effects
 				(font
@@
 		)
 		(property "Supplier" "https://www.digikey.ch/de/products/detail/stackpole-electronics-inc/RNCP0805FTD1K00/2240229"
-			(at 167.64 49.53 0)
+			(at 158.75 26.67 0)
 			(effects
 				(font

Commit message: 3D model for micro USB connector
Parts:
- J9: footprint Connector_USB:USB_Micro-B_Amphenol_10103594-0001LF_Horizontal -> Pedalboard Library:USB_Micro-B_Amphenol_10103594-0001LF_Horizontal
Changed lines of the file:
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@@
 			)
 		)
-		(property "Footprint" "Connector_USB:USB_Micro-B_Amphenol_10103594-0001LF_Horizontal"
+		(property "Footprint" "Pedalboard Library:USB_Micro-B_Amphenol_10103594-0001LF_Horizontal"
 			(at 228.6 40.64 0)
 			(effects

Commit message: USB grounding option and protection
Parts:
- added C50, C51: 1n, Capacitor_SMD:C_0805_2012Metric, symbol Device:C_Small
- added U11: TPD4EUSB30, Package_SON:USON-10_2.5x1.0mm_P0.5mm, symbol Power_Protection:TPD4EUSB30
Connections:
- net GND: now also C50.2, C51.2, U11.3 (GND), U11.8 (GND); no longer J10.5 (Shield), J9.6 (Shield)
- net USB_OTG_N renamed USB_D_N
- net USB_D_N: now also U11.5 (D2-)
- net USB_OTG_P renamed USB_D_P
- net USB_D_P: now also U11.4 (D2+)
- new net: C51.1, J10.5 (Shield)
- new net: C50.1, J9.6 (Shield)
Other:
- moved on the sheet: C39, C40, C41, C42
