File: connect.kicad_sch (KiCad schematic)
At the start: 32 parts, among them J10 USB_A, J9 USB_OTG, U10 AP2553W6, U11 TPD4EUSB30, U8 FSUSB42MUX, U9 USB2514B_Bi, Y1 Crystal_Small

Commit message: Fix typo and ESC errors
Connections:
- net nOSC1 renamed nOCS1
- no-connect marks 79 -> 82
Changed lines of the file:
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@@
+	)
+	(junction
+		(at 217.17 69.85)
+		(diameter 0)
+		(color 0 0 0 0)
 	)
 	(junction
@@
 	)
 	(junction
-		(at 219.71 69.85)
-		(diameter 0)
-		(color 0 0 0 0)
-	)
-	(junction
 		(at 24.13 133.35)
 		(diameter 0)
@@
 	)
 	(no_connect
+		(at 246.38 36.83)
+	)
+	(no_connect
 		(at 26.67 143.51)
 	)
@@
 	)
 	(no_connect
+		(at 246.38 41.91)
+	)
+	(no_connect
 		(at 26.67 138.43)
 	)
@@
 	)
 	(no_connect
+		(at 213.36 130.81)
+	)
+	(no_connect
 		(at 87.63 100.33)
 	)
@@
 	(wire
 		(pts
-			(xy 219.71 68.58) (xy 219.71 69.85)
+			(xy 217.17 67.31) (xy 217.17 69.85)
 		)
 		(stroke
@@
 	(wire
 		(pts
-			(xy 219.71 69.85) (xy 228.6 69.85)
-		)
-		(stroke
-			(width 0)
-			(type default)
-		)
-	)
-	(wire
-		(pts
 			(xy 26.67 102.87) (xy 24.13 102.87)
 		)
@@
 	(wire
 		(pts
-			(xy 217.17 67.31) (xy 217.17 68.58)
-		)
-		(stroke
-			(width 0)
-			(type default)
-		)
-	)
-	(wire
-		(pts
 			(xy 26.67 118.11) (xy 24.13 118.11)
 		)
@@
 	(wire
 		(pts
+			(xy 217.17 69.85) (xy 228.6 69.85)
+		)
+		(stroke
+			(width 0)
+			(type default)
+		)
+	)
+	(wire
+		(pts
 			(xy 120.65 121.92) (xy 128.27 121.92)
 		)
@@
 		(pts
 			(xy 114.3 113.03) (xy 118.11 113.03)
-		)
-		(stroke
-			(width 0)
-			(type default)
-		)
-	)
-	(wire
-		(pts
-			(xy 217.17 69.85) (xy 219.71 69.85)
-		)
-		(stroke
-			(width 0)
-			(type default)
-		)
-	)
-	(wire
-		(pts
-			(xy 217.17 68.58) (xy 219.71 68.58)
 		)
 		(stroke
@@
 		)
 	)
-	(label "nOSC1"
+	(label "nOCS1"
 		(at 251.46 74.93 180)
 		(fields_autoplaced yes)
@@
 		)
 	)
-	(label "nOSC1"
+	(label "nOCS1"
 		(at 217.17 92.71 0)
 		(fields_autoplaced yes)
@@
 		)
 	)
-	(label "nOSC1"
+	(label "nOCS1"
 		(at 217.17 105.41 0)
 		(fields_autoplaced yes)

Commit message: Connect all OCS pins
Connections:
- net nOCS1: now also U9.19 (OCS_N3), U9.21 (OCS_N4)
- no-connect marks 82 -> 80
Changed lines of the file:
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@@
-	)
-	(no_connect
-		(at 213.36 130.81)
 	)
 	(no_connect
@@
 	)
 	(no_connect
-		(at 213.36 118.11)
-	)
-	(no_connect
 		(at 87.63 46.99)
 	)
@@
 	(wire
 		(pts
+			(xy 213.36 118.11) (xy 218.44 118.11)
+		)
+		(stroke
+			(width 0)
+			(type default)
+		)
+	)
+	(wire
+		(pts
 			(xy 266.7 69.85) (xy 266.7 71.12)
 		)
@@
 	(wire
 		(pts
-			(xy 213.36 105.41) (xy 217.17 105.41)
+			(xy 213.36 105.41) (xy 218.44 105.41)
 		)
 		(stroke
@@
 	(wire
 		(pts
+			(xy 213.36 130.81) (xy 218.44 130.81)
+		)
+		(stroke
+			(width 0)
+			(type default)
+		)
+	)
+	(wire
+		(pts
 			(xy 203.2 49.53) (xy 199.39 49.53)
 		)
@@
 	(wire
 		(pts
-			(xy 213.36 92.71) (xy 217.17 92.71)
+			(xy 213.36 92.71) (xy 218.44 92.71)
 		)
 		(stroke
@@
 		)
 	)
+	(label "nOCS1"
+		(at 218.44 118.11 0)
+		(fields_autoplaced yes)
+		(effects
+			(font
+				(size 1.27 1.27)
+			)
+			(justify left bottom)
+		)
+	)
 	(label "USB_UP_P"
 		(at 172.72 62.23 0)
@@
 	)
 	(label "nOCS1"
-		(at 217.17 92.71 0)
+		(at 218.44 92.71 0)
 		(fields_autoplaced yes)
 		(effects
@@
 	)
 	(label "nOCS1"
-		(at 217.17 105.41 0)
+		(at 218.44 130.81 0)
 		(fields_autoplaced yes)
 		(effects
+			(font
+				(size 1.27 1.27)
+			)
+			(justify left bottom)
+		)
+	)
+	(label "nOCS1"
+		(at 218.44 105.41 0)
+		(fields_autoplaced yes)
+		(effects

Commit message: Add Datasheets
Parts:
- J10: Supplier (none) -> https://www.digikey.ch/de/products/detail/molex/0676433910/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
- J9: Supplier (none) -> https://www.digikey.ch/de/products/detail/amphenol-cs-fci/1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
- U11: Supplier (none) -> https://www.digikey.ch/de/products/detail/texas-instruments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
- U8: Supplier (none) -> https://www.digikey.ch/de/products/detail/onsemi/FSUSB42MUX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
- U9: Supplier (none) -> https://www.digikey.ch/de/products/detail/microchip-technol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
Changed lines of the file:
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@@
 			)
 		)
+		(property "Supplier" "https://www.digikey.ch/de/products/detail/onsemi/FSUSB42MUX/2036916"
+			(at 189.23 44.45 0)
+			(effects
+				(font
+					(size 1.27 1.27)
+				)
+				(hide yes)
+			)
+		)
 		(pin "9"
 		)
@@
 			)
 		)
-		(property "Datasheet" "~"
+		(property "Datasheet" "https://www.molex.com/en-us/products/part-detail/676433910?display=pdf"
 			(at 266.7 104.14 0)
 			(effects
@@
 			)
 		)
+		(property "Supplier" "https://www.digikey.ch/de/products/detail/molex/0676433910/3598521"
+			(at 270.51 102.87 0)
+			(effects
+				(font
+					(size 1.27 1.27)
+				)
+				(hide yes)
+			)
+		)
 		(pin "1"
 		)
@@
 			)
 		)
+		(property "Supplier" "https://www.digikey.ch/de/products/detail/microchip-technology/USB2514B-I-M2/5639468"
+			(at 185.42 107.95 0)
+			(effects
+				(font
+					(size 1.27 1.27)
+				)
+				(hide yes)
+			)
+		)
 		(pin "18"
 		)
@@
 			)
 		)
+		(property "Supplier" "https://www.digikey.ch/de/products/detail/texas-instruments/TPD4EUSB30DQAR/2503665"
+			(at 259.08 39.37 0)
+			(effects
+				(font
+					(size 1.27 1.27)
+				)
+				(hide yes)
+			)
+		)
 		(pin "10"
 		)
@@
 			)
 		)
-		(property "Datasheet" "~"
+		(property "Datasheet" "https://cdn.amphenol-cs.com/media/wysiwyg/files/documentation/datasheet/inputoutput/io_usb_micro.pdf"
 			(at 228.6 40.64 0)
 			(effects
@@
 			(at 232.41 39.37 0)
 			(effects
+				(font
+					(size 1.27 1.27)
+				)
+				(hide yes)
+			)
+		)
+		(property "Supplier" "https://www.digikey.ch/de/products/detail/amphenol-cs-fci/10103594-0001LF/2350351"
+			(at 232.41 39.37 0)
+			(effects

Commit message: Cleanup Crystal oscialltor meta data
Parts:
- Y1: Supplier (none) -> https://www.digikey.ch/en/products/detail/cts-frequency-con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
Changed lines of the file:
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@@
 			)
 		)
-		(property "Datasheet" "~"
+		(property "Datasheet" "https://www.ctscorp.com/Files/DataSheets/Passives/FCP/Crystals/crystals-445-datasheet.pdf"
 			(at 120.65 113.03 0)
 			(effects
@@
 			(at 120.65 113.03 0)
 			(effects
+				(font
+					(size 1.27 1.27)
+				)
+				(hide yes)
+			)
+		)
+		(property "Supplier" "https://www.digikey.ch/en/products/detail/cts-frequency-controls/445C33D24M00000/3135787"
+			(at 120.65 113.03 0)
+			(effects

Commit message: Fix symbol warnings
Parts:
- C43: symbol Device:CP -> Device:C_Polarized
Changed lines of the file:
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@@
 	)
 	(symbol
-		(lib_name "GND_4")
 		(lib_id "power:GND")
 		(at 138.43 106.68 0)
@@
 	)
 	(symbol
-		(lib_name "GND_11")
 		(lib_id "power:GND")
 		(at 86.36 189.23 0)
@@
 	)
 	(symbol
-		(lib_name "GND_1")
 		(lib_id "power:GND")
 		(at 148.59 52.07 0)
@@
 	)
 	(symbol
-		(lib_name "GND_5")
 		(lib_id "power:GND")
 		(at 119.38 137.16 0)
@@
 			)
 		)
-		(property "Description" ""
+		(property "Description" "Power symbol creates a global label with name \"GND\" , ground"
 			(at 24.13 157.48 0)
 			(effects
@@
 	)
 	(symbol
-		(lib_name "GND_9")
 		(lib_id "power:GND")
 		(at 260.35 82.55 0)
@@
 	)
 	(symbol
-		(lib_name "GND_12")
 		(lib_id "power:GND")
 		(at 259.08 52.07 0)
@@
 			)
 		)
-		(property "Description" ""
+		(property "Description" "Power symbol creates a global label with name \"GND\" , ground"
 			(at 91.44 157.48 0)
 			(effects
@@
 	)
 	(symbol
-		(lib_name "GND_3")
 		(lib_id "power:GND")
 		(at 185.42 148.59 0)
@@
 	)
 	(symbol
-		(lib_name "GND_10")
 		(lib_id "power:GND")
 		(at 270.51 120.65 0)
@@
 	)
 	(symbol
-		(lib_name "GND_8")
 		(lib_id "power:GND")
 		(at 223.52 77.47 0)
@@
 	)
 	(symbol
-		(lib_name "GND_6")
 		(lib_id "power:GND")
 		(at 120.65 123.19 0)
@@
 	)
 	(symbol
-		(lib_id "Device:CP")
+		(lib_id "Device:C_Polarized")
 		(at 260.35 73.66 0)
 		(mirror y)
@@
 	)
 	(symbol
-		(lib_name "GND_2")
 		(lib_id "power:GND")
 		(at 189.23 54.61 0)
@@
 	)
 	(symbol
-		(lib_name "GND_7")
 		(lib_id "power:GND")
 		(at 232.41 57.15 0)

Commit message: Rename label
Connections:
- net USB2_N renamed USB_RP_N
- net USB2_P renamed USB_RP_P
Changed lines of the file:
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@@
-		)
-	)
-	(label "USB_RP_P"
-		(at 229.87 87.63 0)
-		(fields_autoplaced yes)
-		(effects
-			(font
-				(size 1.27 1.27)
-			)
-			(justify left bottom)
 		)
 	)
@@
 		)
 	)
-	(label "USB_RP_N"
-		(at 229.87 85.09 0)
-		(fields_autoplaced yes)
-		(effects
-			(font
-				(size 1.27 1.27)
-			)
-			(justify left bottom)
-		)
-	)
 	(label "VBUS"
 		(at 254 69.85 0)
@@
 		)
 	)
-	(hierarchical_label "USB2_P"
+	(hierarchical_label "USB_RP_P"
 		(shape input)
 		(at 240.03 87.63 0)
@@
 		)
 	)
-	(hierarchical_label "USB2_N"
+	(hierarchical_label "USB_RP_N"
 		(shape input)
 		(at 240.03 85.09 0)
